File: ulx3s.sch (KiCad schematic (older format))
At the start: 9 parts, among them U1 LFE5U-25F-6BG381C, U2 ESP-12E

Commit message: labeling GPDI pins (General purpose differential interface)
Parts:
- added OLED1: CONN_01X07, symbol CONN_01X07
Connections:
- net labels added: GPDI_5V, GPDI_CEC, GPDI_CLK_N, GPDI_CLK_P, GPDI_D0_N, GPDI_D0_P, GPDI_D1_N, GPDI_D1_P, GPDI_D2_N, GPDI_D2_P, GPDI_ETH_N, GPDI_ETH_P, GPDI_SCL, GPDI_SDA, OLED_CLK, OLED_CS, OLED_DC, OLED_MOSI, OLED_RES
- wire segments 166 -> 193
Other:
- moved on the sheet: GPDI1
Changed lines of the file:
@@
 L MICRO-HDMI-D GPDI1
 U 1 1 56ACD5D4
-P 6150 4650
-F 0 "GPDI1" H 6150 5700 50  0000 C CNN
-F 1 "MICRO-GPDI-D" V 6250 4650 50  0000 C CNN
-F 2 "micro-hdmi-d:MICRO-HDMI-D" H 6150 4650 60  0001 C CNN
-F 3 "" H 6150 4650 60  0000 C CNN
-	1    6150 4650
+P 5800 4600
+F 0 "GPDI1" H 5800 5650 50  0000 C CNN
+F 1 "MICRO-GPDI-D" V 5900 4600 50  0000 C CNN
+F 2 "micro-hdmi-d:MICRO-HDMI-D" H 5800 4600 60  0001 C CNN
+F 3 "" H 5800 4600 60  0000 C CNN
+	1    5800 4600
 	-1   0    0    -1
 $EndComp
@@
 MTDI
 $Sheet
-S 6800 4650 800  600
+S 7350 4650 800  600
 U 56AC389C
 F0 "gpio" 60
@@
 	0    -1   -1   0
 $EndComp
+$Comp
+L CONN_01X07 OLED1
+U 1 1 58D50BB9
+P 7400 3950
+F 0 "OLED1" H 7400 4350 50  0000 C CNN
+F 1 "CONN_01X07" V 7500 3950 50  0000 C CNN
+F 2 "" H 7400 3950 50  0000 C CNN
+F 3 "" H 7400 3950 50  0000 C CNN
+	1    7400 3950
+	-1   0    0    -1
+$EndComp
+Wire Wire Line
+	7600 3650 7900 3650
+Wire Wire Line
+	7600 3750 8200 3750
+Wire Wire Line
+	7600 3850 8200 3850
+Wire Wire Line
+	7600 3950 8200 3950
+Wire Wire Line
+	7600 4050 8200 4050
+Wire Wire Line
+	7600 4150 8200 4150
+Wire Wire Line
+	7600 4250 8200 4250
+Text Label 7650 3850 0    60   ~ 0
+OLED_CLK
+Text Label 7650 3950 0    60   ~ 0
+OLED_MOSI
+Text Label 7650 4050 0    60   ~ 0
+OLED_RES
+Text Label 7650 4150 0    60   ~ 0
+OLED_DC
+Text Label 7650 4250 0    60   ~ 0
+OLED_CS
+$Comp
+L GND #PWR08
+U 1 1 58D52027
+P 7900 3650
+F 0 "#PWR08" H 7900 3400 50  0001 C CNN
+F 1 "GND" H 7900 3500 50  0000 C CNN
+F 2 "" H 7900 3650 60  0000 C CNN
+F 3 "" H 7900 3650 60  0000 C CNN
+	1    7900 3650
+	0    -1   -1   0
+$EndComp
+$Comp
+L VCC #PWR09
+U 1 1 58D522D3
+P 8200 3750
+F 0 "#PWR09" H 8200 3600 50  0001 C CNN
+F 1 "VCC" H 8200 3900 50  0000 C CNN
+F 2 "" H 8200 3750 50  0000 C CNN
+F 3 "" H 8200 3750 50  0000 C CNN
+	1    8200 3750
+	0    1    1    0
+$EndComp
+Wire Wire Line
+	6000 3650 6700 3650
+Text Label 6050 3650 0    60   ~ 0
+GPDI_ETH_N
+Wire Wire Line
+	6000 3750 6700 3750
+Wire Wire Line
+	6000 3850 6700 3850
+Text Label 6050 3750 0    60   ~ 0
+GPDI_ETH_P
+Wire Wire Line
+	6000 5150 6700 5150
+Wire Wire Line
+	6000 3950 6700 3950
+Wire Wire Line
+	6000 4050 6700 4050
+Text Label 6050 3850 0    60   ~ 0
+GPDI_D2_P
+Text Label 6050 4050 0    60   ~ 0
+GPDI_D2_N
+Wire Wire Line
+	6000 4150 6700 4150
+Wire Wire Line
+	6000 4250 6700 4250
+Wire Wire Line
+	6000 4350 6700 4350
+Text Label 6050 4150 0    60   ~ 0
+GPDI_D1_P
+Text Label 6050 4350 0    60   ~ 0
+GPDI_D1_N
+Wire Wire Line
+	6000 4450 6700 4450
+Wire Wire Line
+	6000 4550 6700 4550
+Wire Wire Line
+	6000 4650 6700 4650
+Text Label 6050 4450 0    60   ~ 0
+GPDI_D0_P
+Text Label 6050 4650 0    60   ~ 0
+GPDI_D0_N
+Wire Wire Line
+	6000 4750 6700 4750
+Wire Wire Line
+	6000 4850 6700 4850
+Wire Wire Line
+	6000 4950 6700 4950
+Text Label 6050 4750 0    60   ~ 0
+GPDI_CLK_P
+Text Label 6050 4950 0    60   ~ 0
+GPDI_CLK_N
+Wire Wire Line
+	6000 5050 6700 5050
+Text Label 6050 5050 0    60   ~ 0
+GPDI_CEC
+Wire Wire Line
+	6000 5250 6700 5250
+Text Label 6050 5250 0    60   ~ 0
+GPDI_SCL
+Text Label 6050 5450 0    60   ~ 0
+GPDI_5V
+Wire Wire Line
+	6000 5450 6700 5450
+Wire Wire Line
+	6000 5350 6700 5350
+Text Label 6050 5350 0    60   ~ 0
+GPDI_SDA
+Wire Wire Line
+	6000 5550 6700 5550
+$Comp
+L GND #PWR010
+U 1 1 58D544FB
+P 6700 5550
+F 0 "#PWR010" H 6700 5300 50  0001 C CNN
+F 1 "GND" H 6700 5400 50  0000 C CNN
+F 2 "" H 6700 5550 60  0000 C CNN
+F 3 "" H 6700 5550 60  0000 C CNN
+	1    6700 5550
+	0    -1   -1   0
+$EndComp
+$Comp
+L GND #PWR011
+U 1 1 58D5464C
+P 6700 5150
+F 0 "#PWR011" H 6700 4900 50  0001 C CNN
+F 1 "GND" H 6700 5000 50  0000 C CNN
+F 2 "" H 6700 5150 60  0000 C CNN
+F 3 "" H 6700 5150 60  0000 C CNN
+	1    6700 5150
+	0    -1   -1   0
+$EndComp
+$Comp
+L GND #PWR012
+U 1 1 58D54683
+P 6700 4850
+F 0 "#PWR012" H 6700 4600 50  0001 C CNN
+F 1 "GND" H 6700 4700 50  0000 C CNN
+F 2 "" H 6700 4850 60  0000 C CNN
+F 3 "" H 6700 4850 60  0000 C CNN
+	1    6700 4850
+	0    -1   -1   0
+$EndComp
+$Comp
+L GND #PWR013
+U 1 1 58D54712
+P 6700 4550
+F 0 "#PWR013" H 6700 4300 50  0001 C CNN
+F 1 "GND" H 6700 4400 50  0000 C CNN
+F 2 "" H 6700 4550 60  0000 C CNN
+F 3 "" H 6700 4550 60  0000 C CNN
+	1    6700 4550
+	0    -1   -1   0
+$EndComp
+$Comp
+L GND #PWR014
+U 1 1 58D54749
+P 6700 4250
+F 0 "#PWR014" H 6700 4000 50  0001 C CNN
+F 1 "GND" H 6700 4100 50  0000 C CNN
+F 2 "" H 6700 4250 60  0000 C CNN
+F 3 "" H 6700 4250 60  0000 C CNN
+	1    6700 4250
+	0    -1   -1   0
+$EndComp
+$Comp
+L GND #PWR015
+U 1 1 58D547C2
+P 6700 3950
+F 0 "#PWR015" H 6700 3700 50  0001 C CNN
+F 1 "GND" H 6700 3800 50  0000 C CNN
+F 2 "" H 6700 3950 60  0000 C CNN
+F 3 "" H 6700 3950 60  0000 C CNN
+	1    6700 3950
+	0    -1   -1   0
+$EndComp
