File: analog.sch (KiCad schematic (older format))
At the start: 14 parts, among them U8 MAX11125

Commit message: schematics: replace 45F chip with 85F
Changed lines of the file:
@@
 $EndComp
 Wire Wire Line
-	2950 2350 3600 2350
+	2950 2350 3500 2350
 Wire Wire Line
 	3500 2200 3600 2200
 Wire Wire Line
-	3500 1900 3500 2350
+	3500 1900 3500 2050
 Connection ~ 3500 2350
 Wire Wire Line
@@
 	3500 2850 3600 2850
 Wire Wire Line
-	3500 2550 3500 3000
+	3500 2550 3500 2700
 Wire Wire Line
 	3500 2700 3600 2700
 Connection ~ 3500 2850
 Wire Wire Line
-	2950 2550 3600 2550
+	2950 2550 3500 2550
 Connection ~ 3500 2700
 Text GLabel 3900 2550 2    60   Input ~ 0
@@
 	3700 4500 3800 4500
 Wire Wire Line
-	3800 4500 3800 5000
+	3800 4500 3800 4600
 Wire Wire Line
 	3800 5000 3700 5000
@@
 Connection ~ 3800 4900
 Wire Wire Line
-	3700 4800 3950 4800
+	3700 4800 3800 4800
 Connection ~ 3800 4800
 Wire Wire Line
@@
 $EndComp
 Wire Wire Line
-	2800 5800 2900 5800
+	2800 5800 2850 5800
 Wire Wire Line
 	2900 5600 2850 5600
 Wire Wire Line
-	2850 5600 2850 5800
+	2850 5600 2850 5700
 Connection ~ 2850 5800
 Wire Wire Line
@@
 $EndComp
 Wire Wire Line
-	2800 4250 2900 4250
+	2800 4250 2850 4250
 Wire Wire Line
 	2850 4250 2850 4350
@@
 $EndComp
 Wire Wire Line
-	2950 1700 3600 1700
+	2950 1700 3500 1700
 Wire Wire Line
 	3500 1550 3600 1550
 Wire Wire Line
-	3500 1250 3500 1700
+	3500 1250 3500 1400
 Connection ~ 3500 1700
 Wire Wire Line
@@
 Wire Wire Line
 	2950 1700 2950 2050
+Wire Wire Line
+	3500 2350 3600 2350
+Wire Wire Line
+	3500 2200 3500 2350
+Wire Wire Line
+	3500 2050 3500 2200
+Wire Wire Line
+	3500 2850 3500 3000
+Wire Wire Line
+	3500 2700 3500 2850
+Wire Wire Line
+	3500 2550 3600 2550
+Wire Wire Line
+	3800 4600 3800 4700
+Wire Wire Line
+	3800 4900 3800 5000
+Wire Wire Line
+	3800 4800 3950 4800
+Wire Wire Line
+	3800 4800 3800 4900
+Wire Wire Line
+	3800 4700 3800 4800
+Wire Wire Line
+	2850 5800 2900 5800
+Wire Wire Line
+	2850 5700 2850 5800
+Wire Wire Line
+	2850 4250 2900 4250
+Wire Wire Line
+	3500 1700 3600 1700
+Wire Wire Line
+	3500 1550 3500 1700
+Wire Wire Line
+	3500 1400 3500 1550
 $EndSCHEMATC

Commit message: schematics: hopefully getting rid of all references to micro-gpdi-d
Parts:
- AUDIO1: symbol micro-hdmi-d:JACK_TRS_6PINS -> jack_trs_6pins:JACK_TRS_6PINS
Changed lines of the file:
@@
 $EndDescr
 $Comp
-L micro-hdmi-d:JACK_TRS_6PINS AUDIO1
+L jack_trs_6pins:JACK_TRS_6PINS AUDIO1
 U 1 1 58D82C05
 P 2550 2350

Commit message: schematics: updating resistor footprints
Parts:
- R14, R15, R16, R17, R18, R19, R20, R21: footprint Resistors_SMD:R_0603_HandSoldering -> Resistor_SMD:R_0603_1608Metric_Pad0.84x1.00mm_HandSolder
- R57, R58, R59, R60: footprint Resistors_SMD:R_0603_HandSoldering -> Resistor_SMD:R_0603_1608Metric
Changed lines of the file:
@@
 F 0 "R17" V 3830 2350 50  0000 C CNN
 F 1 "150" V 3750 2350 50  0000 C CNN
-F 2 "Resistors_SMD:R_0603_HandSoldering" V 3680 2350 50  0001 C CNN
+F 2 "Resistor_SMD:R_0603_1608Metric_Pad0.84x1.00mm_HandSolder" V 3680 2350 50  0001 C CNN
 F 3 "" H 3750 2350 50  0000 C CNN
 	1    3750 2350
@@
 F 0 "R16" V 3830 2200 50  0000 C CNN
 F 1 "330" V 3750 2200 50  0000 C CNN
-F 2 "Resistors_SMD:R_0603_HandSoldering" V 3680 2200 50  0001 C CNN
+F 2 "Resistor_SMD:R_0603_1608Metric_Pad0.84x1.00mm_HandSolder" V 3680 2200 50  0001 C CNN
 F 3 "" H 3750 2200 50  0000 C CNN
 	1    3750 2200
@@
 F 0 "R15" V 3830 2050 50  0000 C CNN
 F 1 "680" V 3750 2050 50  0000 C CNN
-F 2 "Resistors_SMD:R_0603_HandSoldering" V 3680 2050 50  0001 C CNN
+F 2 "Resistor_SMD:R_0603_1608Metric_Pad0.84x1.00mm_HandSolder" V 3680 2050 50  0001 C CNN
 F 3 "" H 3750 2050 50  0000 C CNN
 	1    3750 2050
@@
 F 0 "R14" V 3830 1900 50  0000 C CNN
 F 1 "1.2k" V 3750 1900 50  0000 C CNN
-F 2 "Resistors_SMD:R_0603_HandSoldering" V 3680 1900 50  0001 C CNN
+F 2 "Resistor_SMD:R_0603_1608Metric_Pad0.84x1.00mm_HandSolder" V 3680 1900 50  0001 C CNN
 F 3 "" H 3750 1900 50  0000 C CNN
 	1    3750 1900
@@
 F 0 "R21" V 3830 3000 50  0000 C CNN
 F 1 "150" V 3750 3000 50  0000 C CNN
-F 2 "Resistors_SMD:R_0603_HandSoldering" V 3680 3000 50  0001 C CNN
+F 2 "Resistor_SMD:R_0603_1608Metric_Pad0.84x1.00mm_HandSolder" V 3680 3000 50  0001 C CNN
 F 3 "" H 3750 3000 50  0000 C CNN
 	1    3750 3000
@@
 F 0 "R20" V 3830 2850 50  0000 C CNN
 F 1 "330" V 3750 2850 50  0000 C CNN
-F 2 "Resistors_SMD:R_0603_HandSoldering" V 3680 2850 50  0001 C CNN
+F 2 "Resistor_SMD:R_0603_1608Metric_Pad0.84x1.00mm_HandSolder" V 3680 2850 50  0001 C CNN
 F 3 "" H 3750 2850 50  0000 C CNN
 	1    3750 2850
@@
 F 0 "R19" V 3830 2700 50  0000 C CNN
 F 1 "680" V 3750 2700 50  0000 C CNN
-F 2 "Resistors_SMD:R_0603_HandSoldering" V 3680 2700 50  0001 C CNN
+F 2 "Resistor_SMD:R_0603_1608Metric_Pad0.84x1.00mm_HandSolder" V 3680 2700 50  0001 C CNN
 F 3 "" H 3750 2700 50  0000 C CNN
 	1    3750 2700
@@
 F 0 "R18" V 3830 2550 50  0000 C CNN
 F 1 "1.2k" V 3750 2550 50  0000 C CNN
-F 2 "Resistors_SMD:R_0603_HandSoldering" V 3680 2550 50  0001 C CNN
+F 2 "Resistor_SMD:R_0603_1608Metric_Pad0.84x1.00mm_HandSolder" V 3680 2550 50  0001 C CNN
 F 3 "" H 3750 2550 50  0000 C CNN
 	1    3750 2550
@@
 F 0 "R60" V 3830 1700 50  0000 C CNN
 F 1 "150" V 3750 1700 50  0000 C CNN
-F 2 "Resistors_SMD:R_0603_HandSoldering" V 3680 1700 50  0001 C CNN
+F 2 "Resistor_SMD:R_0603_1608Metric" V 3680 1700 50  0001 C CNN
 F 3 "" H 3750 1700 50  0000 C CNN
 	1    3750 1700
@@
 F 0 "R59" V 3830 1550 50  0000 C CNN
 F 1 "330" V 3750 1550 50  0000 C CNN
-F 2 "Resistors_SMD:R_0603_HandSoldering" V 3680 1550 50  0001 C CNN
+F 2 "Resistor_SMD:R_0603_1608Metric" V 3680 1550 50  0001 C CNN
 F 3 "" H 3750 1550 50  0000 C CNN
 	1    3750 1550
@@
 F 0 "R58" V 3830 1400 50  0000 C CNN
 F 1 "680" V 3750 1400 50  0000 C CNN
-F 2 "Resistors_SMD:R_0603_HandSoldering" V 3680 1400 50  0001 C CNN
+F 2 "Resistor_SMD:R_0603_1608Metric" V 3680 1400 50  0001 C CNN
 F 3 "" H 3750 1400 50  0000 C CNN
 	1    3750 1400
@@
 F 0 "R57" V 3830 1250 50  0000 C CNN
 F 1 "1.2k" V 3750 1250 50  0000 C CNN
-F 2 "Resistors_SMD:R_0603_HandSoldering" V 3680 1250 50  0001 C CNN
+F 2 "Resistor_SMD:R_0603_1608Metric" V 3680 1250 50  0001 C CNN
 F 3 "" H 3750 1250 50  0000 C CNN
 	1    3750 1250

Commit message: schematics: using generalized form of MAX1112x footprint instead of MAX11123
Parts:
- U8: symbol max1112x:MAX11123 -> max1112x:MAX1112x
Changed lines of the file:
@@
 $EndComp
 $Comp
-L max1112x:MAX11123 U8
+L max1112x:MAX1112x U8
 U 1 1 595A6DC1
 P 3300 4900

Commit message: schematics: set part numbers for most resistors
Parts:
- R14, R18: MFG_PN (none) -> RC0603FR-101K2L
- R15, R19, R58: MFG_PN (none) -> RC0603FR-10680RL
- R16, R20, R59: MFG_PN (none) -> RC0603JR-07330RP
- R17, R21, R60: MFG_PN (none) -> AC0603FR-07150RL
- R57: MFG_PN (none) -> RC0603FR-101K2L; MFG_URL (none) -> www.yageo.com
Changed lines of the file:
@@
 F 2 "Resistor_SMD:R_0603_1608Metric_Pad0.84x1.00mm_HandSolder" V 3680 2350 50  0001 C CNN
 F 3 "" H 3750 2350 50  0000 C CNN
+F 4 "AC0603FR-07150RL" V 3750 2350 50  0001 C CNN "MFG_PN"
 	1    3750 2350
 	0    1    1    0
@@
 F 2 "Resistor_SMD:R_0603_1608Metric_Pad0.84x1.00mm_HandSolder" V 3680 2200 50  0001 C CNN
 F 3 "" H 3750 2200 50  0000 C CNN
+F 4 "RC0603JR-07330RP" V 3750 2200 50  0001 C CNN "MFG_PN"
 	1    3750 2200
 	0    1    1    0
@@
 F 2 "Resistor_SMD:R_0603_1608Metric_Pad0.84x1.00mm_HandSolder" V 3680 2050 50  0001 C CNN
 F 3 "" H 3750 2050 50  0000 C CNN
+F 4 "RC0603FR-10680RL" V 3750 2050 50  0001 C CNN "MFG_PN"
 	1    3750 2050
 	0    1    1    0
@@
 F 2 "Resistor_SMD:R_0603_1608Metric_Pad0.84x1.00mm_HandSolder" V 3680 1900 50  0001 C CNN
 F 3 "" H 3750 1900 50  0000 C CNN
+F 4 "RC0603FR-101K2L" V 3750 1900 50  0001 C CNN "MFG_PN"
 	1    3750 1900
 	0    1    1    0
@@
 F 2 "Resistor_SMD:R_0603_1608Metric_Pad0.84x1.00mm_HandSolder" V 3680 3000 50  0001 C CNN
 F 3 "" H 3750 3000 50  0000 C CNN
+F 4 "AC0603FR-07150RL" V 3750 3000 50  0001 C CNN "MFG_PN"
 	1    3750 3000
 	0    1    1    0
@@
 F 2 "Resistor_SMD:R_0603_1608Metric_Pad0.84x1.00mm_HandSolder" V 3680 2850 50  0001 C CNN
 F 3 "" H 3750 2850 50  0000 C CNN
+F 4 "RC0603JR-07330RP" V 3750 2850 50  0001 C CNN "MFG_PN"
 	1    3750 2850
 	0    1    1    0
@@
 F 2 "Resistor_SMD:R_0603_1608Metric_Pad0.84x1.00mm_HandSolder" V 3680 2700 50  0001 C CNN
 F 3 "" H 3750 2700 50  0000 C CNN
+F 4 "RC0603FR-10680RL" V 3750 2700 50  0001 C CNN "MFG_PN"
 	1    3750 2700
 	0    1    1    0
@@
 F 2 "Resistor_SMD:R_0603_1608Metric_Pad0.84x1.00mm_HandSolder" V 3680 2550 50  0001 C CNN
 F 3 "" H 3750 2550 50  0000 C CNN
+F 4 "RC0603FR-101K2L" V 3750 2550 50  0001 C CNN "MFG_PN"
 	1    3750 2550
 	0    1    1    0
@@
 F 2 "Resistor_SMD:R_0603_1608Metric" V 3680 1700 50  0001 C CNN
 F 3 "" H 3750 1700 50  0000 C CNN
+F 4 "AC0603FR-07150RL" V 3750 1700 50  0001 C CNN "MFG_PN"
 	1    3750 1700
 	0    1    1    0
@@
 F 2 "Resistor_SMD:R_0603_1608Metric" V 3680 1550 50  0001 C CNN
 F 3 "" H 3750 1550 50  0000 C CNN
+F 4 "RC0603JR-07330RP" V 3750 1550 50  0001 C CNN "MFG_PN"
 	1    3750 1550
 	0    1    1    0
@@
 F 2 "Resistor_SMD:R_0603_1608Metric" V 3680 1400 50  0001 C CNN
 F 3 "" H 3750 1400 50  0000 C CNN
+F 4 "RC0603FR-10680RL" V 3750 1400 50  0001 C CNN "MFG_PN"
 	1    3750 1400
 	0    1    1    0
@@
 F 2 "Resistor_SMD:R_0603_1608Metric" V 3680 1250 50  0001 C CNN
 F 3 "" H 3750 1250 50  0000 C CNN
+F 4 "www.yageo.com" V 3750 1250 50  0001 C CNN "MFG_URL"
+F 5 "RC0603FR-101K2L" V 3750 1250 50  0001 C CNN "MFG_PN"
 	1    3750 1250
 	0    1    1    0

Commit message: schematics: changing old rescue symbols with new from kicad 5 library
Parts:
- R14, R15, R16, R17, R18, R19, R20, R21, R57, R58, R59, R60: symbol ulx3s-rescue:R -> Device:R
Changed lines of the file:
@@
 $EndComp
 $Comp
-L ulx3s-rescue:R R17
+L Device:R R17
 U 1 1 58D90455
 P 3750 2350
@@
 $EndComp
 $Comp
-L ulx3s-rescue:R R16
+L Device:R R16
 U 1 1 58D904AE
 P 3750 2200
@@
 $EndComp
 $Comp
-L ulx3s-rescue:R R15
+L Device:R R15
 U 1 1 58D904D5
 P 3750 2050
@@
 $EndComp
 $Comp
-L ulx3s-rescue:R R14
+L Device:R R14
 U 1 1 58D90500
 P 3750 1900
@@
 AUDIO_L3
 $Comp
-L ulx3s-rescue:R R21
+L Device:R R21
 U 1 1 58D907CA
 P 3750 3000
@@
 $EndComp
 $Comp
-L ulx3s-rescue:R R20
+L Device:R R20
 U 1 1 58D907D0
 P 3750 2850
@@
 $EndComp
 $Comp
-L ulx3s-rescue:R R19
+L Device:R R19
 U 1 1 58D907D6
 P 3750 2700
@@
 $EndComp
 $Comp
-L ulx3s-rescue:R R18
+L Device:R R18
 U 1 1 58D907DC
 P 3750 2550
@@
 JACK pinout for SJ-43516-SMT-TR\nhttp://www.cui.com/product/resource/sj-4351x-smt-series.pdf\npin 1 - sleeve (GND)\npin 2 - tip (left channel)\npin 3 - ring1 (right channel)\npin 4 - ring2 (video)\npin 5 - tip switch\npin 6 - ring1 switch
 $Comp
-L ulx3s-rescue:R R60
+L Device:R R60
 U 1 1 5A05BC31
 P 3750 1700
@@
 $EndComp
 $Comp
-L ulx3s-rescue:R R59
+L Device:R R59
 U 1 1 5A05BC37
 P 3750 1550
@@
 $EndComp
 $Comp
-L ulx3s-rescue:R R58
+L Device:R R58
 U 1 1 5A05BC3D
 P 3750 1400
@@
 $EndComp
 $Comp
-L ulx3s-rescue:R R57
+L Device:R R57
 U 1 1 5A05BC43
 P 3750 1250

Commit message: schematics: normal (non-handsoldering) footrpints of audio DAC resistors
Parts:
- R14, R15, R16, R17, R18, R19, R20, R21: footprint Resistor_SMD:R_0603_1608Metric_Pad0.84x1.00mm_HandSolder -> Resistor_SMD:R_0603_1608Metric
Changed lines of the file:
@@
 F 0 "R17" V 3830 2350 50  0000 C CNN
 F 1 "150" V 3750 2350 50  0000 C CNN
-F 2 "Resistor_SMD:R_0603_1608Metric_Pad0.84x1.00mm_HandSolder" V 3680 2350 50  0001 C CNN
+F 2 "Resistor_SMD:R_0603_1608Metric" V 3680 2350 50  0001 C CNN
 F 3 "" H 3750 2350 50  0000 C CNN
 F 4 "AC0603FR-07150RL" V 3750 2350 50  0001 C CNN "MFG_PN"
@@
 F 0 "R16" V 3830 2200 50  0000 C CNN
 F 1 "330" V 3750 2200 50  0000 C CNN
-F 2 "Resistor_SMD:R_0603_1608Metric_Pad0.84x1.00mm_HandSolder" V 3680 2200 50  0001 C CNN
+F 2 "Resistor_SMD:R_0603_1608Metric" V 3680 2200 50  0001 C CNN
 F 3 "" H 3750 2200 50  0000 C CNN
 F 4 "RC0603JR-07330RP" V 3750 2200 50  0001 C CNN "MFG_PN"
@@
 F 0 "R15" V 3830 2050 50  0000 C CNN
 F 1 "680" V 3750 2050 50  0000 C CNN
-F 2 "Resistor_SMD:R_0603_1608Metric_Pad0.84x1.00mm_HandSolder" V 3680 2050 50  0001 C CNN
+F 2 "Resistor_SMD:R_0603_1608Metric" V 3680 2050 50  0001 C CNN
 F 3 "" H 3750 2050 50  0000 C CNN
 F 4 "RC0603FR-10680RL" V 3750 2050 50  0001 C CNN "MFG_PN"
@@
 F 0 "R14" V 3830 1900 50  0000 C CNN
 F 1 "1.2k" V 3750 1900 50  0000 C CNN
-F 2 "Resistor_SMD:R_0603_1608Metric_Pad0.84x1.00mm_HandSolder" V 3680 1900 50  0001 C CNN
+F 2 "Resistor_SMD:R_0603_1608Metric" V 3680 1900 50  0001 C CNN
 F 3 "" H 3750 1900 50  0000 C CNN
 F 4 "RC0603FR-101K2L" V 3750 1900 50  0001 C CNN "MFG_PN"
@@
 F 0 "R21" V 3830 3000 50  0000 C CNN
 F 1 "150" V 3750 3000 50  0000 C CNN
-F 2 "Resistor_SMD:R_0603_1608Metric_Pad0.84x1.00mm_HandSolder" V 3680 3000 50  0001 C CNN
+F 2 "Resistor_SMD:R_0603_1608Metric" V 3680 3000 50  0001 C CNN
 F 3 "" H 3750 3000 50  0000 C CNN
 F 4 "AC0603FR-07150RL" V 3750 3000 50  0001 C CNN "MFG_PN"
@@
 F 0 "R20" V 3830 2850 50  0000 C CNN
 F 1 "330" V 3750 2850 50  0000 C CNN
-F 2 "Resistor_SMD:R_0603_1608Metric_Pad0.84x1.00mm_HandSolder" V 3680 2850 50  0001 C CNN
+F 2 "Resistor_SMD:R_0603_1608Metric" V 3680 2850 50  0001 C CNN
 F 3 "" H 3750 2850 50  0000 C CNN
 F 4 "RC0603JR-07330RP" V 3750 2850 50  0001 C CNN "MFG_PN"
@@
 F 0 "R19" V 3830 2700 50  0000 C CNN
 F 1 "680" V 3750 2700 50  0000 C CNN
-F 2 "Resistor_SMD:R_0603_1608Metric_Pad0.84x1.00mm_HandSolder" V 3680 2700 50  0001 C CNN
+F 2 "Resistor_SMD:R_0603_1608Metric" V 3680 2700 50  0001 C CNN
 F 3 "" H 3750 2700 50  0000 C CNN
 F 4 "RC0603FR-10680RL" V 3750 2700 50  0001 C CNN "MFG_PN"
@@
 F 0 "R18" V 3830 2550 50  0000 C CNN
 F 1 "1.2k" V 3750 2550 50  0000 C CNN
-F 2 "Resistor_SMD:R_0603_1608Metric_Pad0.84x1.00mm_HandSolder" V 3680 2550 50  0001 C CNN
+F 2 "Resistor_SMD:R_0603_1608Metric" V 3680 2550 50  0001 C CNN
 F 3 "" H 3750 2550 50  0000 C CNN
 F 4 "RC0603FR-101K2L" V 3750 2550 50  0001 C CNN "MFG_PN"

Commit message: schematics: MFG_URL for R,C
Parts:
- R58, R59, R60: MFG_URL (none) -> www.yageo.com
Changed lines of the file:
@@
 F 2 "Resistor_SMD:R_0603_1608Metric" V 3680 1700 50  0001 C CNN
 F 3 "" H 3750 1700 50  0000 C CNN
-F 4 "AC0603FR-07150RL" V 3750 1700 50  0001 C CNN "MFG_PN"
+F 4 "www.yageo.com" V 3750 1700 50  0001 C CNN "MFG_URL"
+F 5 "AC0603FR-07150RL" V 3750 1700 50  0001 C CNN "MFG_PN"
 	1    3750 1700
 	0    1    1    0
@@
 F 2 "Resistor_SMD:R_0603_1608Metric" V 3680 1550 50  0001 C CNN
 F 3 "" H 3750 1550 50  0000 C CNN
-F 4 "RC0603JR-07330RP" V 3750 1550 50  0001 C CNN "MFG_PN"
+F 4 "www.yageo.com" V 3750 1550 50  0001 C CNN "MFG_URL"
+F 5 "RC0603JR-07330RP" V 3750 1550 50  0001 C CNN "MFG_PN"
 	1    3750 1550
 	0    1    1    0
@@
 F 2 "Resistor_SMD:R_0603_1608Metric" V 3680 1400 50  0001 C CNN
 F 3 "" H 3750 1400 50  0000 C CNN
-F 4 "RC0603FR-10680RL" V 3750 1400 50  0001 C CNN "MFG_PN"
+F 4 "www.yageo.com" V 3750 1400 50  0001 C CNN "MFG_URL"
+F 5 "RC0603FR-10680RL" V 3750 1400 50  0001 C CNN "MFG_PN"
 	1    3750 1400
 	0    1    1    0
