File: analog.sch (KiCad schematic (older format))
At the start: 14 parts, among them U8 MAX11125

Commit message: schematics: change filed names for parts BOM suitable for 1-click-bom.tsv MFG_PN->MPN, Distributor1_PN->Mouser, Distributor1_URL->Mouser_URL
Parts:
- AUDIO1: Distributor1_PN 490-SJ-43516-SMT-TR -> (none); Distributor1_URL www.mouser.com -> (none); MFG_PN SJ-43516-SMT-TR -> (none); MPN (none) -> SJ-43516-SMT-TR; Mouser (none) -> 490-SJ-43516-SMT-TR; Mouser_URL (none) -> www.mouser.com
- R14, R18, R57: MFG_PN RC0603FR-101K2L -> (none); MPN (none) -> RC0603FR-101K2L
- R15, R19, R58: MFG_PN RC0603FR-10680RL -> (none); MPN (none) -> RC0603FR-10680RL
- R16, R20, R59: MFG_PN RC0603JR-07330RP -> (none); MPN (none) -> RC0603JR-07330RP
- R17, R21, R60: MFG_PN AC0603FR-07150RL -> (none); MPN (none) -> AC0603FR-07150RL
- U8: Distributor1_PN 700-MAX11125ATI+ -> (none); Distributor1_URL www.mouser.com -> (none); MFG_PN MAX11125ATI+ -> (none); MPN (none) -> MAX11125ATI+; Mouser (none) -> 700-MAX11125ATI+; Mouser_URL (none) -> www.mouser.com
Changed lines of the file:
@@
 F 3 "http://www.cui.com/product/resource/sj-4351x-smt-series.pdf" H 2650 2200 50  0001 C CNN
 F 4 "www.cui.com" H 2550 2350 60  0001 C CNN "MFG_URL"
-F 5 "SJ-43516-SMT-TR" H 2550 2350 60  0001 C CNN "MFG_PN"
-F 6 "www.mouser.com" H 2550 2350 60  0001 C CNN "Distributor1_URL"
-F 7 "490-SJ-43516-SMT-TR " H 2550 2350 60  0001 C CNN "Distributor1_PN"
+F 5 "SJ-43516-SMT-TR" H 2550 2350 60  0001 C CNN "MPN"
+F 6 "www.mouser.com" H 2550 2350 60  0001 C CNN "Mouser_URL"
+F 7 "490-SJ-43516-SMT-TR " H 2550 2350 60  0001 C CNN "Mouser"
 	1    2550 2350
 	1    0    0    -1
@@
 F 2 "Resistor_SMD:R_0603_1608Metric" V 3680 2350 50  0001 C CNN
 F 3 "" H 3750 2350 50  0000 C CNN
-F 4 "AC0603FR-07150RL" V 3750 2350 50  0001 C CNN "MFG_PN"
+F 4 "AC0603FR-07150RL" V 3750 2350 50  0001 C CNN "MPN"
 	1    3750 2350
 	0    1    1    0
@@
 F 2 "Resistor_SMD:R_0603_1608Metric" V 3680 2200 50  0001 C CNN
 F 3 "" H 3750 2200 50  0000 C CNN
-F 4 "RC0603JR-07330RP" V 3750 2200 50  0001 C CNN "MFG_PN"
+F 4 "RC0603JR-07330RP" V 3750 2200 50  0001 C CNN "MPN"
 	1    3750 2200
 	0    1    1    0
@@
 F 2 "Resistor_SMD:R_0603_1608Metric" V 3680 2050 50  0001 C CNN
 F 3 "" H 3750 2050 50  0000 C CNN
-F 4 "RC0603FR-10680RL" V 3750 2050 50  0001 C CNN "MFG_PN"
+F 4 "RC0603FR-10680RL" V 3750 2050 50  0001 C CNN "MPN"
 	1    3750 2050
 	0    1    1    0
@@
 F 2 "Resistor_SMD:R_0603_1608Metric" V 3680 1900 50  0001 C CNN
 F 3 "" H 3750 1900 50  0000 C CNN
-F 4 "RC0603FR-101K2L" V 3750 1900 50  0001 C CNN "MFG_PN"
+F 4 "RC0603FR-101K2L" V 3750 1900 50  0001 C CNN "MPN"
 	1    3750 1900
 	0    1    1    0
@@
 F 2 "Resistor_SMD:R_0603_1608Metric" V 3680 3000 50  0001 C CNN
 F 3 "" H 3750 3000 50  0000 C CNN
-F 4 "AC0603FR-07150RL" V 3750 3000 50  0001 C CNN "MFG_PN"
+F 4 "AC0603FR-07150RL" V 3750 3000 50  0001 C CNN "MPN"
 	1    3750 3000
 	0    1    1    0
@@
 F 2 "Resistor_SMD:R_0603_1608Metric" V 3680 2850 50  0001 C CNN
 F 3 "" H 3750 2850 50  0000 C CNN
-F 4 "RC0603JR-07330RP" V 3750 2850 50  0001 C CNN "MFG_PN"
+F 4 "RC0603JR-07330RP" V 3750 2850 50  0001 C CNN "MPN"
 	1    3750 2850
 	0    1    1    0
@@
 F 2 "Resistor_SMD:R_0603_1608Metric" V 3680 2700 50  0001 C CNN
 F 3 "" H 3750 2700 50  0000 C CNN
-F 4 "RC0603FR-10680RL" V 3750 2700 50  0001 C CNN "MFG_PN"
+F 4 "RC0603FR-10680RL" V 3750 2700 50  0001 C CNN "MPN"
 	1    3750 2700
 	0    1    1    0
@@
 F 2 "Resistor_SMD:R_0603_1608Metric" V 3680 2550 50  0001 C CNN
 F 3 "" H 3750 2550 50  0000 C CNN
-F 4 "RC0603FR-101K2L" V 3750 2550 50  0001 C CNN "MFG_PN"
+F 4 "RC0603FR-101K2L" V 3750 2550 50  0001 C CNN "MPN"
 	1    3750 2550
 	0    1    1    0
@@
 F 3 "https://datasheets.maximintegrated.com/en/ds/MAX11120-MAX11128.pdf" H 3300 4950 50  0001 C CNN
 F 4 "www.maximintegrated.com" H 3300 4900 60  0001 C CNN "MFG_URL"
-F 5 "MAX11125ATI+" H 3300 4900 60  0001 C CNN "MFG_PN"
-F 6 "www.mouser.com" H 3300 4900 60  0001 C CNN "Distributor1_URL"
-F 7 "700-MAX11125ATI+" H 3300 4900 60  0001 C CNN "Distributor1_PN"
+F 5 "MAX11125ATI+" H 3300 4900 60  0001 C CNN "MPN"
+F 6 "www.mouser.com" H 3300 4900 60  0001 C CNN "Mouser_URL"
+F 7 "700-MAX11125ATI+" H 3300 4900 60  0001 C CNN "Mouser"
 	1    3300 4900
 	1    0    0    -1
@@
 F 3 "" H 3750 1700 50  0000 C CNN
 F 4 "www.yageo.com" V 3750 1700 50  0001 C CNN "MFG_URL"
-F 5 "AC0603FR-07150RL" V 3750 1700 50  0001 C CNN "MFG_PN"
+F 5 "AC0603FR-07150RL" V 3750 1700 50  0001 C CNN "MPN"
 	1    3750 1700
 	0    1    1    0
@@
 F 3 "" H 3750 1550 50  0000 C CNN
 F 4 "www.yageo.com" V 3750 1550 50  0001 C CNN "MFG_URL"
-F 5 "RC0603JR-07330RP" V 3750 1550 50  0001 C CNN "MFG_PN"
+F 5 "RC0603JR-07330RP" V 3750 1550 50  0001 C CNN "MPN"
 	1    3750 1550
 	0    1    1    0
@@
 F 3 "" H 3750 1400 50  0000 C CNN
 F 4 "www.yageo.com" V 3750 1400 50  0001 C CNN "MFG_URL"
-F 5 "RC0603FR-10680RL" V 3750 1400 50  0001 C CNN "MFG_PN"
+F 5 "RC0603FR-10680RL" V 3750 1400 50  0001 C CNN "MPN"
 	1    3750 1400
 	0    1    1    0
@@
 F 3 "" H 3750 1250 50  0000 C CNN
 F 4 "www.yageo.com" V 3750 1250 50  0001 C CNN "MFG_URL"
-F 5 "RC0603FR-101K2L" V 3750 1250 50  0001 C CNN "MFG_PN"
+F 5 "RC0603FR-101K2L" V 3750 1250 50  0001 C CNN "MPN"
 	1    3750 1250
 	0    1    1    0

Commit message: schematics: Mouser PN for R,C,BTN
Parts:
- R14: Mouser (none) -> 603-RC0603FR-101K2L
- R15: Mouser (none) -> 603-RC0603FR-10680RL
- R16: Mouser (none) -> 603-RC0603JR-07330RP
Changed lines of the file:
@@
 F 3 "" H 3750 2200 50  0000 C CNN
 F 4 "RC0603JR-07330RP" V 3750 2200 50  0001 C CNN "MPN"
+F 5 "603-RC0603JR-07330RP" V 3750 2200 50  0001 C CNN "Mouser"
 	1    3750 2200
 	0    1    1    0
@@
 F 3 "" H 3750 2050 50  0000 C CNN
 F 4 "RC0603FR-10680RL" V 3750 2050 50  0001 C CNN "MPN"
+F 5 "603-RC0603FR-10680RL" V 3750 2050 50  0001 C CNN "Mouser"
 	1    3750 2050
 	0    1    1    0
@@
 F 3 "" H 3750 1900 50  0000 C CNN
 F 4 "RC0603FR-101K2L" V 3750 1900 50  0001 C CNN "MPN"
+F 5 "603-RC0603FR-101K2L" V 3750 1900 50  0001 C CNN "Mouser"
 	1    3750 1900
 	0    1    1    0

Commit message: schematics: Digikey PN for most parts except R
Parts:
- AUDIO1: Digikey (none) -> CP-43516SJCT-ND
- U8: Digikey (none) -> MAX11125ATI+-ND
Changed lines of the file:
@@
 F 6 "www.mouser.com" H 2550 2350 60  0001 C CNN "Mouser_URL"
 F 7 "490-SJ-43516-SMT-TR " H 2550 2350 60  0001 C CNN "Mouser"
+F 8 "CP-43516SJCT-ND" H 2550 2350 50  0001 C CNN "Digikey"
 	1    2550 2350
 	1    0    0    -1
@@
 F 6 "www.mouser.com" H 3300 4900 60  0001 C CNN "Mouser_URL"
 F 7 "700-MAX11125ATI+" H 3300 4900 60  0001 C CNN "Mouser"
+F 8 "MAX11125ATI+-ND" H 3300 4900 50  0001 C CNN "Digikey"
 	1    3300 4900
 	1    0    0    -1

Commit message: schematics: rename MFG_URL -> MFG1_URL
Parts:
- AUDIO1: MFG1_URL (none) -> www.cui.com; MFG_URL www.cui.com -> (none)
- R57, R58, R59, R60: MFG1_URL (none) -> www.yageo.com; MFG_URL www.yageo.com -> (none)
- U8: MFG1_URL (none) -> www.maximintegrated.com; MFG_URL www.maximintegrated.com -> (none)
Changed lines of the file:
@@
 F 2 "audio-jack:CUI_SJ-43516-SMT" H 2650 2200 50  0001 C CNN
 F 3 "http://www.cui.com/product/resource/sj-4351x-smt-series.pdf" H 2650 2200 50  0001 C CNN
-F 4 "www.cui.com" H 2550 2350 60  0001 C CNN "MFG_URL"
+F 4 "www.cui.com" H 2550 2350 60  0001 C CNN "MFG1_URL"
 F 5 "SJ-43516-SMT-TR" H 2550 2350 60  0001 C CNN "MPN"
 F 6 "www.mouser.com" H 2550 2350 60  0001 C CNN "Mouser_URL"
@@
 F 2 "Housings_DFN_QFN:QFN-28-1EP_5x5mm_Pitch0.5mm" H 3300 4950 50  0001 C CNN
 F 3 "https://datasheets.maximintegrated.com/en/ds/MAX11120-MAX11128.pdf" H 3300 4950 50  0001 C CNN
-F 4 "www.maximintegrated.com" H 3300 4900 60  0001 C CNN "MFG_URL"
+F 4 "www.maximintegrated.com" H 3300 4900 60  0001 C CNN "MFG1_URL"
 F 5 "MAX11125ATI+" H 3300 4900 60  0001 C CNN "MPN"
 F 6 "www.mouser.com" H 3300 4900 60  0001 C CNN "Mouser_URL"
@@
 F 2 "Resistor_SMD:R_0603_1608Metric" V 3680 1700 50  0001 C CNN
 F 3 "" H 3750 1700 50  0000 C CNN
-F 4 "www.yageo.com" V 3750 1700 50  0001 C CNN "MFG_URL"
+F 4 "www.yageo.com" V 3750 1700 50  0001 C CNN "MFG1_URL"
 F 5 "AC0603FR-07150RL" V 3750 1700 50  0001 C CNN "MPN"
 	1    3750 1700
@@
 F 2 "Resistor_SMD:R_0603_1608Metric" V 3680 1550 50  0001 C CNN
 F 3 "" H 3750 1550 50  0000 C CNN
-F 4 "www.yageo.com" V 3750 1550 50  0001 C CNN "MFG_URL"
+F 4 "www.yageo.com" V 3750 1550 50  0001 C CNN "MFG1_URL"
 F 5 "RC0603JR-07330RP" V 3750 1550 50  0001 C CNN "MPN"
 	1    3750 1550
@@
 F 2 "Resistor_SMD:R_0603_1608Metric" V 3680 1400 50  0001 C CNN
 F 3 "" H 3750 1400 50  0000 C CNN
-F 4 "www.yageo.com" V 3750 1400 50  0001 C CNN "MFG_URL"
+F 4 "www.yageo.com" V 3750 1400 50  0001 C CNN "MFG1_URL"
 F 5 "RC0603FR-10680RL" V 3750 1400 50  0001 C CNN "MPN"
 	1    3750 1400
@@
 F 2 "Resistor_SMD:R_0603_1608Metric" V 3680 1250 50  0001 C CNN
 F 3 "" H 3750 1250 50  0000 C CNN
-F 4 "www.yageo.com" V 3750 1250 50  0001 C CNN "MFG_URL"
+F 4 "www.yageo.com" V 3750 1250 50  0001 C CNN "MFG1_URL"
 F 5 "RC0603FR-101K2L" V 3750 1250 50  0001 C CNN "MPN"
 	1    3750 1250

Commit message: schematics: add alternate PNs for some parts
Parts:
- U8: MFG2_URL (none) -> www.maximintegrated.com; MPN2 (none) -> MAX11123ATI+; Mouser2 (none) -> 700-MAX11123ATI+
Changed lines of the file:
@@
 F 4 "www.maximintegrated.com" H 3300 4900 60  0001 C CNN "MFG1_URL"
 F 5 "MAX11125ATI+" H 3300 4900 60  0001 C CNN "MPN"
-F 6 "www.mouser.com" H 3300 4900 60  0001 C CNN "Mouser_URL"
-F 7 "700-MAX11125ATI+" H 3300 4900 60  0001 C CNN "Mouser"
-F 8 "MAX11125ATI+-ND" H 3300 4900 50  0001 C CNN "Digikey"
+F 6 "www.maximintegrated.com" H 3300 4900 50  0001 C CNN "MFG2_URL"
+F 7 "MAX11123ATI+" H 3300 4900 50  0001 C CNN "MPN2"
+F 8 "www.mouser.com" H 3300 4900 60  0001 C CNN "Mouser_URL"
+F 9 "700-MAX11125ATI+" H 3300 4900 60  0001 C CNN "Mouser"
+F 10 "700-MAX11123ATI+" H 3300 4900 50  0001 C CNN "Mouser2"
+F 11 "MAX11125ATI+-ND" H 3300 4900 50  0001 C CNN "Digikey"
 	1    3300 4900
 	1    0    0    -1

Commit message: schematics: Digikey PN for R
Parts:
- R57: Digikey (none) -> 311-1.20KHRCT-ND
- R58: Digikey (none) -> 311-680HRCT-ND
- R59: Digikey (none) -> YAG1298CT-ND
- R60: Digikey (none) -> 311-150HRCT-ND
Changed lines of the file:
@@
 F 4 "www.yageo.com" V 3750 1700 50  0001 C CNN "MFG1_URL"
 F 5 "AC0603FR-07150RL" V 3750 1700 50  0001 C CNN "MPN"
+F 6 "311-150HRCT-ND" V 3750 1700 50  0001 C CNN "Digikey"
 	1    3750 1700
 	0    1    1    0
@@
 F 4 "www.yageo.com" V 3750 1550 50  0001 C CNN "MFG1_URL"
 F 5 "RC0603JR-07330RP" V 3750 1550 50  0001 C CNN "MPN"
+F 6 "YAG1298CT-ND" V 3750 1550 50  0001 C CNN "Digikey"
 	1    3750 1550
 	0    1    1    0
@@
 F 4 "www.yageo.com" V 3750 1400 50  0001 C CNN "MFG1_URL"
 F 5 "RC0603FR-10680RL" V 3750 1400 50  0001 C CNN "MPN"
+F 6 "311-680HRCT-ND" V 3750 1400 50  0001 C CNN "Digikey"
 	1    3750 1400
 	0    1    1    0
@@
 F 4 "www.yageo.com" V 3750 1250 50  0001 C CNN "MFG1_URL"
 F 5 "RC0603FR-101K2L" V 3750 1250 50  0001 C CNN "MPN"
+F 6 "311-1.20KHRCT-ND" V 3750 1250 50  0001 C CNN "Digikey"
 	1    3750 1250
 	0    1    1    0

Commit message: schematics: updating available PN for R,C
Parts:
- R14: Digikey (none) -> 311-1.20KHRCT-ND; Mouser 603-RC0603FR-101K2L -> 603-AC0603JR-071K2L
- R57: Digikey 311-1.20KHRCT-ND -> (none)
Changed lines of the file:
@@
 F 3 "" H 3750 1900 50  0000 C CNN
 F 4 "RC0603FR-101K2L" V 3750 1900 50  0001 C CNN "MPN"
-F 5 "603-RC0603FR-101K2L" V 3750 1900 50  0001 C CNN "Mouser"
+F 5 "603-AC0603JR-071K2L" V 3750 1900 50  0001 C CNN "Mouser"
+F 6 "311-1.20KHRCT-ND" V 3750 1900 50  0001 C CNN "Digikey"
 	1    3750 1900
 	0    1    1    0
@@
 F 4 "www.yageo.com" V 3750 1250 50  0001 C CNN "MFG1_URL"
 F 5 "RC0603FR-101K2L" V 3750 1250 50  0001 C CNN "MPN"
-F 6 "311-1.20KHRCT-ND" V 3750 1250 50  0001 C CNN "Digikey"
 	1    3750 1250
 	0    1    1    0

Commit message: schematics: experimentally renaming MFG1_URL->MNF1_URL to not be recognized as manufacturer name
Parts:
- AUDIO1: MFG1 (none) -> CUI; MFG1_URL www.cui.com -> (none); MNF1_URL (none) -> www.cui.com
Changed lines of the file:
@@
 F 2 "audio-jack:CUI_SJ-43516-SMT" H 2650 2200 50  0001 C CNN
 F 3 "http://www.cui.com/product/resource/sj-4351x-smt-series.pdf" H 2650 2200 50  0001 C CNN
-F 4 "www.cui.com" H 2550 2350 60  0001 C CNN "MFG1_URL"
-F 5 "SJ-43516-SMT-TR" H 2550 2350 60  0001 C CNN "MPN"
-F 6 "www.mouser.com" H 2550 2350 60  0001 C CNN "Mouser_URL"
-F 7 "490-SJ-43516-SMT-TR " H 2550 2350 60  0001 C CNN "Mouser"
-F 8 "CP-43516SJCT-ND" H 2550 2350 50  0001 C CNN "Digikey"
+F 4 "www.cui.com" H 2550 2350 60  0001 C CNN "MNF1_URL"
+F 5 "CUI" H 2550 2350 50  0001 C CNN "MFG1"
+F 6 "SJ-43516-SMT-TR" H 2550 2350 60  0001 C CNN "MPN"
+F 7 "www.mouser.com" H 2550 2350 60  0001 C CNN "Mouser_URL"
+F 8 "490-SJ-43516-SMT-TR " H 2550 2350 60  0001 C CNN "Mouser"
+F 9 "CP-43516SJCT-ND" H 2550 2350 50  0001 C CNN "Digikey"
 	1    2550 2350
 	1    0    0    -1
