File: analog.sch (KiCad schematic (older format))
At the start: 17 parts, among them U8 MAX11125

Commit message: schematics: corrected Mouser PN for 680 ohm (was 680K)
Parts:
- R15: Mouser 603-AC0603FR-07680KL -> 652-CR0603FX-5900ELF; Mouser3 (none) -> 603-RC0603FR-07680RL
Changed lines of the file:
@@
 F 3 "" H 3750 2050 50  0000 C CNN
 F 4 "RC0603FR-10680RL" V 3750 2050 50  0001 C CNN "MPN"
-F 5 "603-AC0603FR-07680KL" V 3750 2050 50  0001 C CNN "Mouser"
+F 5 "652-CR0603FX-5900ELF" V 3750 2050 50  0001 C CNN "Mouser"
 F 6 "603-RC0603FR-10680RL" V 3750 2050 50  0001 C CNN "Mouser2"
-F 7 "FR012" V 3750 2050 50  0001 C CNN "Koncar"
-F 8 "TB" V 3750 2050 50  0001 C CNN "Side"
+F 7 "603-RC0603FR-07680RL" V 3750 2050 50  0001 C CNN "Mouser3"
+F 8 "FR012" V 3750 2050 50  0001 C CNN "Koncar"
+F 9 "TB" V 3750 2050 50  0001 C CNN "Side"
 	1    3750 2050
 	0    1    1    0

Commit message: schematics: change resistor value 680->590 ohm to improve DAC
Parts:
- R15, R19, R58: value 680 -> 590
Changed lines of the file:
@@
 P 3750 2050
 F 0 "R15" V 3830 2050 50  0000 C CNN
-F 1 "680" V 3750 2050 50  0000 C CNN
+F 1 "590" V 3750 2050 50  0000 C CNN
 F 2 "Resistor_SMD:R_0603_1608Metric" V 3680 2050 50  0001 C CNN
 F 3 "" H 3750 2050 50  0000 C CNN
@@
 P 3750 2700
 F 0 "R19" V 3830 2700 50  0000 C CNN
-F 1 "680" V 3750 2700 50  0000 C CNN
+F 1 "590" V 3750 2700 50  0000 C CNN
 F 2 "Resistor_SMD:R_0603_1608Metric" V 3680 2700 50  0001 C CNN
 F 3 "" H 3750 2700 50  0000 C CNN
@@
 P 3750 1400
 F 0 "R58" V 3830 1400 50  0000 C CNN
-F 1 "680" V 3750 1400 50  0000 C CNN
+F 1 "590" V 3750 1400 50  0000 C CNN
 F 2 "Resistor_SMD:R_0603_1608Metric" V 3680 1400 50  0001 C CNN
 F 3 "" H 3750 1400 50  0000 C CNN

Commit message: schematics: change resistor value 330->300 ohm to improve DAC
Parts:
- R15: MPN RC0603FR-10680RL -> CR0603-FX-5900ELF
- R16: value 330 -> 300; Mouser 603-RC0603JR-07330RP -> 603-RC0603FR-10300RL; Mouser2 (none) -> 603-RC0603JR-07330RP
- R20, R59: value 330 -> 300
Changed lines of the file:
@@
 P 3750 2200
 F 0 "R16" V 3830 2200 50  0000 C CNN
-F 1 "330" V 3750 2200 50  0000 C CNN
+F 1 "300" V 3750 2200 50  0000 C CNN
 F 2 "Resistor_SMD:R_0603_1608Metric" V 3680 2200 50  0001 C CNN
 F 3 "" H 3750 2200 50  0000 C CNN
 F 4 "RC0603JR-07330RP" V 3750 2200 50  0001 C CNN "MPN"
-F 5 "603-RC0603JR-07330RP" V 3750 2200 50  0001 C CNN "Mouser"
-F 6 "FR010" V 3750 2200 50  0001 C CNN "Koncar"
+F 5 "603-RC0603FR-10300RL" V 3750 2200 50  0001 C CNN "Mouser"
+F 6 "603-RC0603JR-07330RP" V 3750 2200 50  0001 C CNN "Mouser2"
+F 7 "FR010" V 3750 2200 50  0001 C CNN "Koncar"
 	1    3750 2200
 	0    1    1    0
@@
 F 2 "Resistor_SMD:R_0603_1608Metric" V 3680 2050 50  0001 C CNN
 F 3 "" H 3750 2050 50  0000 C CNN
-F 4 "RC0603FR-10680RL" V 3750 2050 50  0001 C CNN "MPN"
+F 4 "CR0603-FX-5900ELF" V 3750 2050 50  0001 C CNN "MPN"
 F 5 "652-CR0603FX-5900ELF" V 3750 2050 50  0001 C CNN "Mouser"
 F 6 "603-RC0603FR-10680RL" V 3750 2050 50  0001 C CNN "Mouser2"
@@
 P 3750 2850
 F 0 "R20" V 3830 2850 50  0000 C CNN
-F 1 "330" V 3750 2850 50  0000 C CNN
+F 1 "300" V 3750 2850 50  0000 C CNN
 F 2 "Resistor_SMD:R_0603_1608Metric" V 3680 2850 50  0001 C CNN
 F 3 "" H 3750 2850 50  0000 C CNN
@@
 P 3750 1550
 F 0 "R59" V 3830 1550 50  0000 C CNN
-F 1 "330" V 3750 1550 50  0000 C CNN
+F 1 "300" V 3750 1550 50  0000 C CNN
 F 2 "Resistor_SMD:R_0603_1608Metric" V 3680 1550 50  0001 C CNN
 F 3 "" H 3750 1550 50  0000 C CNN

Commit message: schematics: DAC closer to 75 ohm impedance: 130, 270, 550 ohm
Parts:
- R14: MNF1_URL (none) -> www.yageo.com
- R15: value 590 -> 550; Digikey (none) -> 311-549HRCT-ND; MNF1_URL (none) -> www.yageo.com; MPN CR0603-FX-5900ELF -> RC0603FR-07549RL; Mouser 652-CR0603FX-5900ELF -> 603-RC0603FR-07549RL; Mouser2 603-RC0603FR-10680RL -> (none); Mouser3 603-RC0603FR-07680RL -> (none)
- R16: value 300 -> 270; Digikey (none) -> 311-270HRCT-ND; MNF1_URL (none) -> www.yageo.com; Mouser2 603-RC0603JR-07330RP -> (none)
- R17: value 150 -> 130; Digikey (none) -> 311-130HRCT-ND; MNF1_URL (none) -> www.yageo.com; MPN (none) -> RC0603FR-07130RL; Mouser (none) -> 603-RC0603FR-07130RL
- R18: MPN RC0603FR-101K2L -> (none)
- R19: value 590 -> 550; MPN RC0603FR-10680RL -> (none)
- R20: value 300 -> 270; MPN RC0603JR-07330RP -> (none)
- R21: value 150 -> 130
- R57: MNF1_URL www.yageo.com -> (none); MPN RC0603FR-101K2L -> (none)
- R58: value 590 -> 550; Digikey 311-680HRCT-ND -> (none); MNF1_URL www.yageo.com -> (none); MPN RC0603FR-10680RL -> (none)
- R59: value 300 -> 270; Digikey YAG1298CT-ND -> (none); MNF1_URL www.yageo.com -> (none); MPN RC0603JR-07330RP -> (none)
- R60: value 150 -> 130; MNF1_URL www.yageo.com -> (none)
Other:
- note added: "Output resistance: 75 ohm\nInternal resistance of FPGA pin: 10 ohm\n1/(1/(130+10)+1/(270+10)+1/(550+10)+1/(1190+10))=75"
Changed lines of the file:
@@
 P 3750 2350
 F 0 "R17" V 3830 2350 50  0000 C CNN
-F 1 "150" V 3750 2350 50  0000 C CNN
+F 1 "130" V 3750 2350 50  0000 C CNN
 F 2 "Resistor_SMD:R_0603_1608Metric" V 3680 2350 50  0001 C CNN
 F 3 "" H 3750 2350 50  0000 C CNN
-F 4 "FR004" V 3750 2350 50  0001 C CNN "Koncar"
+F 4 "www.yageo.com" V 3750 2350 50  0001 C CNN "MNF1_URL"
+F 5 "RC0603FR-07130RL" V 3750 2350 50  0001 C CNN "MPN"
+F 6 "603-RC0603FR-07130RL" V 3750 2350 50  0001 C CNN "Mouser"
+F 7 "311-130HRCT-ND" V 3750 2350 50  0001 C CNN "Digikey"
+F 8 "FR004" V 3750 2350 50  0001 C CNN "Koncar"
 	1    3750 2350
 	0    1    1    0
@@
 P 3750 2200
 F 0 "R16" V 3830 2200 50  0000 C CNN
-F 1 "300" V 3750 2200 50  0000 C CNN
+F 1 "270" V 3750 2200 50  0000 C CNN
 F 2 "Resistor_SMD:R_0603_1608Metric" V 3680 2200 50  0001 C CNN
 F 3 "" H 3750 2200 50  0000 C CNN
-F 4 "RC0603JR-07330RP" V 3750 2200 50  0001 C CNN "MPN"
-F 5 "603-RC0603FR-10300RL" V 3750 2200 50  0001 C CNN "Mouser"
-F 6 "603-RC0603JR-07330RP" V 3750 2200 50  0001 C CNN "Mouser2"
-F 7 "FR010" V 3750 2200 50  0001 C CNN "Koncar"
+F 4 "www.yageo.com" V 3750 2200 50  0001 C CNN "MNF1_URL"
+F 5 "RC0603JR-07330RP" V 3750 2200 50  0001 C CNN "MPN"
+F 6 "603-RC0603FR-10300RL" V 3750 2200 50  0001 C CNN "Mouser"
+F 7 "311-270HRCT-ND" V 3750 2200 50  0001 C CNN "Digikey"
+F 8 "FR010" V 3750 2200 50  0001 C CNN "Koncar"
 	1    3750 2200
 	0    1    1    0
@@
 P 3750 2050
 F 0 "R15" V 3830 2050 50  0000 C CNN
-F 1 "590" V 3750 2050 50  0000 C CNN
+F 1 "550" V 3750 2050 50  0000 C CNN
 F 2 "Resistor_SMD:R_0603_1608Metric" V 3680 2050 50  0001 C CNN
 F 3 "" H 3750 2050 50  0000 C CNN
-F 4 "CR0603-FX-5900ELF" V 3750 2050 50  0001 C CNN "MPN"
-F 5 "652-CR0603FX-5900ELF" V 3750 2050 50  0001 C CNN "Mouser"
-F 6 "603-RC0603FR-10680RL" V 3750 2050 50  0001 C CNN "Mouser2"
-F 7 "603-RC0603FR-07680RL" V 3750 2050 50  0001 C CNN "Mouser3"
+F 4 "www.yageo.com" V 3750 2050 50  0001 C CNN "MNF1_URL"
+F 5 "RC0603FR-07549RL" V 3750 2050 50  0001 C CNN "MPN"
+F 6 "603-RC0603FR-07549RL" V 3750 2050 50  0001 C CNN "Mouser"
+F 7 "311-549HRCT-ND" V 3750 2050 50  0001 C CNN "Digikey"
 F 8 "FR012" V 3750 2050 50  0001 C CNN "Koncar"
 F 9 "TB" V 3750 2050 50  0001 C CNN "Side"
@@
 F 2 "Resistor_SMD:R_0603_1608Metric" V 3680 1900 50  0001 C CNN
 F 3 "" H 3750 1900 50  0000 C CNN
-F 4 "RC0603FR-101K2L" V 3750 1900 50  0001 C CNN "MPN"
-F 5 "603-AC0603JR-071K2L" V 3750 1900 50  0001 C CNN "Mouser"
-F 6 "311-1.20KHRCT-ND" V 3750 1900 50  0001 C CNN "Digikey"
-F 7 "FR002" V 3750 1900 50  0001 C CNN "Koncar"
+F 4 "www.yageo.com" V 3750 1900 50  0001 C CNN "MNF1_URL"
+F 5 "RC0603FR-101K2L" V 3750 1900 50  0001 C CNN "MPN"
+F 6 "603-AC0603JR-071K2L" V 3750 1900 50  0001 C CNN "Mouser"
+F 7 "311-1.20KHRCT-ND" V 3750 1900 50  0001 C CNN "Digikey"
+F 8 "FR002" V 3750 1900 50  0001 C CNN "Koncar"
 	1    3750 1900
 	0    1    1    0
@@
 P 3750 3000
 F 0 "R21" V 3830 3000 50  0000 C CNN
-F 1 "150" V 3750 3000 50  0000 C CNN
+F 1 "130" V 3750 3000 50  0000 C CNN
 F 2 "Resistor_SMD:R_0603_1608Metric" V 3680 3000 50  0001 C CNN
 F 3 "" H 3750 3000 50  0000 C CNN
@@
 P 3750 2850
 F 0 "R20" V 3830 2850 50  0000 C CNN
-F 1 "300" V 3750 2850 50  0000 C CNN
+F 1 "270" V 3750 2850 50  0000 C CNN
 F 2 "Resistor_SMD:R_0603_1608Metric" V 3680 2850 50  0001 C CNN
 F 3 "" H 3750 2850 50  0000 C CNN
-F 4 "RC0603JR-07330RP" V 3750 2850 50  0001 C CNN "MPN"
 	1    3750 2850
 	0    1    1    0
@@
 P 3750 2700
 F 0 "R19" V 3830 2700 50  0000 C CNN
-F 1 "590" V 3750 2700 50  0000 C CNN
+F 1 "550" V 3750 2700 50  0000 C CNN
 F 2 "Resistor_SMD:R_0603_1608Metric" V 3680 2700 50  0001 C CNN
 F 3 "" H 3750 2700 50  0000 C CNN
-F 4 "RC0603FR-10680RL" V 3750 2700 50  0001 C CNN "MPN"
 	1    3750 2700
 	0    1    1    0
@@
 F 2 "Resistor_SMD:R_0603_1608Metric" V 3680 2550 50  0001 C CNN
 F 3 "" H 3750 2550 50  0000 C CNN
-F 4 "RC0603FR-101K2L" V 3750 2550 50  0001 C CNN "MPN"
 	1    3750 2550
 	0    1    1    0
@@
 P 3750 1700
 F 0 "R60" V 3830 1700 50  0000 C CNN
-F 1 "150" V 3750 1700 50  0000 C CNN
+F 1 "130" V 3750 1700 50  0000 C CNN
 F 2 "Resistor_SMD:R_0603_1608Metric" V 3680 1700 50  0001 C CNN
 F 3 "" H 3750 1700 50  0000 C CNN
-F 4 "www.yageo.com" V 3750 1700 50  0001 C CNN "MNF1_URL"
 	1    3750 1700
 	0    1    1    0
@@
 P 3750 1550
 F 0 "R59" V 3830 1550 50  0000 C CNN
-F 1 "300" V 3750 1550 50  0000 C CNN
+F 1 "270" V 3750 1550 50  0000 C CNN
 F 2 "Resistor_SMD:R_0603_1608Metric" V 3680 1550 50  0001 C CNN
 F 3 "" H 3750 1550 50  0000 C CNN
-F 4 "www.yageo.com" V 3750 1550 50  0001 C CNN "MNF1_URL"
-F 5 "RC0603JR-07330RP" V 3750 1550 50  0001 C CNN "MPN"
-F 6 "YAG1298CT-ND" V 3750 1550 50  0001 C CNN "Digikey"
 	1    3750 1550
 	0    1    1    0
@@
 P 3750 1400
 F 0 "R58" V 3830 1400 50  0000 C CNN
-F 1 "590" V 3750 1400 50  0000 C CNN
+F 1 "550" V 3750 1400 50  0000 C CNN
 F 2 "Resistor_SMD:R_0603_1608Metric" V 3680 1400 50  0001 C CNN
 F 3 "" H 3750 1400 50  0000 C CNN
-F 4 "www.yageo.com" V 3750 1400 50  0001 C CNN "MNF1_URL"
-F 5 "RC0603FR-10680RL" V 3750 1400 50  0001 C CNN "MPN"
-F 6 "311-680HRCT-ND" V 3750 1400 50  0001 C CNN "Digikey"
 	1    3750 1400
 	0    1    1    0
@@
 F 2 "Resistor_SMD:R_0603_1608Metric" V 3680 1250 50  0001 C CNN
 F 3 "" H 3750 1250 50  0000 C CNN
-F 4 "www.yageo.com" V 3750 1250 50  0001 C CNN "MNF1_URL"
-F 5 "RC0603FR-101K2L" V 3750 1250 50  0001 C CNN "MPN"
 	1    3750 1250
 	0    1    1    0
@@
 NoConn ~ 2900 5350
 NoConn ~ 3700 5100
+Text Notes 2950 3500 0    60   ~ 0
+Output resistance: 75 ohm\nInternal resistance of FPGA pin: 10 ohm\n1/(1/(130+10)+1/(270+10)+1/(550+10)+1/(1190+10))=75
 $EndSCHEMATC

Commit message: schematics: updating DAC 550->549 ohm, 1.2k->1.1k
Parts:
- R14: value 1.2k -> 1.1k; Digikey 311-1.20KHRCT-ND -> P1.10KHCT-ND; MPN RC0603FR-101K2L -> RC0603FR-071K1L; Mouser 603-AC0603JR-071K2L -> 603-RC0603FR-071K1L
- R15, R19, R58: value 550 -> 549
- R18, R57: value 1.2k -> 1.1k
Other:
- note added: "Output resistance: 75 ohm\nInternal resistance of FPGA pin: 10 ohm\n1/(1/(130+10)+1/(270+10)+1/(549+10)+1/(1100+10))=74.6"
- note removed: "Output resistance: 75 ohm\nInternal resistance of FPGA pin: 10 ohm\n1/(1/(130+10)+1/(270+10)+1/(550+10)+1/(1190+10))=75"
Changed lines of the file:
@@
 P 3750 2050
 F 0 "R15" V 3830 2050 50  0000 C CNN
-F 1 "550" V 3750 2050 50  0000 C CNN
+F 1 "549" V 3750 2050 50  0000 C CNN
 F 2 "Resistor_SMD:R_0603_1608Metric" V 3680 2050 50  0001 C CNN
 F 3 "" H 3750 2050 50  0000 C CNN
@@
 P 3750 1900
 F 0 "R14" V 3830 1900 50  0000 C CNN
-F 1 "1.2k" V 3750 1900 50  0000 C CNN
+F 1 "1.1k" V 3750 1900 50  0000 C CNN
 F 2 "Resistor_SMD:R_0603_1608Metric" V 3680 1900 50  0001 C CNN
 F 3 "" H 3750 1900 50  0000 C CNN
 F 4 "www.yageo.com" V 3750 1900 50  0001 C CNN "MNF1_URL"
-F 5 "RC0603FR-101K2L" V 3750 1900 50  0001 C CNN "MPN"
-F 6 "603-AC0603JR-071K2L" V 3750 1900 50  0001 C CNN "Mouser"
-F 7 "311-1.20KHRCT-ND" V 3750 1900 50  0001 C CNN "Digikey"
+F 5 " RC0603FR-071K1L" V 3750 1900 50  0001 C CNN "MPN"
+F 6 "603-RC0603FR-071K1L" V 3750 1900 50  0001 C CNN "Mouser"
+F 7 "P1.10KHCT-ND" V 3750 1900 50  0001 C CNN "Digikey"
 F 8 "FR002" V 3750 1900 50  0001 C CNN "Koncar"
 	1    3750 1900
@@
 P 3750 2700
 F 0 "R19" V 3830 2700 50  0000 C CNN
-F 1 "550" V 3750 2700 50  0000 C CNN
+F 1 "549" V 3750 2700 50  0000 C CNN
 F 2 "Resistor_SMD:R_0603_1608Metric" V 3680 2700 50  0001 C CNN
 F 3 "" H 3750 2700 50  0000 C CNN
@@
 P 3750 2550
 F 0 "R18" V 3830 2550 50  0000 C CNN
-F 1 "1.2k" V 3750 2550 50  0000 C CNN
+F 1 "1.1k" V 3750 2550 50  0000 C CNN
 F 2 "Resistor_SMD:R_0603_1608Metric" V 3680 2550 50  0001 C CNN
 F 3 "" H 3750 2550 50  0000 C CNN
@@
 P 3750 1400
 F 0 "R58" V 3830 1400 50  0000 C CNN
-F 1 "550" V 3750 1400 50  0000 C CNN
+F 1 "549" V 3750 1400 50  0000 C CNN
 F 2 "Resistor_SMD:R_0603_1608Metric" V 3680 1400 50  0001 C CNN
 F 3 "" H 3750 1400 50  0000 C CNN
@@
 P 3750 1250
 F 0 "R57" V 3830 1250 50  0000 C CNN
-F 1 "1.2k" V 3750 1250 50  0000 C CNN
+F 1 "1.1k" V 3750 1250 50  0000 C CNN
 F 2 "Resistor_SMD:R_0603_1608Metric" V 3680 1250 50  0001 C CNN
 F 3 "" H 3750 1250 50  0000 C CNN
@@
 NoConn ~ 3700 5100
 Text Notes 2950 3500 0    60   ~ 0
-Output resistance: 75 ohm\nInternal resistance of FPGA pin: 10 ohm\n1/(1/(130+10)+1/(270+10)+1/(550+10)+1/(1190+10))=75
+Output resistance: 75 ohm\nInternal resistance of FPGA pin: 10 ohm\n1/(1/(130+10)+1/(270+10)+1/(549+10)+1/(1100+10))=74.6
 $EndSCHEMATC

Commit message: schematics: correct 270 ohm PN
Parts:
- R16: MPN RC0603JR-07330RP -> RC0603FR-07270RL; Mouser 603-RC0603FR-10300RL -> 603-RC0603FR-07270RL
Changed lines of the file:
@@
 F 3 "" H 3750 2200 50  0000 C CNN
 F 4 "www.yageo.com" V 3750 2200 50  0001 C CNN "MNF1_URL"
-F 5 "RC0603JR-07330RP" V 3750 2200 50  0001 C CNN "MPN"
-F 6 "603-RC0603FR-10300RL" V 3750 2200 50  0001 C CNN "Mouser"
+F 5 "RC0603FR-07270RL" V 3750 2200 50  0001 C CNN "MPN"
+F 6 "603-RC0603FR-07270RL" V 3750 2200 50  0001 C CNN "Mouser"
 F 7 "311-270HRCT-ND" V 3750 2200 50  0001 C CNN "Digikey"
 F 8 "FR010" V 3750 2200 50  0001 C CNN "Koncar"

Commit message: schematics: cheaper manufacturers PNs and some prices
Parts:
- AUDIO1: Vertical (none) -> SJ-43516-SMT-TR; Vertical_price100 (none) -> 0.8015$
- U8: Digikey_price100 (none) -> 2.92$
Changed lines of the file:
@@
 F 8 "490-SJ-43516-SMT-TR " H 2300 2350 60  0001 C CNN "Mouser"
 F 9 "CP-43516SJCT-ND" H 2300 2350 50  0001 C CNN "Digikey"
-F 10 "FAU001" H 2300 2350 50  0001 C CNN "Koncar"
-F 11 "T" H 2300 2350 50  0001 C CNN "Side"
+F 10 "SJ-43516-SMT-TR" H 2300 2350 50  0001 C CNN "Vertical"
+F 11 "0.8015$" H 2300 2350 50  0001 C CNN "Vertical_price100"
+F 12 "FAU001" H 2300 2350 50  0001 C CNN "Koncar"
+F 13 "T" H 2300 2350 50  0001 C CNN "Side"
 	1    2300 2350
 	1    0    0    -1
@@
 F 11 "700-MAX11123ATI+" H 3300 4900 50  0001 C CNN "Mouser2"
 F 12 "MAX11125ATI+-ND" H 3300 4900 50  0001 C CNN "Digikey"
-F 13 "700-MAX11123ATI+" H 3300 4900 50  0001 C CNN "LowCost"
-F 14 "FU005" H 3300 4900 50  0001 C CNN "Koncar"
-F 15 "T" H 3300 4900 50  0001 C CNN "Side"
+F 13 "2.92$" H 3300 4900 50  0001 C CNN "Digikey_price100"
+F 14 "700-MAX11123ATI+" H 3300 4900 50  0001 C CNN "LowCost"
+F 15 "FU005" H 3300 4900 50  0001 C CNN "Koncar"
+F 16 "T" H 3300 4900 50  0001 C CNN "Side"
 	1    3300 4900
 	1    0    0    -1

Commit message: renaming *_price -> price_* fields that may be misinterpreted by 1-clock-bom
Parts:
- AUDIO1: Vertical_price100 0.8015$ -> (none); price100_Vertical (none) -> 0.8015$
- U8: Digikey_price100 2.92$ -> (none); price100_Digikey (none) -> 2.92$
Changed lines of the file:
@@
 F 9 "CP-43516SJCT-ND" H 2300 2350 50  0001 C CNN "Digikey"
 F 10 "SJ-43516-SMT-TR" H 2300 2350 50  0001 C CNN "Vertical"
-F 11 "0.8015$" H 2300 2350 50  0001 C CNN "Vertical_price100"
+F 11 "0.8015$" H 2300 2350 50  0001 C CNN "price100_Vertical"
 F 12 "FAU001" H 2300 2350 50  0001 C CNN "Koncar"
 F 13 "T" H 2300 2350 50  0001 C CNN "Side"
@@
 F 11 "700-MAX11123ATI+" H 3300 4900 50  0001 C CNN "Mouser2"
 F 12 "MAX11125ATI+-ND" H 3300 4900 50  0001 C CNN "Digikey"
-F 13 "2.92$" H 3300 4900 50  0001 C CNN "Digikey_price100"
+F 13 "2.92$" H 3300 4900 50  0001 C CNN "price100_Digikey"
 F 14 "700-MAX11123ATI+" H 3300 4900 50  0001 C CNN "LowCost"
 F 15 "FU005" H 3300 4900 50  0001 C CNN "Koncar"
