File: wifi.sch (KiCad schematic (older format))
At the start: 5 parts, among them J3 WIFI_OFF, U9 ESP-WROOM-32

Commit message: schematics: hopefully getting rid of all references to micro-gpdi-d
Parts:
- J3: footprint Socket_Strips:Socket_Strip_Straight_2x01 -> Connector_PinHeader_2.54mm:PinHeader_1x02_P2.54mm_Horizontal; symbol micro-hdmi-d:CONN_02X01 -> Connector_Generic:Conn_02x01
Changed lines of the file:
@@
 $EndComp
 $Comp
-L micro-hdmi-d:CONN_02X01 J3
+L Connector_Generic:Conn_02x01 J3
 U 1 1 58EE29FF
-P 4550 3250
-F 0 "J3" H 4550 3350 50  0000 C CNN
-F 1 "WIFI_OFF" H 4550 3150 50  0000 C CNN
-F 2 "Socket_Strips:Socket_Strip_Straight_2x01" H 4550 2050 50  0001 C CNN
-F 3 "" H 4550 2050 50  0000 C CNN
-F 4 "Do not install" H 4550 3250 60  0001 C CNN "Note"
-	1    4550 3250
+P 4550 3200
+F 0 "J3" H 4550 3300 50  0000 C CNN
+F 1 "WIFI_OFF" H 4550 3100 50  0000 C CNN
+F 2 "Connector_PinHeader_2.54mm:PinHeader_1x02_P2.54mm_Horizontal" H 4550 2000 50  0001 C CNN
+F 3 "" H 4550 2000 50  0000 C CNN
+F 4 "Do not install" H 4550 3200 60  0001 C CNN "Note"
+	1    4550 3200
 	0    1    1    0
 $EndComp

Commit message: schematics: updating resistor footprints
Parts:
- R34, R35: footprint Resistors_SMD:R_0603_HandSoldering -> Resistor_SMD:R_0603_1608Metric_Pad0.84x1.00mm_HandSolder
Changed lines of the file:
@@
 F 0 "R34" V 4630 2350 50  0000 C CNN
 F 1 "15k" V 4550 2350 50  0000 C CNN
-F 2 "Resistors_SMD:R_0603_HandSoldering" V 4480 2350 50  0001 C CNN
+F 2 "Resistor_SMD:R_0603_1608Metric_Pad0.84x1.00mm_HandSolder" V 4480 2350 50  0001 C CNN
 F 3 "" H 4550 2350 50  0000 C CNN
 	1    4550 2350
@@
 F 0 "R35" V 4630 2750 50  0000 C CNN
 F 1 "470" V 4550 2750 50  0000 C CNN
-F 2 "Resistors_SMD:R_0603_HandSoldering" V 4480 2750 50  0001 C CNN
+F 2 "Resistor_SMD:R_0603_1608Metric_Pad0.84x1.00mm_HandSolder" V 4480 2750 50  0001 C CNN
 F 3 "" H 4550 2750 50  0000 C CNN
 	1    4550 2750

Commit message: schematics: Remove "Do not install" from ESP32
Parts:
- U9: Note Do not install -> (none)
Changed lines of the file:
@@
 F 5 "ESP-WROOM-32" H 6650 3450 60  0001 C CNN "MFG_PN"
 F 6 "www.mouser.com" H 6650 3450 60  0001 C CNN "Distributor1_URL"
-F 7 "Do not install" H 6650 3450 60  0001 C CNN "Note"
 	1    6650 3450
 	1    0    0    -1

Commit message: schematics: change to vertical pin headers (for silkscreen)
Parts:
- J3: footprint Connector_PinHeader_2.54mm:PinHeader_1x02_P2.54mm_Horizontal -> Connector_PinHeader_2.54mm:PinHeader_1x02_P2.54mm_Vertical
Changed lines of the file:
@@
 F 0 "J3" H 4550 3300 50  0000 C CNN
 F 1 "WIFI_OFF" H 4550 3100 50  0000 C CNN
-F 2 "Connector_PinHeader_2.54mm:PinHeader_1x02_P2.54mm_Horizontal" H 4550 2000 50  0001 C CNN
+F 2 "Connector_PinHeader_2.54mm:PinHeader_1x02_P2.54mm_Vertical" H 4550 2000 50  0001 C CNN
 F 3 "" H 4550 2000 50  0000 C CNN
 F 4 "Do not install" H 4550 3200 60  0001 C CNN "Note"

Commit message: schematics: updating R,C part numbers
Parts:
- C21: MFG_PN (none) -> CC0805ZKY5V5BB226
- R34: MFG_PN (none) -> AC0603FR-1015KL
- R35: MFG_PN (none) -> RC0603FR-07470RL
Changed lines of the file:
@@
 F 2 "Resistor_SMD:R_0603_1608Metric_Pad0.84x1.00mm_HandSolder" V 4480 2350 50  0001 C CNN
 F 3 "" H 4550 2350 50  0000 C CNN
+F 4 "AC0603FR-1015KL" V 4550 2350 50  0001 C CNN "MFG_PN"
 	1    4550 2350
 	1    0    0    -1
@@
 F 2 "Resistor_SMD:R_0603_1608Metric_Pad0.84x1.00mm_HandSolder" V 4480 2750 50  0001 C CNN
 F 3 "" H 4550 2750 50  0000 C CNN
+F 4 "RC0603FR-07470RL" V 4550 2750 50  0001 C CNN "MFG_PN"
 	1    4550 2750
 	1    0    0    -1
@@
 F 2 "Capacitor_SMD:C_0805_2012Metric" H 3688 2950 50  0001 C CNN
 F 3 "" H 3650 3100 50  0000 C CNN
+F 4 "CC0805ZKY5V5BB226" H 3650 3100 50  0001 C CNN "MFG_PN"
 	1    3650 3100
 	1    0    0    -1

Commit message: schematics: changing old rescue symbols with new from kicad 5 library
Parts:
- C21: symbol ulx3s-rescue:C -> Device:C
- R34, R35: symbol ulx3s-rescue:R -> Device:R
Changed lines of the file:
@@
 $EndComp
 $Comp
-L ulx3s-rescue:R R34
+L Device:R R34
 U 1 1 58ED6C6D
 P 4550 2350
@@
 Programming pins:\nTXD RXD EN GPIO0
 $Comp
-L ulx3s-rescue:R R35
+L Device:R R35
 U 1 1 58FD4C5D
 P 4550 2750
@@
 $EndComp
 $Comp
-L ulx3s-rescue:C C21
+L Device:C C21
 U 1 1 5924A09B
 P 3650 3100

Commit message: schematics: MFG_URL for R,C
Parts:
- C21, R34: MFG_URL (none) -> www.yageo.com
- R35: footprint Resistor_SMD:R_0603_1608Metric_Pad0.84x1.00mm_HandSolder -> Resistor_SMD:R_0603_1608Metric; MFG_URL (none) -> www.yageo.com
Changed lines of the file:
@@
 F 2 "Resistor_SMD:R_0603_1608Metric_Pad0.84x1.00mm_HandSolder" V 4480 2350 50  0001 C CNN
 F 3 "" H 4550 2350 50  0000 C CNN
-F 4 "AC0603FR-1015KL" V 4550 2350 50  0001 C CNN "MFG_PN"
+F 4 "www.yageo.com" V 4550 2350 50  0001 C CNN "MFG_URL"
+F 5 "AC0603FR-1015KL" V 4550 2350 50  0001 C CNN "MFG_PN"
 	1    4550 2350
 	1    0    0    -1
@@
 F 0 "R35" V 4630 2750 50  0000 C CNN
 F 1 "470" V 4550 2750 50  0000 C CNN
-F 2 "Resistor_SMD:R_0603_1608Metric_Pad0.84x1.00mm_HandSolder" V 4480 2750 50  0001 C CNN
+F 2 "Resistor_SMD:R_0603_1608Metric" V 4480 2750 50  0001 C CNN
 F 3 "" H 4550 2750 50  0000 C CNN
-F 4 "RC0603FR-07470RL" V 4550 2750 50  0001 C CNN "MFG_PN"
+F 4 "www.yageo.com" V 4550 2750 50  0001 C CNN "MFG_URL"
+F 5 "RC0603FR-07470RL" V 4550 2750 50  0001 C CNN "MFG_PN"
 	1    4550 2750
 	1    0    0    -1
@@
 F 2 "Capacitor_SMD:C_0805_2012Metric" H 3688 2950 50  0001 C CNN
 F 3 "" H 3650 3100 50  0000 C CNN
-F 4 "CC0805ZKY5V5BB226" H 3650 3100 50  0001 C CNN "MFG_PN"
+F 4 "www.yageo.com" H 3650 3100 50  0001 C CNN "MFG_URL"
+F 5 "CC0805ZKY5V5BB226" H 3650 3100 50  0001 C CNN "MFG_PN"
 	1    3650 3100
 	1    0    0    -1

Commit message: schematics: changing all resistor footprints to normal 0603 (not handsoldering)
Parts:
- R34: footprint Resistor_SMD:R_0603_1608Metric_Pad0.84x1.00mm_HandSolder -> Resistor_SMD:R_0603_1608Metric
Changed lines of the file:
@@
 F 0 "R34" V 4630 2350 50  0000 C CNN
 F 1 "15k" V 4550 2350 50  0000 C CNN
-F 2 "Resistor_SMD:R_0603_1608Metric_Pad0.84x1.00mm_HandSolder" V 4480 2350 50  0001 C CNN
+F 2 "Resistor_SMD:R_0603_1608Metric" V 4480 2350 50  0001 C CNN
 F 3 "" H 4550 2350 50  0000 C CNN
 F 4 "www.yageo.com" V 4550 2350 50  0001 C CNN "MFG_URL"
