File: wifi.sch (KiCad schematic (older format))
At the start: 5 parts, among them J3 WIFI_OFF, U9 ESP-WROOM-32

Commit message: schematics: PN update: PCA9306D, PCT8523, ESP32, FCI-10118192-0001LF
Parts:
- U9: Distributor1_PN (none) -> 356-ESP-WROOM-32
Changed lines of the file:
@@
 F 5 "ESP-WROOM-32" H 6650 3450 60  0001 C CNN "MFG_PN"
 F 6 "www.mouser.com" H 6650 3450 60  0001 C CNN "Distributor1_URL"
+F 7 "356-ESP-WROOM-32 " H 6650 3450 50  0001 C CNN "Distributor1_PN"
 	1    6650 3450
 	1    0    0    -1

Commit message: schematics: change filed names for parts BOM suitable for 1-click-bom.tsv MFG_PN->MPN, Distributor1_PN->Mouser, Distributor1_URL->Mouser_URL
Parts:
- C21: MFG_PN CC0805ZKY5V5BB226 -> (none); MPN (none) -> CC0805ZKY5V5BB226
- R34: MFG_PN AC0603FR-1015KL -> (none); MPN (none) -> AC0603FR-1015KL
- R35: MFG_PN RC0603FR-07470RL -> (none); MPN (none) -> RC0603FR-07470RL
- U9: Distributor1_PN 356-ESP-WROOM-32 -> (none); Distributor1_URL www.mouser.com -> (none); MFG_PN ESP-WROOM-32 -> (none); MPN (none) -> ESP-WROOM-32; Mouser (none) -> 356-ESP-WROOM-32; Mouser_URL (none) -> www.mouser.com
Changed lines of the file:
@@
 F 3 "http://espressif.com/sites/default/files/documentation/esp32_datasheet_en.pdf" H 6200 3900 60  0001 C CNN
 F 4 "espressif.com" H 6650 3450 60  0001 C CNN "MFG_URL"
-F 5 "ESP-WROOM-32" H 6650 3450 60  0001 C CNN "MFG_PN"
-F 6 "www.mouser.com" H 6650 3450 60  0001 C CNN "Distributor1_URL"
-F 7 "356-ESP-WROOM-32 " H 6650 3450 50  0001 C CNN "Distributor1_PN"
+F 5 "ESP-WROOM-32" H 6650 3450 60  0001 C CNN "MPN"
+F 6 "www.mouser.com" H 6650 3450 60  0001 C CNN "Mouser_URL"
+F 7 "356-ESP-WROOM-32 " H 6650 3450 50  0001 C CNN "Mouser"
 	1    6650 3450
 	1    0    0    -1
@@
 F 3 "" H 4550 2350 50  0000 C CNN
 F 4 "www.yageo.com" V 4550 2350 50  0001 C CNN "MFG_URL"
-F 5 "AC0603FR-1015KL" V 4550 2350 50  0001 C CNN "MFG_PN"
+F 5 "AC0603FR-1015KL" V 4550 2350 50  0001 C CNN "MPN"
 	1    4550 2350
 	1    0    0    -1
@@
 F 3 "" H 4550 2750 50  0000 C CNN
 F 4 "www.yageo.com" V 4550 2750 50  0001 C CNN "MFG_URL"
-F 5 "RC0603FR-07470RL" V 4550 2750 50  0001 C CNN "MFG_PN"
+F 5 "RC0603FR-07470RL" V 4550 2750 50  0001 C CNN "MPN"
 	1    4550 2750
 	1    0    0    -1
@@
 F 3 "" H 3650 3100 50  0000 C CNN
 F 4 "www.yageo.com" H 3650 3100 50  0001 C CNN "MFG_URL"
-F 5 "CC0805ZKY5V5BB226" H 3650 3100 50  0001 C CNN "MFG_PN"
+F 5 "CC0805ZKY5V5BB226" H 3650 3100 50  0001 C CNN "MPN"
 	1    3650 3100
 	1    0    0    -1

Commit message: schematics: Mouser PN for R,C,BTN
Parts:
- R35: Mouser (none) -> 603-RC0603FR-07470RL
Changed lines of the file:
@@
 F 4 "www.yageo.com" V 4550 2750 50  0001 C CNN "MFG_URL"
 F 5 "RC0603FR-07470RL" V 4550 2750 50  0001 C CNN "MPN"
+F 6 "603-RC0603FR-07470RL" V 4550 2750 50  0001 C CNN "Mouser"
 	1    4550 2750
 	1    0    0    -1

Commit message: schematics: rename MFG_URL -> MFG1_URL
Parts:
- C21, R34, R35: MFG1_URL (none) -> www.yageo.com; MFG_URL www.yageo.com -> (none)
- U9: MFG1_URL (none) -> espressif.com; MFG_URL espressif.com -> (none)
Changed lines of the file:
@@
 F 2 "ESP32:ESP32-WROOM" H 7000 4800 60  0001 C CNN
 F 3 "http://espressif.com/sites/default/files/documentation/esp32_datasheet_en.pdf" H 6200 3900 60  0001 C CNN
-F 4 "espressif.com" H 6650 3450 60  0001 C CNN "MFG_URL"
+F 4 "espressif.com" H 6650 3450 60  0001 C CNN "MFG1_URL"
 F 5 "ESP-WROOM-32" H 6650 3450 60  0001 C CNN "MPN"
 F 6 "www.mouser.com" H 6650 3450 60  0001 C CNN "Mouser_URL"
@@
 F 2 "Resistor_SMD:R_0603_1608Metric" V 4480 2350 50  0001 C CNN
 F 3 "" H 4550 2350 50  0000 C CNN
-F 4 "www.yageo.com" V 4550 2350 50  0001 C CNN "MFG_URL"
+F 4 "www.yageo.com" V 4550 2350 50  0001 C CNN "MFG1_URL"
 F 5 "AC0603FR-1015KL" V 4550 2350 50  0001 C CNN "MPN"
 	1    4550 2350
@@
 F 2 "Resistor_SMD:R_0603_1608Metric" V 4480 2750 50  0001 C CNN
 F 3 "" H 4550 2750 50  0000 C CNN
-F 4 "www.yageo.com" V 4550 2750 50  0001 C CNN "MFG_URL"
+F 4 "www.yageo.com" V 4550 2750 50  0001 C CNN "MFG1_URL"
 F 5 "RC0603FR-07470RL" V 4550 2750 50  0001 C CNN "MPN"
 F 6 "603-RC0603FR-07470RL" V 4550 2750 50  0001 C CNN "Mouser"
@@
 F 2 "Capacitor_SMD:C_0805_2012Metric" H 3688 2950 50  0001 C CNN
 F 3 "" H 3650 3100 50  0000 C CNN
-F 4 "www.yageo.com" H 3650 3100 50  0001 C CNN "MFG_URL"
+F 4 "www.yageo.com" H 3650 3100 50  0001 C CNN "MFG1_URL"
 F 5 "CC0805ZKY5V5BB226" H 3650 3100 50  0001 C CNN "MPN"
 	1    3650 3100

Commit message: schematics: rename "Do not install" -> "Leave empty"
Parts:
- J3: Note Do not install -> Leave empty
Changed lines of the file:
@@
 F 2 "Connector_PinHeader_2.54mm:PinHeader_1x02_P2.54mm_Vertical" H 4550 2000 50  0001 C CNN
 F 3 "" H 4550 2000 50  0000 C CNN
-F 4 "Do not install" H 4550 3200 60  0001 C CNN "Note"
+F 4 "Leave empty" H 4550 3200 60  0001 C CNN "Note"
 	1    4550 3200
 	0    1    1    0

Commit message: schematics: Digikey PN for R
Parts:
- R35: Digikey (none) -> 311-470HRCT-ND
Changed lines of the file:
@@
 F 5 "RC0603FR-07470RL" V 4550 2750 50  0001 C CNN "MPN"
 F 6 "603-RC0603FR-07470RL" V 4550 2750 50  0001 C CNN "Mouser"
+F 7 "311-470HRCT-ND" V 4550 2750 50  0001 C CNN "Digikey"
 	1    4550 2750
 	1    0    0    -1

Commit message: schematics: Distributor PN for ESP32 and available SD card slot
Parts:
- U9: Digikey (none) -> 1904-1010-1-ND
Changed lines of the file:
@@
 F 6 "www.mouser.com" H 6650 3450 60  0001 C CNN "Mouser_URL"
 F 7 "356-ESP-WROOM-32 " H 6650 3450 50  0001 C CNN "Mouser"
+F 8 "1904-1010-1-ND" H 6650 3450 50  0001 C CNN "Digikey"
 	1    6650 3450
 	1    0    0    -1

Commit message: schematics: reducing number of different resistors, using 4x 1N4148 instead of 4x BAT54 schottky diodes.
Parts:
- R35: value 470 -> 680; Digikey 311-470HRCT-ND -> (none); MFG1_URL www.yageo.com -> (none); MPN RC0603FR-07470RL -> (none); Mouser 603-RC0603FR-07470RL -> (none)
Changed lines of the file:
@@
 P 4550 2750
 F 0 "R35" V 4630 2750 50  0000 C CNN
-F 1 "470" V 4550 2750 50  0000 C CNN
+F 1 "680" V 4550 2750 50  0000 C CNN
 F 2 "Resistor_SMD:R_0603_1608Metric" V 4480 2750 50  0001 C CNN
 F 3 "" H 4550 2750 50  0000 C CNN
-F 4 "www.yageo.com" V 4550 2750 50  0001 C CNN "MFG1_URL"
-F 5 "RC0603FR-07470RL" V 4550 2750 50  0001 C CNN "MPN"
-F 6 "603-RC0603FR-07470RL" V 4550 2750 50  0001 C CNN "Mouser"
-F 7 "311-470HRCT-ND" V 4550 2750 50  0001 C CNN "Digikey"
 	1    4550 2750
 	1    0    0    -1
