File: usb.sch (KiCad schematic (older format))
At the start: 25 parts, among them J4 CONN_02X03, U1 LFE5U-85F-6BG381C, U6 FT231XS, Y1 FNETHE025

Commit message: schematics: MFG_PN for 1N4148 diodes
Parts:
- R56: MFG_PN (none) -> RC0603JR-070RL
Changed lines of the file:
@@
 F 3 "" H 6450 4250 50  0000 C CNN
 F 4 "Do not install" H 6450 4250 60  0001 C CNN "Note"
+F 5 "RC0603JR-070RL" V 6450 4250 50  0001 C CNN "MFG_PN"
 	1    6450 4250
 	-1   0    0    1

Commit message: schematics: MFG_URL for R,C
Parts:
- R40, R49, R50, R52, R53, R54, R56, R63, R64, R9: MFG_URL (none) -> www.yageo.com
Changed lines of the file:
@@
 F 2 "Resistor_SMD:R_0603_1608Metric_Pad0.84x1.00mm_HandSolder" V 4630 3600 50  0001 C CNN
 F 3 "" H 4700 3600 50  0000 C CNN
-F 4 "AC0603FR-1015KL" V 4700 3600 50  0001 C CNN "MFG_PN"
+F 4 "www.yageo.com" V 4700 3600 50  0001 C CNN "MFG_URL"
+F 5 "AC0603FR-1015KL" V 4700 3600 50  0001 C CNN "MFG_PN"
 	1    4700 3600
 	0    1    1    0
@@
 F 2 "Resistor_SMD:R_0603_1608Metric" V 2180 4850 50  0001 C CNN
 F 3 "" H 2250 4850 50  0000 C CNN
-F 4 "RC0603FR-071K5L" V 2250 4850 50  0001 C CNN "MFG_PN"
+F 4 "www.yageo.com" V 2250 4850 50  0001 C CNN "MFG_URL"
+F 5 "RC0603FR-071K5L" V 2250 4850 50  0001 C CNN "MFG_PN"
 	1    2250 4850
 	0    -1   -1   0
@@
 F 2 "Resistor_SMD:R_0603_1608Metric" V 2230 1800 50  0001 C CNN
 F 3 "" H 2300 1800 50  0000 C CNN
-F 4 "AC0603JR-0727RL" V 2300 1800 50  0001 C CNN "MFG_PN"
+F 4 "www.yageo.com" V 2300 1800 50  0001 C CNN "MFG_URL"
+F 5 "AC0603JR-0727RL" V 2300 1800 50  0001 C CNN "MFG_PN"
 	1    2300 1800
 	0    1    1    0
@@
 F 2 "Resistor_SMD:R_0603_1608Metric" V 2230 1900 50  0001 C CNN
 F 3 "" H 2300 1900 50  0000 C CNN
-F 4 "AC0603JR-0727RL" V 2300 1900 50  0001 C CNN "MFG_PN"
+F 4 "www.yageo.com" V 2300 1900 50  0001 C CNN "MFG_URL"
+F 5 "AC0603JR-0727RL" V 2300 1900 50  0001 C CNN "MFG_PN"
 	1    2300 1900
 	0    1    1    0
@@
 F 2 "Resistor_SMD:R_0603_1608Metric" V 2180 2750 50  0001 C CNN
 F 3 "" H 2250 2750 50  0000 C CNN
-F 4 "AC0603JR-0727RL" V 2250 2750 50  0001 C CNN "MFG_PN"
+F 4 "www.yageo.com" V 2250 2750 50  0001 C CNN "MFG_URL"
+F 5 "AC0603JR-0727RL" V 2250 2750 50  0001 C CNN "MFG_PN"
 	1    2250 2750
 	0    1    1    0
@@
 F 2 "Resistor_SMD:R_0603_1608Metric" V 2180 2850 50  0001 C CNN
 F 3 "" H 2250 2850 50  0000 C CNN
-F 4 "AC0603JR-0727RL" V 2250 2850 50  0001 C CNN "MFG_PN"
+F 4 "www.yageo.com" V 2250 2850 50  0001 C CNN "MFG_URL"
+F 5 "AC0603JR-0727RL" V 2250 2850 50  0001 C CNN "MFG_PN"
 	1    2250 2850
 	0    1    1    0
@@
 F 2 "Resistor_SMD:R_0603_1608Metric" V 2180 5450 50  0001 C CNN
 F 3 "" H 2250 5450 50  0000 C CNN
-F 4 "RC0603FR-071K5L" V 2250 5450 50  0001 C CNN "MFG_PN"
+F 4 "www.yageo.com" V 2250 5450 50  0001 C CNN "MFG_URL"
+F 5 "RC0603FR-071K5L" V 2250 5450 50  0001 C CNN "MFG_PN"
 	1    2250 5450
 	0    1    1    0
@@
 F 3 "" H 6450 4250 50  0000 C CNN
 F 4 "Do not install" H 6450 4250 60  0001 C CNN "Note"
-F 5 "RC0603JR-070RL" V 6450 4250 50  0001 C CNN "MFG_PN"
+F 5 "www.yageo.com" V 6450 4250 50  0001 C CNN "MFG_URL"
+F 6 "RC0603JR-070RL" V 6450 4250 50  0001 C CNN "MFG_PN"
 	1    6450 4250
 	-1   0    0    1
@@
 F 2 "Resistor_SMD:R_0603_1608Metric_Pad0.84x1.00mm_HandSolder" V 2180 4650 50  0001 C CNN
 F 3 "" H 2250 4650 50  0000 C CNN
-F 4 "AC0603FR-1015KL" V 2250 4650 50  0001 C CNN "MFG_PN"
+F 4 "www.yageo.com" V 2250 4650 50  0001 C CNN "MFG_URL"
+F 5 "AC0603FR-1015KL" V 2250 4650 50  0001 C CNN "MFG_PN"
 	1    2250 4650
 	0    -1   -1   0
@@
 F 2 "Resistor_SMD:R_0603_1608Metric_Pad0.84x1.00mm_HandSolder" V 2180 5250 50  0001 C CNN
 F 3 "" H 2250 5250 50  0000 C CNN
-F 4 "AC0603FR-1015KL" V 2250 5250 50  0001 C CNN "MFG_PN"
+F 4 "www.yageo.com" V 2250 5250 50  0001 C CNN "MFG_URL"
+F 5 "AC0603FR-1015KL" V 2250 5250 50  0001 C CNN "MFG_PN"
 	1    2250 5250
 	0    -1   -1   0

Commit message: schematics: cheaper schottky diodes
Parts:
- D23, D24, D25: Distributor1_PN 621-BAT54WSQ-7-F -> 863-NSR0530HT1G; Distributor1_PN2 (none) -> 621-BAT54WSQ-7-F; MFG2_PN (none) -> BAT54WSQ-7-F; MFG2_URL (none) -> www.diodes.com; MFG_PN BAT54WSQ-7-F -> NSR0530HT1G; MFG_URL www.diodes.com -> www.onsemi.com
- D26: Distributor1_PN 621-BAT54WSQ-7-F -> 863-NSR0530HT1G; Distributor1_PN1 (none) -> 621-BAT54WSQ-7-F; MFG1_PN (none) -> BAT54WSQ-7-F; MFG1_URL (none) -> www.diodes.com; MFG_PN BAT54WSQ-7-F -> NSR0530HT1G; MFG_URL www.diodes.com -> www.onsemi.com
Changed lines of the file:
@@
 F 2 "Diode_SMD:D_SOD-323_HandSoldering" V 1950 4650 50  0001 C CNN
 F 3 "https://www.diodes.com/assets/Datasheets/ds30065.pdf" V 1950 4650 50  0001 C CNN
-F 4 "www.diodes.com" H 1950 4650 50  0001 C CNN "MFG_URL"
-F 5 "BAT54WSQ-7-F" H 1950 4650 50  0001 C CNN "MFG_PN"
-F 6 "www.mouser.com" H 1950 4650 50  0001 C CNN "Distributor1_URL"
-F 7 "621-BAT54WSQ-7-F" H 1950 4650 50  0001 C CNN "Distributor1_PN"
+F 4 "www.onsemi.com" H 1950 4650 50  0001 C CNN "MFG_URL"
+F 5 "NSR0530HT1G " H 1950 4650 50  0001 C CNN "MFG_PN"
+F 6 "www.diodes.com" H 1950 4650 50  0001 C CNN "MFG2_URL"
+F 7 "BAT54WSQ-7-F" H 1950 4650 50  0001 C CNN "MFG2_PN"
+F 8 "www.mouser.com" H 1950 4650 50  0001 C CNN "Distributor1_URL"
+F 9 "863-NSR0530HT1G " H 1950 4650 50  0001 C CNN "Distributor1_PN"
+F 10 "621-BAT54WSQ-7-F" H 1950 4650 50  0001 C CNN "Distributor1_PN2"
 	1    1950 4650
 	1    0    0    -1
@@
 F 2 "Diode_SMD:D_SOD-323_HandSoldering" V 1950 5250 50  0001 C CNN
 F 3 "https://www.diodes.com/assets/Datasheets/ds30065.pdf" V 1950 5250 50  0001 C CNN
-F 4 "www.diodes.com" H 1950 5250 50  0001 C CNN "MFG_URL"
-F 5 "BAT54WSQ-7-F" H 1950 5250 50  0001 C CNN "MFG_PN"
-F 6 "www.mouser.com" H 1950 5250 50  0001 C CNN "Distributor1_URL"
-F 7 "621-BAT54WSQ-7-F" H 1950 5250 50  0001 C CNN "Distributor1_PN"
+F 4 "www.onsemi.com" H 1950 5250 50  0001 C CNN "MFG_URL"
+F 5 "NSR0530HT1G " H 1950 5250 50  0001 C CNN "MFG_PN"
+F 6 "www.diodes.com" H 1950 5250 50  0001 C CNN "MFG2_URL"
+F 7 "BAT54WSQ-7-F" H 1950 5250 50  0001 C CNN "MFG2_PN"
+F 8 "www.mouser.com" H 1950 5250 50  0001 C CNN "Distributor1_URL"
+F 9 "863-NSR0530HT1G " H 1950 5250 50  0001 C CNN "Distributor1_PN"
+F 10 "621-BAT54WSQ-7-F" H 1950 5250 50  0001 C CNN "Distributor1_PN2"
 	1    1950 5250
 	1    0    0    -1
@@
 F 2 "Diode_SMD:D_SOD-323_HandSoldering" V 1950 4850 50  0001 C CNN
 F 3 "https://www.diodes.com/assets/Datasheets/ds30065.pdf" V 1950 4850 50  0001 C CNN
-F 4 "www.diodes.com" H 1950 4850 50  0001 C CNN "MFG_URL"
-F 5 "BAT54WSQ-7-F" H 1950 4850 50  0001 C CNN "MFG_PN"
-F 6 "www.mouser.com" H 1950 4850 50  0001 C CNN "Distributor1_URL"
-F 7 "621-BAT54WSQ-7-F" H 1950 4850 50  0001 C CNN "Distributor1_PN"
+F 4 "www.onsemi.com" H 1950 4850 50  0001 C CNN "MFG_URL"
+F 5 "NSR0530HT1G " H 1950 4850 50  0001 C CNN "MFG_PN"
+F 6 "www.diodes.com" H 1950 4850 50  0001 C CNN "MFG2_URL"
+F 7 "BAT54WSQ-7-F" H 1950 4850 50  0001 C CNN "MFG2_PN"
+F 8 "www.mouser.com" H 1950 4850 50  0001 C CNN "Distributor1_URL"
+F 9 "863-NSR0530HT1G " H 1950 4850 50  0001 C CNN "Distributor1_PN"
+F 10 "621-BAT54WSQ-7-F" H 1950 4850 50  0001 C CNN "Distributor1_PN2"
 	1    1950 4850
 	-1   0    0    1
@@
 F 2 "Diode_SMD:D_SOD-323_HandSoldering" V 1950 5450 50  0001 C CNN
 F 3 "https://www.diodes.com/assets/Datasheets/ds30065.pdf" V 1950 5450 50  0001 C CNN
-F 4 "www.diodes.com" H 1950 5450 50  0001 C CNN "MFG_URL"
-F 5 "BAT54WSQ-7-F" H 1950 5450 50  0001 C CNN "MFG_PN"
-F 6 "www.mouser.com" H 1950 5450 50  0001 C CNN "Distributor1_URL"
-F 7 "621-BAT54WSQ-7-F" H 1950 5450 50  0001 C CNN "Distributor1_PN"
+F 4 "www.onsemi.com" H 1950 5450 50  0001 C CNN "MFG_URL"
+F 5 "NSR0530HT1G " H 1950 5450 50  0001 C CNN "MFG_PN"
+F 6 "www.diodes.com" H 1950 5450 50  0001 C CNN "MFG1_URL"
+F 7 "BAT54WSQ-7-F" H 1950 5450 50  0001 C CNN "MFG1_PN"
+F 8 "www.mouser.com" H 1950 5450 50  0001 C CNN "Distributor1_URL"
+F 9 "863-NSR0530HT1G " H 1950 5450 50  0001 C CNN "Distributor1_PN"
+F 10 "621-BAT54WSQ-7-F" H 1950 5450 50  0001 C CNN "Distributor1_PN1"
 	1    1950 5450
 	-1   0    0    1

Commit message: schematics: changing all resistor footprints to normal 0603 (not handsoldering)
Parts:
- R63, R64, R9: footprint Resistor_SMD:R_0603_1608Metric_Pad0.84x1.00mm_HandSolder -> Resistor_SMD:R_0603_1608Metric
Changed lines of the file:
@@
 F 0 "R9" V 4780 3600 50  0000 C CNN
 F 1 "15k" V 4700 3600 50  0000 C CNN
-F 2 "Resistor_SMD:R_0603_1608Metric_Pad0.84x1.00mm_HandSolder" V 4630 3600 50  0001 C CNN
+F 2 "Resistor_SMD:R_0603_1608Metric" V 4630 3600 50  0001 C CNN
 F 3 "" H 4700 3600 50  0000 C CNN
 F 4 "www.yageo.com" V 4700 3600 50  0001 C CNN "MFG_URL"
@@
 F 0 "R63" V 2330 4650 50  0000 C CNN
 F 1 "15k" V 2250 4650 50  0000 C CNN
-F 2 "Resistor_SMD:R_0603_1608Metric_Pad0.84x1.00mm_HandSolder" V 2180 4650 50  0001 C CNN
+F 2 "Resistor_SMD:R_0603_1608Metric" V 2180 4650 50  0001 C CNN
 F 3 "" H 2250 4650 50  0000 C CNN
 F 4 "www.yageo.com" V 2250 4650 50  0001 C CNN "MFG_URL"
@@
 F 0 "R64" V 2330 5250 50  0000 C CNN
 F 1 "15k" V 2250 5250 50  0000 C CNN
-F 2 "Resistor_SMD:R_0603_1608Metric_Pad0.84x1.00mm_HandSolder" V 2180 5250 50  0001 C CNN
+F 2 "Resistor_SMD:R_0603_1608Metric" V 2180 5250 50  0001 C CNN
 F 3 "" H 2250 5250 50  0000 C CNN
 F 4 "www.yageo.com" V 2250 5250 50  0001 C CNN "MFG_URL"

Commit message: schematics: inductor footprint that fits sizes 1008 and 1210 (2520 and 3225 metric)
Connections:
- net labels added: US2VBUS
Changed lines of the file:
@@
 	-1   0    0    1
 $EndComp
+Text Label 1850 2650 0    60   ~ 0
+US2VBUS
 $EndSCHEMATC

Commit message: schematics: PN update: PCA9306D, PCT8523, ESP32, FCI-10118192-0001LF
Parts:
- US1, US2: Distributor1_PN (none) -> 649-10118192-0001LF
Changed lines of the file:
@@
 F 5 "10118192-0001LF" H 1500 1900 60  0001 C CNN "MFG_PN"
 F 6 "www.mouser.com" H 1500 1900 60  0001 C CNN "Distributor1_URL"
+F 7 "649-10118192-0001LF " H 1500 1900 50  0001 C CNN "Distributor1_PN"
 	1    1500 1900
 	0    -1   1    0
@@
 F 5 "10118192-0001LF" H 1500 2850 60  0001 C CNN "MFG_PN"
 F 6 "www.mouser.com" H 1500 2850 60  0001 C CNN "Distributor1_URL"
+F 7 "649-10118192-0001LF " H 1500 2850 50  0001 C CNN "Distributor1_PN"
 	1    1500 2850
 	0    -1   1    0

Commit message: schematics: change filed names for parts BOM suitable for 1-click-bom.tsv MFG_PN->MPN, Distributor1_PN->Mouser, Distributor1_URL->Mouser_URL
Parts:
- D20, D21: Distributor1_PN 821-BZT52C3V6S -> (none); Distributor1_URL www.mouser.com -> (none); MFG_PN BZT52C3V6S -> (none); MPN (none) -> BZT52C3V6S; Mouser (none) -> 821-BZT52C3V6S; Mouser_URL (none) -> www.mouser.com
- D23, D24, D25, D26: Distributor1_PN 863-NSR0530HT1G -> (none); Distributor1_URL www.mouser.com -> (none); MFG_PN NSR0530HT1G -> (none); MPN (none) -> NSR0530HT1G; Mouser (none) -> 863-NSR0530HT1G; Mouser_URL (none) -> www.mouser.com
- D8, D9: Distributor1_PN 511-STPS2L30AF -> (none); Distributor1_URL www.mouser.com -> (none); MFG_PN STPS2L30AF -> (none); MPN (none) -> STPS2L30AF; Mouser (none) -> 511-STPS2L30AF; Mouser_URL (none) -> www.mouser.com
- R40, R54: MFG_PN RC0603FR-071K5L -> (none); MPN (none) -> RC0603FR-071K5L
- R49, R50, R52, R53: MFG_PN AC0603JR-0727RL -> (none); MPN (none) -> AC0603JR-0727RL
- R56: MFG_PN RC0603JR-070RL -> (none); MPN (none) -> RC0603JR-070RL
- R63, R64, R9: MFG_PN AC0603FR-1015KL -> (none); MPN (none) -> AC0603FR-1015KL
- U1: Distributor1_URL www.mouser.com -> (none); MFG_PN LFE5U-85F-6BG381C -> (none); MPN (none) -> LFE5U-85F-6BG381C; Mouser_URL (none) -> www.mouser.com
- U1: Distributor1_PN 842-LFE5U85F6BG381C -> (none); Distributor1_URL www.mouser.com -> (none); MFG_PN LFE5U-85F-6BG381C -> (none); MPN (none) -> LFE5U-85F-6BG381C; Mouser (none) -> 842-LFE5U85F6BG381C; Mouser_URL (none) -> www.mouser.com
- U6: Distributor1_PN 895-FT231XS-R -> (none); Distributor1_URL www.mouser.com -> (none); MFG_PN FT231XS -> (none); MPN (none) -> FT231XS; Mouser (none) -> 895-FT231XS-R; Mouser_URL (none) -> www.mouser.com
- US1, US2: Distributor1_PN 649-10118192-0001LF -> (none); Distributor1_URL www.mouser.com -> (none); MFG_PN 10118192-0001LF -> (none); MPN (none) -> 10118192-0001LF; Mouser (none) -> 649-10118192-0001LF; Mouser_URL (none) -> www.mouser.com
- Y1: Distributor1_PN 729-FNETHE025 -> (none); Distributor1_URL www.mouser.com -> (none); MFG_PN FNETHE025 -> (none); MPN (none) -> FNETHE025; Mouser (none) -> 729-FNETHE025; Mouser_URL (none) -> www.mouser.com

Commit message: schematics: for "Do not install" parts, have MFG_PN so the part number won't appear in 1-click-bom
Parts:
- R56: MFG_PN (none) -> RC0603JR-070RL; MPN RC0603JR-070RL -> (none)
Changed lines of the file:
@@
 F 4 "Do not install" H 6450 4250 60  0001 C CNN "Note"
 F 5 "www.yageo.com" V 6450 4250 50  0001 C CNN "MFG_URL"
-F 6 "RC0603JR-070RL" V 6450 4250 50  0001 C CNN "MPN"
+F 6 "RC0603JR-070RL" V 6450 4250 50  0001 C CNN "MFG_PN"
 	1    6450 4250
 	-1   0    0    1
