File: usb.sch (KiCad schematic (older format))
At the start: 25 parts, among them J4 CONN_02X03, U1 LFE5U-85F-6BG381C, U6 FT231XS, Y1 FNETHE025

Commit message: schematics: USB footprints reduced pad size for improved centering
Parts:
- D9: renamed from RD9; value 0 -> STPS2L30AF
- US1, US2: footprint usb_otg:USB-MICRO-B-FCI-10118192-0001LF -> usb_otg:USB-MICRO-B-FCI-10118192-0001LF-small-pads
Changed lines of the file:
@@
 $EndComp
 $Comp
-L Device:D_Schottky_Small RD9
+L Device:D_Schottky_Small D9
 U 1 1 58D6C83C
 P 2600 2650
-F 0 "RD9" H 2400 2700 50  0000 L CNN
-F 1 "0" H 2650 2700 50  0000 L CNN
+F 0 "D9" H 2400 2700 50  0000 L CNN
+F 1 "STPS2L30AF" H 2650 2700 50  0000 L CNN
 F 2 "Diode_SMD:D_SMA_Handsoldering" V 2600 2650 60  0001 C CNN
 F 3 "" V 2600 2650 60  0000 C CNN
@@
 F 0 "US1" H 1825 1775 50  0000 C CNN
 F 1 "MICRO_USB" H 1500 2100 50  0000 C CNN
-F 2 "usb_otg:USB-MICRO-B-FCI-10118192-0001LF" V 1450 1800 50  0001 C CNN
+F 2 "usb_otg:USB-MICRO-B-FCI-10118192-0001LF-small-pads" V 1450 1800 50  0001 C CNN
 F 3 "portal.fciconnect.com/Comergent/fci/drawing/10118192.pdf" H 1450 1800 50  0001 C CNN
 F 4 "www.fciconnect.com" H 1500 1900 60  0001 C CNN "MNF1_URL"
@@
 F 0 "US2" H 1825 2725 50  0000 C CNN
 F 1 "MICRO_USB" H 1500 3050 50  0000 C CNN
-F 2 "usb_otg:USB-MICRO-B-FCI-10118192-0001LF" V 1450 2750 50  0001 C CNN
+F 2 "usb_otg:USB-MICRO-B-FCI-10118192-0001LF-small-pads" V 1450 2750 50  0001 C CNN
 F 3 "portal.fciconnect.com/Comergent/fci/drawing/10118192.pdf" H 1450 2750 50  0001 C CNN
 F 4 "www.fciconnect.com" H 1500 2850 60  0001 C CNN "MNF1_URL"

Commit message: schematics: 3 power schottky diodes replaced with 0-ohm jumpers
Parts:
- D8: footprint Diode_SMD:D_SMA_Handsoldering -> Diode_SMD:D_SMA
- RD9: renamed from D9; value STPS2L30AF -> 0; footprint Diode_SMD:D_SMA_Handsoldering -> Resistor_SMD:R_0805_2012Metric_Pad1.29x1.40mm_HandSolder; symbol Device:D_Schottky_Small -> Device:Jumper_NC_Small
Other:
- note added: "STPS2L30AF"
Changed lines of the file:
@@
 F 0 "D8" H 2350 1650 50  0000 L CNN
 F 1 "STPS2L30AF" H 1800 1650 50  0000 L CNN
-F 2 "Diode_SMD:D_SMA_Handsoldering" V 2300 1700 60  0001 C CNN
+F 2 "Diode_SMD:D_SMA" V 2300 1700 60  0001 C CNN
 F 3 "" V 2300 1700 60  0000 C CNN
 F 4 "www.st.com" H 2300 1700 50  0001 C CNN "MNF1_URL"
@@
 $EndComp
 $Comp
-L Device:D_Schottky_Small D9
+L Device:Jumper_NC_Small RD9
 U 1 1 58D6C83C
-P 2600 2650
-F 0 "D9" H 2400 2700 50  0000 L CNN
-F 1 "STPS2L30AF" H 2650 2700 50  0000 L CNN
-F 2 "Diode_SMD:D_SMA_Handsoldering" V 2600 2650 60  0001 C CNN
-F 3 "" V 2600 2650 60  0000 C CNN
-F 4 "Yageo" H 2600 2650 50  0001 C CNN "MFG1"
-F 5 "www.yageo.com" H 2600 2650 50  0001 C CNN "MNF1_URL"
-F 6 "RC0805JR-070RL" H 2600 2650 50  0001 C CNN "MPN"
-F 7 "ST" H 2600 2650 50  0001 C CNN "MFG2"
-F 8 "STPS2L30AF" H 2600 2650 60  0001 C CNN "MPN2"
-F 9 "www.mouser.com" H 2600 2650 60  0001 C CNN "Mouser_URL"
-F 10 "603-RC0805JR-070RL" H 2600 2650 50  0001 C CNN "Mouser"
-F 11 "511-STPS2L30AF " H 2600 2650 60  0001 C CNN "Mouser2"
-F 12 "YAG1327CT-ND" H 2600 2650 50  0001 C CNN "Digikey"
-	1    2600 2650
+P 2650 2650
+F 0 "RD9" H 2650 2750 50  0000 C CNN
+F 1 "0" H 2650 2600 50  0000 C CNN
+F 2 "Resistor_SMD:R_0805_2012Metric_Pad1.29x1.40mm_HandSolder" V 2650 2650 60  0001 C CNN
+F 3 "" V 2650 2650 60  0000 C CNN
+F 4 "Yageo" H 2650 2650 50  0001 C CNN "MFG1"
+F 5 "www.yageo.com" H 2650 2650 50  0001 C CNN "MNF1_URL"
+F 6 "RC0805JR-070RL" H 2650 2650 50  0001 C CNN "MPN"
+F 7 "ST" H 2650 2650 50  0001 C CNN "MFG2"
+F 8 "STPS2L30AF" H 2650 2650 60  0001 C CNN "MPN2"
+F 9 "www.mouser.com" H 2650 2650 60  0001 C CNN "Mouser_URL"
+F 10 "603-RC0805JR-070RL" H 2650 2650 50  0001 C CNN "Mouser"
+F 11 "511-STPS2L30AF " H 2650 2650 60  0001 C CNN "Mouser2"
+F 12 "YAG1327CT-ND" H 2650 2650 50  0001 C CNN "Digikey"
+	1    2650 2650
 	1    0    0    -1
 $EndComp
@@
 L power:+5V #PWR0108
 U 1 1 58D6C83D
-P 3200 2650
-F 0 "#PWR0108" H 3200 2500 50  0001 C CNN
-F 1 "+5V" H 3200 2790 50  0000 C CNN
-F 2 "" H 3200 2650 60  0000 C CNN
-F 3 "" H 3200 2650 60  0000 C CNN
-	1    3200 2650
+P 3000 2650
+F 0 "#PWR0108" H 3000 2500 50  0001 C CNN
+F 1 "+5V" H 3000 2790 50  0000 C CNN
+F 2 "" H 3000 2650 60  0000 C CNN
+F 3 "" H 3000 2650 60  0000 C CNN
+	1    3000 2650
 	0    1    1    0
 $EndComp
@@
 	2400 1700 3050 1700
 Wire Wire Line
-	2700 2650 3200 2650
-Wire Wire Line
-	1800 2650 2500 2650
+	2750 2650 3000 2650
+Wire Wire Line
+	1800 2650 2550 2650
 Wire Wire Line
 	1800 2100 1850 2100
@@
 Text Notes 1550 6050 0    60   ~ 0
 Deviation from USB specification in\npulldowns for BOM simplificaton.\nWith series diode, correct value R63 R64 \nshould be 12k but 15k is used.
+Wire Notes Line
+	2550 2400 2650 2400
+Wire Notes Line
+	2650 2450 2650 2350
+Wire Notes Line
+	2700 2450 2650 2400
+Wire Notes Line
+	2650 2400 2700 2350
+Wire Notes Line
+	2700 2350 2700 2450
+Wire Notes Line
+	2700 2400 2800 2400
+Text Notes 2400 2350 0    60   ~ 0
+STPS2L30AF
 $EndSCHEMATC

Commit message: schematics: revert USB default footprint
Parts:
- US1, US2: footprint usb_otg:USB-MICRO-B-FCI-10118192-0001LF-small-pads -> usb_otg:USB-MICRO-B-FCI-10118192-0001LF
Changed lines of the file:
@@
 F 0 "US1" H 1825 1775 50  0000 C CNN
 F 1 "MICRO_USB" H 1500 2100 50  0000 C CNN
-F 2 "usb_otg:USB-MICRO-B-FCI-10118192-0001LF-small-pads" V 1450 1800 50  0001 C CNN
+F 2 "usb_otg:USB-MICRO-B-FCI-10118192-0001LF" V 1450 1800 50  0001 C CNN
 F 3 "portal.fciconnect.com/Comergent/fci/drawing/10118192.pdf" H 1450 1800 50  0001 C CNN
 F 4 "www.fciconnect.com" H 1500 1900 60  0001 C CNN "MNF1_URL"
@@
 F 0 "US2" H 1825 2725 50  0000 C CNN
 F 1 "MICRO_USB" H 1500 3050 50  0000 C CNN
-F 2 "usb_otg:USB-MICRO-B-FCI-10118192-0001LF-small-pads" V 1450 2750 50  0001 C CNN
+F 2 "usb_otg:USB-MICRO-B-FCI-10118192-0001LF" V 1450 2750 50  0001 C CNN
 F 3 "portal.fciconnect.com/Comergent/fci/drawing/10118192.pdf" H 1450 2750 50  0001 C CNN
 F 4 "www.fciconnect.com" H 1500 2850 60  0001 C CNN "MNF1_URL"

Commit message: schematics: alternative PN for USB connectors
Parts:
- US1: Datasheet2 (none) -> https://www.molex.com/pdm_docs/sd/473460001_sd.pdf; Digikey2 (none) -> WM17141CT-ND; MFG1 (none) -> FCI; MFG2 (none) -> Molex; MNF2_URL (none) -> www.molex.com; MPN2 (none) -> 47346-0001; Mouser2 (none) -> 538-47346-0001
- US2: MNF1_URL www.fciconnect.com -> (none); MPN 10118192-0001LF -> (none); Mouser 649-10118192-0001LF -> (none); Mouser_URL www.mouser.com -> (none)
Changed lines of the file:
@@
 F 1 "MICRO_USB" H 1500 2100 50  0000 C CNN
 F 2 "usb_otg:USB-MICRO-B-FCI-10118192-0001LF" V 1450 1800 50  0001 C CNN
-F 3 "portal.fciconnect.com/Comergent/fci/drawing/10118192.pdf" H 1450 1800 50  0001 C CNN
-F 4 "www.fciconnect.com" H 1500 1900 60  0001 C CNN "MNF1_URL"
-F 5 "10118192-0001LF" H 1500 1900 60  0001 C CNN "MPN"
-F 6 "www.mouser.com" H 1500 1900 60  0001 C CNN "Mouser_URL"
-F 7 "649-10118192-0001LF " H 1500 1900 50  0001 C CNN "Mouser"
-F 8 "609-4613-1-ND" H 1500 1900 50  0001 C CNN "Digikey"
+F 3 "http://portal.fciconnect.com/Comergent/fci/drawing/10118192.pdf" H 1450 1800 50  0001 C CNN
+F 4 "FCI" H 1500 1900 50  0001 C CNN "MFG1"
+F 5 "www.fciconnect.com" H 1500 1900 60  0001 C CNN "MNF1_URL"
+F 6 "10118192-0001LF" H 1500 1900 60  0001 C CNN "MPN"
+F 7 "https://www.molex.com/pdm_docs/sd/473460001_sd.pdf" H 1500 1900 50  0001 C CNN "Datasheet2"
+F 8 "Molex" H 1500 1900 50  0001 C CNN "MFG2"
+F 9 "www.molex.com" H 1500 1900 50  0001 C CNN "MNF2_URL"
+F 10 "47346-0001" H 1500 1900 50  0001 C CNN "MPN2"
+F 11 "www.mouser.com" H 1500 1900 60  0001 C CNN "Mouser_URL"
+F 12 "649-10118192-0001LF " H 1500 1900 50  0001 C CNN "Mouser"
+F 13 "538-47346-0001" H 1500 1900 50  0001 C CNN "Mouser2"
+F 14 "609-4613-1-ND" H 1500 1900 50  0001 C CNN "Digikey"
+F 15 "WM17141CT-ND" H 1500 1900 50  0001 C CNN "Digikey2"
 	1    1500 1900
 	0    -1   1    0
@@
 F 2 "usb_otg:USB-MICRO-B-FCI-10118192-0001LF" V 1450 2750 50  0001 C CNN
 F 3 "portal.fciconnect.com/Comergent/fci/drawing/10118192.pdf" H 1450 2750 50  0001 C CNN
-F 4 "www.fciconnect.com" H 1500 2850 60  0001 C CNN "MNF1_URL"
-F 5 "10118192-0001LF" H 1500 2850 60  0001 C CNN "MPN"
-F 6 "www.mouser.com" H 1500 2850 60  0001 C CNN "Mouser_URL"
-F 7 "649-10118192-0001LF " H 1500 2850 50  0001 C CNN "Mouser"
 	1    1500 2850
 	0    -1   1    0

Commit message: schematics: PN for 15k resistors
Parts:
- R9: Digikey (none) -> YAG3569CT-ND; MPN AC0603FR-1015KL -> RC0603FR-1015KL; Mouser (none) -> 603-RC0603FR-1015KL
Changed lines of the file:
@@
 F 3 "" H 4700 3600 50  0000 C CNN
 F 4 "www.yageo.com" V 4700 3600 50  0001 C CNN "MNF1_URL"
-F 5 "AC0603FR-1015KL" V 4700 3600 50  0001 C CNN "MPN"
+F 5 "RC0603FR-1015KL" V 4700 3600 50  0001 C CNN "MPN"
+F 6 "603-RC0603FR-1015KL" V 4700 3600 50  0001 C CNN "Mouser"
+F 7 "YAG3569CT-ND" V 4700 3600 50  0001 C CNN "Digikey"
 	1    4700 3600
 	0    1    1    0

Commit message: schematics: using new footprints
Parts:
- U6: footprint Housings_SSOP:SSOP-20_4.4x6.5mm_Pitch0.65mm -> ft231x:FT231X-SSOP-20_4.4x6.5mm_Pitch0.65mm
Changed lines of the file:
@@
 F 0 "U6" H 5150 4200 50  0000 L CNN
 F 1 "FT231XS" H 6000 4200 50  0000 L CNN
-F 2 "Housings_SSOP:SSOP-20_4.4x6.5mm_Pitch0.65mm" H 5700 3400 50  0001 C CNN
+F 2 "ft231x:FT231X-SSOP-20_4.4x6.5mm_Pitch0.65mm" H 5700 3400 50  0001 C CNN
 F 3 "www.ftdichip.com/Documents/DataSheets/ICs/DS_FT231X.pdf" H 5700 3400 50  0001 C CNN
 F 4 "www.ftdichip.com" H 5700 3400 60  0001 C CNN "MNF1_URL"

Commit message: schematics: PN cleanup
Parts:
- R40: Digikey 311-1.5KLDCT-ND -> (none); MNF1_URL www.yageo.com -> (none); MPN RC0603FR-071K5L -> (none); Mouser 603-RC0603FR-131K5L -> (none)
- R54: MNF1_URL www.yageo.com -> (none); MPN RC0603FR-071K5L -> (none)
Changed lines of the file:
@@
 F 2 "Resistor_SMD:R_0603_1608Metric" V 2180 4850 50  0001 C CNN
 F 3 "" H 2250 4850 50  0000 C CNN
-F 4 "www.yageo.com" V 2250 4850 50  0001 C CNN "MNF1_URL"
-F 5 "RC0603FR-071K5L" V 2250 4850 50  0001 C CNN "MPN"
-F 6 "603-RC0603FR-131K5L" V 2250 4850 50  0001 C CNN "Mouser"
-F 7 "311-1.5KLDCT-ND" V 2250 4850 50  0001 C CNN "Digikey"
 	1    2250 4850
 	0    -1   -1   0
@@
 F 2 "Resistor_SMD:R_0603_1608Metric" V 2180 5450 50  0001 C CNN
 F 3 "" H 2250 5450 50  0000 C CNN
-F 4 "www.yageo.com" V 2250 5450 50  0001 C CNN "MNF1_URL"
-F 5 "RC0603FR-071K5L" V 2250 5450 50  0001 C CNN "MPN"
 	1    2250 5450
 	0    1    1    0

Commit message: schematics: PN cleanup
Parts:
- RD9: Digikey YAG1327CT-ND -> (none); Mouser 603-RC0805JR-070RL -> (none); Mouser2 511-STPS2L30AF -> (none); Mouser_URL www.mouser.com -> (none)
Changed lines of the file:
@@
 F 7 "ST" H 2650 2650 50  0001 C CNN "MFG2"
 F 8 "STPS2L30AF" H 2650 2650 60  0001 C CNN "MPN2"
-F 9 "www.mouser.com" H 2650 2650 60  0001 C CNN "Mouser_URL"
-F 10 "603-RC0805JR-070RL" H 2650 2650 50  0001 C CNN "Mouser"
-F 11 "511-STPS2L30AF " H 2650 2650 60  0001 C CNN "Mouser2"
-F 12 "YAG1327CT-ND" H 2650 2650 50  0001 C CNN "Digikey"
 	1    2650 2650
 	1    0    0    -1
