File: blinkey.sch (KiCad schematic (older format))
At the start: 34 parts, among them SW1 DIPSW

Commit message: schematics: change filed names for parts BOM suitable for 1-click-bom.tsv MFG_PN->MPN, Distributor1_PN->Mouser, Distributor1_URL->Mouser_URL
Parts:
- BTN1, BTN2, BTN3, BTN4, BTN5, BTN6: Distributor1_URL www.mouser.com -> (none); MFG_PN PTS645SL50SMTR92 LFS -> (none); MPN (none) -> PTS645SL50SMTR92 LFS; Mouser_URL (none) -> www.mouser.com
- C46: MFG_PN CC0805MRX5R6BB225 -> (none); MPN (none) -> CC0805MRX5R6BB225
- D0, D19, D4: Distributor1_PN 859-LTST-C170KRKT -> (none); Distributor1_URL www.mouser.com -> (none); MFG_PN LTST-C170KRKT -> (none); MPN (none) -> LTST-C170KRKT; Mouser (none) -> 859-LTST-C170KRKT; Mouser_URL (none) -> www.mouser.com
- D1, D5: Distributor1_PN 859-LTST-C170KFKT -> (none); Distributor1_URL www.mouser.com -> (none); MFG_PN LTST-C170KFKT -> (none); MPN (none) -> LTST-C170KFKT; Mouser (none) -> 859-LTST-C170KFKT; Mouser_URL (none) -> www.mouser.com
- D18, D2, D6: Distributor1_PN 859-LTST-C170KGKT -> (none); Distributor1_URL www.mouser.com -> (none); MFG_PN LTST-C170KGKT -> (none); MPN (none) -> LTST-C170KGKT; Mouser (none) -> 859-LTST-C170KGKT; Mouser_URL (none) -> www.mouser.com
- D22, D3, D7: Distributor1_PN 859-LTST-C170TBKT -> (none); Distributor1_URL www.mouser.com -> (none); MFG_PN LTST-C170TBKT -> (none); MPN (none) -> LTST-C170TBKT; Mouser (none) -> 859-LTST-C170TBKT; Mouser_URL (none) -> www.mouser.com
- OLED1: Distributor1_URL www.mouser.com -> (none); MFG_PN DM-OLEDC095-626 -> (none); MPN (none) -> DM-OLEDC095-626; Mouser_URL (none) -> www.mouser.com
- R36, R37, R41, R42, R43, R44, R45, R46, R47, R48, R62: MFG_PN RC0603FR-071KL -> (none); MPN (none) -> RC0603FR-071KL
- R39, R51, R7: MFG_PN AC0603FR-07150RL -> (none); MPN (none) -> AC0603FR-07150RL
- SW1: Distributor1_PN 774-2194MST -> (none); Distributor1_URL www.mouser.com -> (none); MFG_PN 219-4MST -> (none); MPN (none) -> 219-4MST; Mouser (none) -> 774-2194MST; Mouser_URL (none) -> www.mouser.com

Commit message: schematics: Mouser PN for R,C,BTN
Parts:
- R7: Mouser (none) -> 603-AC0603FR-07150RL
Changed lines of the file:
@@
 F 4 "www.yageo.com" V 1900 2750 50  0001 C CNN "MFG_URL"
 F 5 "AC0603FR-07150RL" V 1900 2750 50  0001 C CNN "MPN"
+F 6 "603-AC0603FR-07150RL" V 1900 2750 50  0001 C CNN "Mouser"
 	1    1900 2750
 	0    -1   -1   0

Commit message: schematics: Digikey PN for most parts except R
Parts:
- D0: Digikey (none) -> 160-1415-1-ND
- D1, D2: Digikey (none) -> 160-1413-1-ND
- D3: Digikey (none) -> 160-1579-1-ND
- SW1: Digikey (none) -> CT2194MST-ND
Changed lines of the file:
@@
 F 6 "www.mouser.com" H 8000 3200 60  0001 C CNN "Mouser_URL"
 F 7 "774-2194MST " H 8000 3200 60  0001 C CNN "Mouser"
+F 8 "CT2194MST-ND" H 8000 3200 50  0001 C CNN "Digikey"
 	1    8000 3200
 	1    0    0    -1
@@
 F 6 "www.mouser.com" H 4550 3150 60  0001 C CNN "Mouser_URL"
 F 7 "859-LTST-C170TBKT" H 4550 3150 60  0001 C CNN "Mouser"
+F 8 "160-1579-1-ND" H 4550 3150 50  0001 C CNN "Digikey"
 	1    4550 3150
 	1    0    0    -1
@@
 F 6 "www.mouser.com" H 4550 2950 60  0001 C CNN "Mouser_URL"
 F 7 "859-LTST-C170KGKT " H 4550 2950 60  0001 C CNN "Mouser"
+F 8 "160-1413-1-ND" H 4550 2950 50  0001 C CNN "Digikey"
 	1    4550 2950
 	1    0    0    -1
@@
 F 6 "www.mouser.com" H 4550 2550 60  0001 C CNN "Mouser_URL"
 F 7 "859-LTST-C170KRKT" H 4550 2550 60  0001 C CNN "Mouser"
+F 8 "160-1415-1-ND" H 4550 2550 50  0001 C CNN "Digikey"
 	1    4550 2550
 	1    0    0    -1
@@
 F 6 "www.mouser.com" H 4550 2750 60  0001 C CNN "Mouser_URL"
 F 7 "859-LTST-C170KFKT" H 4550 2750 60  0001 C CNN "Mouser"
+F 8 "160-1413-1-ND" H 4550 2750 50  0001 C CNN "Digikey"
 	1    4550 2750
 	1    0    0    -1

Commit message: schematics: corrected mistake in PN for green LED and some C
Parts:
- D2: Digikey 160-1413-1-ND -> 160-1414-1-ND
Changed lines of the file:
@@
 F 6 "www.mouser.com" H 4550 2950 60  0001 C CNN "Mouser_URL"
 F 7 "859-LTST-C170KGKT " H 4550 2950 60  0001 C CNN "Mouser"
-F 8 "160-1413-1-ND" H 4550 2950 50  0001 C CNN "Digikey"
+F 8 "160-1414-1-ND" H 4550 2950 50  0001 C CNN "Digikey"
 	1    4550 2950
 	1    0    0    -1

Commit message: schematics: rename MFG_URL -> MFG1_URL
Parts:
- BTN1, BTN2, BTN3, BTN4, BTN5, BTN6: MFG1_URL (none) -> www.ckswitches.com; MFG_URL www.ckswitches.com -> (none)
- C46, R36, R37, R39, R41, R42, R43, R44, R45, R46, R47, R48, R51, R62, R7: MFG1_URL (none) -> www.yageo.com; MFG_URL www.yageo.com -> (none)
- D0, D1, D19, D22, D3, D4, D5, D7: MFG1_URL (none) -> www.liteon.com; MFG_URL www.liteon.com -> (none)
- D18, D2, D6: MFG1_URL (none) -> www.lite-on.com; MFG_URL www.lite-on.com -> (none)
- OLED1: MFG1_URL (none) -> www.displaymodule.com; MFG_URL www.displaymodule.com -> (none)
- SW1: MFG1_URL (none) -> www.jameco.com; MFG_URL www.jameco.com -> (none)

Commit message: schematics: alternate PN for L1,2,3 and U3,4,5 and some diodes
Parts:
- D2: MFG1_URL www.lite-on.com -> www.liteon.com
Changed lines of the file:
@@
 F 2 "LED_SMD:LED_0805_2012Metric" H 4550 2950 50  0001 C CNN
 F 3 "http://optoelectronics.liteon.com/upload/download/DS22-2000-073/LTST-C170KGKT.pdf" H 4550 2950 50  0001 C CNN
-F 4 "www.lite-on.com" H 4550 2950 60  0001 C CNN "MFG1_URL"
+F 4 "www.liteon.com" H 4550 2950 60  0001 C CNN "MFG1_URL"
 F 5 "LTST-C170KGKT" H 4550 2950 60  0001 C CNN "MPN"
 F 6 "www.mouser.com" H 4550 2950 60  0001 C CNN "Mouser_URL"

Commit message: schematics: rename "Do not install" -> "Leave empty"
Parts:
- OLED1: Note Do not install -> Leave empty
Changed lines of the file:
@@
 F 5 "DM-OLEDC095-626" H 4750 1550 60  0001 C CNN "MPN"
 F 6 "www.mouser.com" H 4750 1550 60  0001 C CNN "Mouser_URL"
-F 7 "Do not install" H 4750 1550 60  0001 C CNN "Note"
+F 7 "Leave empty" H 4750 1550 60  0001 C CNN "Note"
 	1    4750 1550
 	0    1    1    0

Commit message: schematics: Digikey PN for R
Parts:
- R7: Digikey (none) -> 311-150HRCT-ND
Changed lines of the file:
@@
 F 5 "AC0603FR-07150RL" V 1900 2750 50  0001 C CNN "MPN"
 F 6 "603-AC0603FR-07150RL" V 1900 2750 50  0001 C CNN "Mouser"
+F 7 "311-150HRCT-ND" V 1900 2750 50  0001 C CNN "Digikey"
 	1    1900 2750
 	0    -1   -1   0
