File: blinkey.sch (KiCad schematic (older format))
At the start: 34 parts, among them SW1 SW_DIP_x04

Commit message: schematics: some PN's for LCSC
Parts:
- SW1: LCSC (none) -> C319050; MNF2_URL (none) -> https://datasheet.lcsc.com/szlcsc/1912111437_XKB-Enterprise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; MPN2 (none) -> DSHP04TS-S
Changed lines of the file:
@@
 F 4 "www.jameco.com" H 8100 3300 50  0001 C CNN "MNF1_URL"
 F 5 "219-4MST" H 8100 3300 50  0001 C CNN "MPN"
-F 6 "774-2194MST" H 8100 3300 50  0001 C CNN "Mouser"
-F 7 "CT2194MST-ND" H 8100 3300 50  0001 C CNN "Digikey"
-F 8 "FSW002" H 8100 3300 50  0001 C CNN "Koncar"
-F 9 "T" H 8100 3300 50  0001 C CNN "Side"
+F 6 "https://datasheet.lcsc.com/szlcsc/1912111437_XKB-Enterprise-DSHP04TS-S_C319050.pdf" H 8100 3300 50  0001 C CNN "MNF2_URL"
+F 7 "DSHP04TS-S" H 8100 3300 50  0001 C CNN "MPN2"
+F 8 "774-2194MST" H 8100 3300 50  0001 C CNN "Mouser"
+F 9 "CT2194MST-ND" H 8100 3300 50  0001 C CNN "Digikey"
+F 10 "C319050" H 8100 3300 50  0001 C CNN "LCSC"
+F 11 "FSW002" H 8100 3300 50  0001 C CNN "Koncar"
+F 12 "T" H 8100 3300 50  0001 C CNN "Side"
 	1    8100 3300
 	1    0    0    -1

Commit message: schematics: blue LED LCSC PN
Parts:
- D18, D2: LCSC (none) -> C364562
- D22: LCSC (none) -> C98222
Changed lines of the file:
@@
 F 6 "859-LTST-C170TGKT" H 4550 2950 50  0001 C CNN "Mouser"
 F 7 "160-1887-1-ND" H 4550 2950 50  0001 C CNN "Digikey"
-F 8 "LTST-C170TGKT" H 4550 2950 50  0001 C CNN "TME"
-F 9 "0.0789$" H 4550 2950 50  0001 C CNN "price300_TME"
-F 10 "LTST-C170KRKT" H 4550 2950 50  0001 C CNN "LowCost"
-F 11 "FV005" H 4550 2950 50  0001 C CNN "Koncar"
-F 12 "T" H 4550 2950 50  0001 C CNN "Side"
+F 8 "C364562" H 4550 2950 50  0001 C CNN "LCSC"
+F 9 "LTST-C170TGKT" H 4550 2950 50  0001 C CNN "TME"
+F 10 "0.0789$" H 4550 2950 50  0001 C CNN "price300_TME"
+F 11 "LTST-C170KRKT" H 4550 2950 50  0001 C CNN "LowCost"
+F 12 "FV005" H 4550 2950 50  0001 C CNN "Koncar"
+F 13 "T" H 4550 2950 50  0001 C CNN "Side"
 	1    4550 2950
 	1    0    0    -1
@@
 F 13 "859-LTST-C171TBKT" H 5500 5850 50  0001 C CNN "Mouse_r3"
 F 14 "160-1579-1-ND" H 5500 5850 50  0001 C CNN "Digikey"
-F 15 "FV004" H 5500 5850 50  0001 C CNN "Koncar"
-F 16 "T" H 5500 5850 50  0001 C CNN "Side"
+F 15 "C98222" H 5500 5850 50  0001 C CNN "LCSC"
+F 16 "FV004" H 5500 5850 50  0001 C CNN "Koncar"
+F 17 "T" H 5500 5850 50  0001 C CNN "Side"
 	1    5500 5850
 	1    0    0    -1
@@
 F 6 "859-LTST-C170TGKT" H 5500 4600 50  0001 C CNN "Mouser"
 F 7 "160-1887-1-ND" H 5500 4600 50  0001 C CNN "Digikey"
-F 8 "FV005" H 5500 4600 50  0001 C CNN "Koncar"
-F 9 "T" H 5500 4600 50  0001 C CNN "Side"
+F 8 "C364562" H 5500 4600 50  0001 C CNN "LCSC"
+F 9 "FV005" H 5500 4600 50  0001 C CNN "Koncar"
+F 10 "T" H 5500 4600 50  0001 C CNN "Side"
 	1    5500 4600
 	1    0    0    -1

Commit message: schematics: LCSC PN update
Parts:
- D22, D3: LCSC C98222 -> C375453
Changed lines of the file:
@@
 F 13 "859-LTST-C171TBKT" H 4550 3150 50  0001 C CNN "Mouse_r3"
 F 14 "160-1579-1-ND" H 4550 3150 50  0001 C CNN "Digikey"
-F 15 "C98222" H 4550 3150 50  0001 C CNN "LCSC"
+F 15 "C375453" H 4550 3150 50  0001 C CNN "LCSC"
 F 16 "0.02930$" H 4550 3150 50  0001 C CNN "price300_LCSC"
 F 17 "LTST-C170KRKT" H 4550 3150 50  0001 C CNN "LowCost"
@@
 F 13 "859-LTST-C171TBKT" H 5500 5850 50  0001 C CNN "Mouse_r3"
 F 14 "160-1579-1-ND" H 5500 5850 50  0001 C CNN "Digikey"
-F 15 "C98222" H 5500 5850 50  0001 C CNN "LCSC"
+F 15 "C375453" H 5500 5850 50  0001 C CNN "LCSC"
 F 16 "FV004" H 5500 5850 50  0001 C CNN "Koncar"
 F 17 "T" H 5500 5850 50  0001 C CNN "Side"

Commit message: schematics: mouser blue LED PN back to original
Parts:
- D22, D3: Mouse_r1 859-LTST-C170TBKT -> 593-LSM0805463V; Mouser 593-LSM0805463V -> 859-LTST-C170TBKT
Changed lines of the file:
@@
 F 8 "https://www.rohm.com/datasheet/SML-M13UT" H 4550 3150 50  0001 C CNN "Datasheet3"
 F 9 "SMLMN2BCTT86C" H 4550 3150 50  0001 C CNN "MP_N3"
-F 10 "593-LSM0805463V" H 4550 3150 50  0001 C CNN "Mouser"
-F 11 "859-LTST-C170TBKT" H 4550 3150 60  0001 C CNN "Mouse_r1"
+F 10 "859-LTST-C170TBKT" H 4550 3150 60  0001 C CNN "Mouser"
+F 11 "593-LSM0805463V" H 4550 3150 50  0001 C CNN "Mouse_r1"
 F 12 "755-SMLMN2BCTT86C" H 4550 3150 50  0001 C CNN "Mouse_r2"
 F 13 "859-LTST-C171TBKT" H 4550 3150 50  0001 C CNN "Mouse_r3"
@@
 F 8 "https://www.rohm.com/datasheet/SML-M13UT" H 5500 5850 50  0001 C CNN "Datasheet3"
 F 9 "SMLMN2BCTT86C" H 5500 5850 50  0001 C CNN "MP_N3"
-F 10 "593-LSM0805463V" H 5500 5850 50  0001 C CNN "Mouser"
-F 11 "859-LTST-C170TBKT" H 5500 5850 60  0001 C CNN "Mouse_r1"
+F 10 "859-LTST-C170TBKT" H 5500 5850 60  0001 C CNN "Mouser"
+F 11 "593-LSM0805463V" H 5500 5850 50  0001 C CNN "Mouse_r1"
 F 12 "755-SMLMN2BCTT86C" H 5500 5850 50  0001 C CNN "Mouse_r2"
 F 13 "859-LTST-C171TBKT" H 5500 5850 50  0001 C CNN "Mouse_r3"

Commit message: schematics: red LED PN mouser update
Parts:
- D0: Mouse (none) -> 859-LTST-C170KRKT; Mouse_r1 859-LTST-C170KRKT -> (none); Mouser 743-IN-S85ATR -> (none); Mouser_r2 (none) -> 743-IN-S85ATR
- D19: Mouser 859-LTST-C170KRKT -> (none)
Changed lines of the file:
@@
 F 5 "LTST-C170KRKT" H 4550 5350 60  0001 C CNN "MPN"
 F 6 "www.mouser.com" H 4550 5350 60  0001 C CNN "Mouser_URL"
-F 7 "859-LTST-C170KRKT" H 4550 5350 60  0001 C CNN "Mouser"
 	1    4550 5350
 	-1   0    0    1
@@
 F 4 "www.liteon.com" H 4550 2550 60  0001 C CNN "MNF1_URL"
 F 5 "LTST-C170KRKT" H 4550 2550 60  0001 C CNN "MPN"
-F 6 "743-IN-S85ATR" H 4550 2550 50  0001 C CNN "Mouser"
-F 7 "859-LTST-C170KRKT" H 4550 2550 60  0001 C CNN "Mouse_r1"
+F 6 "859-LTST-C170KRKT" H 4550 2550 60  0001 C CNN "Mouse"
+F 7 "743-IN-S85ATR" H 4550 2550 50  0001 C CNN "Mouser_r2"
 F 8 "160-1415-1-ND" H 4550 2550 50  0001 C CNN "Digikey"
 F 9 "C94868" H 4550 2550 50  0001 C CNN "LCSC"

Commit message: schematics: fix mouser alternate red LED PN
Parts:
- D0: Mouse_r2 (none) -> 743-IN-S85ATR; Mouser_r2 743-IN-S85ATR -> (none)
Changed lines of the file:
@@
 F 5 "LTST-C170KRKT" H 4550 2550 60  0001 C CNN "MPN"
 F 6 "859-LTST-C170KRKT" H 4550 2550 60  0001 C CNN "Mouse"
-F 7 "743-IN-S85ATR" H 4550 2550 50  0001 C CNN "Mouser_r2"
+F 7 "743-IN-S85ATR" H 4550 2550 50  0001 C CNN "Mouse_r2"
 F 8 "160-1415-1-ND" H 4550 2550 50  0001 C CNN "Digikey"
 F 9 "C94868" H 4550 2550 50  0001 C CNN "LCSC"

Commit message: schematics: red LED again PN update
Parts:
- D0: Mouse 859-LTST-C170KRKT -> (none); Mouser (none) -> 859-LTST-C170KRKT
Changed lines of the file:
@@
 F 4 "www.liteon.com" H 4550 2550 60  0001 C CNN "MNF1_URL"
 F 5 "LTST-C170KRKT" H 4550 2550 60  0001 C CNN "MPN"
-F 6 "859-LTST-C170KRKT" H 4550 2550 60  0001 C CNN "Mouse"
+F 6 "859-LTST-C170KRKT" H 4550 2550 60  0001 C CNN "Mouser"
 F 7 "743-IN-S85ATR" H 4550 2550 50  0001 C CNN "Mouse_r2"
 F 8 "160-1415-1-ND" H 4550 2550 50  0001 C CNN "Digikey"

Commit message: schematics: v3.1.1 WiFi/JTAG LED to 3.3V. USB-serial has electrical default pull-up so this LED will be OFF by default. For ESP32 it will have inverted logic, ON when logical 0.
Connections:
- wire segments 68 -> 67
Changed lines of the file:
@@
 Title "ULX3S"
 Date ""
-Rev "1.0.2"
+Rev "1.0.3"
 Comp "EMARD"
 Comment1 "Buttons, LEDs, OLED display"
@@
 Wire Wire Line
 	4400 5850 4250 5850
-Wire Wire Line
-	4250 5850 4250 6200
-$Comp
-L power:GND #PWR085
-U 1 1 5A07AFE2
-P 4250 6200
-F 0 "#PWR085" H 4250 5950 50  0001 C CNN
-F 1 "GND" H 4250 6050 50  0000 C CNN
-F 2 "" H 4250 6200 50  0000 C CNN
-F 3 "" H 4250 6200 50  0000 C CNN
-	1    4250 6200
-	1    0    0    -1
-$EndComp
 Text Label 7450 3400 0    60   ~ 0
 SWPU
@@
 F 17 "T" H 5500 5850 50  0001 C CNN "Side"
 	1    5500 5850
-	1    0    0    -1
+	-1   0    0    1
 $EndComp
 $Comp
@@
 Wire Wire Line
 	4750 1950 4850 1950
+$Comp
+L power:+3V3 #PWR?
+U 1 1 5F0C55F7
+P 4250 5850
+F 0 "#PWR?" H 4250 5700 50  0001 C CNN
+F 1 "+3V3" H 4250 5990 50  0000 C CNN
+F 2 "" H 4250 5850 50  0000 C CNN
+F 3 "" H 4250 5850 50  0000 C CNN
+	1    4250 5850
+	0    -1   -1   0
+$EndComp
 $EndSCHEMATC
