File: blinkey.sch (KiCad schematic (older format))
At the start: 34 parts, among them SW1 SW_DIP_x04

Commit message: schematics: newark PNs for some semiconductors and connectors (not all)
Parts:
- D0: Newark (none) -> 61AC0090
- D1: Newark (none) -> 61AC0088
- D2: MPN LTST-C170TGKT -> LTST-C170TGKT; Newark (none) -> 75R0588
- D3: Newar_k2 (none) -> 19J8850; Newark (none) -> 94T2911
Changed lines of the file:
@@
 F 13 "859-LTST-C171TBKT" H 4550 3150 50  0001 C CNN "Mouse_r3"
 F 14 "160-1579-1-ND" H 4550 3150 50  0001 C CNN "Digikey"
-F 15 "C375453" H 4550 3150 50  0001 C CNN "LCSC"
-F 16 "0.02930$" H 4550 3150 50  0001 C CNN "price300_LCSC"
-F 17 "LTST-C170KRKT" H 4550 3150 50  0001 C CNN "LowCost"
-F 18 "FV004" H 4550 3150 50  0001 C CNN "Koncar"
-F 19 "T" H 4550 3150 50  0001 C CNN "Side"
+F 15 "94T2911" H 4550 3150 50  0001 C CNN "Newark"
+F 16 "19J8850" H 4550 3150 50  0001 C CNN "Newar_k2"
+F 17 "C375453" H 4550 3150 50  0001 C CNN "LCSC"
+F 18 "0.02930$" H 4550 3150 50  0001 C CNN "price300_LCSC"
+F 19 "LTST-C170KRKT" H 4550 3150 50  0001 C CNN "LowCost"
+F 20 "FV004" H 4550 3150 50  0001 C CNN "Koncar"
+F 21 "T" H 4550 3150 50  0001 C CNN "Side"
 	1    4550 3150
 	1    0    0    -1
@@
 F 3 "http://optoelectronics.liteon.com/upload/download/DS22-2000-073/LTST-C170KGKT.pdf" H 4550 2950 50  0001 C CNN
 F 4 "www.liteon.com" H 4550 2950 60  0001 C CNN "MNF1_URL"
-F 5 "LTST-C170TGKT " H 4550 2950 50  0001 C CNN "MPN"
+F 5 "LTST-C170TGKT" H 4550 2950 50  0001 C CNN "MPN"
 F 6 "859-LTST-C170TGKT" H 4550 2950 50  0001 C CNN "Mouser"
 F 7 "160-1887-1-ND" H 4550 2950 50  0001 C CNN "Digikey"
-F 8 "C364562" H 4550 2950 50  0001 C CNN "LCSC"
-F 9 "LTST-C170TGKT" H 4550 2950 50  0001 C CNN "TME"
-F 10 "0.0789$" H 4550 2950 50  0001 C CNN "price300_TME"
-F 11 "LTST-C170KRKT" H 4550 2950 50  0001 C CNN "LowCost"
-F 12 "FV005" H 4550 2950 50  0001 C CNN "Koncar"
-F 13 "T" H 4550 2950 50  0001 C CNN "Side"
+F 8 "75R0588" H 4550 2950 50  0001 C CNN "Newark"
+F 9 "C364562" H 4550 2950 50  0001 C CNN "LCSC"
+F 10 "LTST-C170TGKT" H 4550 2950 50  0001 C CNN "TME"
+F 11 "0.0789$" H 4550 2950 50  0001 C CNN "price300_TME"
+F 12 "LTST-C170KRKT" H 4550 2950 50  0001 C CNN "LowCost"
+F 13 "FV005" H 4550 2950 50  0001 C CNN "Koncar"
+F 14 "T" H 4550 2950 50  0001 C CNN "Side"
 	1    4550 2950
 	1    0    0    -1
@@
 F 7 "743-IN-S85ATR" H 4550 2550 50  0001 C CNN "Mouse_r2"
 F 8 "160-1415-1-ND" H 4550 2550 50  0001 C CNN "Digikey"
-F 9 "C94868" H 4550 2550 50  0001 C CNN "LCSC"
-F 10 "0.0195$" H 4550 2550 50  0001 C CNN "price400_LCSC"
-F 11 "FV007" H 4550 2550 50  0001 C CNN "Koncar"
-F 12 "TB" H 4550 2550 50  0001 C CNN "Side"
+F 9 "61AC0090" H 4550 2550 50  0001 C CNN "Newark"
+F 10 "C94868" H 4550 2550 50  0001 C CNN "LCSC"
+F 11 "0.0195$" H 4550 2550 50  0001 C CNN "price400_LCSC"
+F 12 "FV007" H 4550 2550 50  0001 C CNN "Koncar"
+F 13 "TB" H 4550 2550 50  0001 C CNN "Side"
 	1    4550 2550
 	1    0    0    -1
@@
 F 6 "859-LTST-C170KFKT" H 4550 2750 60  0001 C CNN "Mouser"
 F 7 "160-1413-1-ND" H 4550 2750 50  0001 C CNN "Digikey"
-F 8 "C284931" H 4550 2750 50  0001 C CNN "LCSC"
-F 9 "0.02075$" H 4550 2750 50  0001 C CNN "price200_LCSC"
-F 10 "LTST-C170KRKT" H 4550 2750 50  0001 C CNN "LowCost"
-F 11 "FV006" H 4550 2750 50  0001 C CNN "Koncar"
-F 12 "T" H 4550 2750 50  0001 C CNN "Side"
+F 8 "61AC0088" H 4550 2750 50  0001 C CNN "Newark"
+F 9 "C284931" H 4550 2750 50  0001 C CNN "LCSC"
+F 10 "0.02075$" H 4550 2750 50  0001 C CNN "price200_LCSC"
+F 11 "LTST-C170KRKT" H 4550 2750 50  0001 C CNN "LowCost"
+F 12 "FV006" H 4550 2750 50  0001 C CNN "Koncar"
+F 13 "T" H 4550 2750 50  0001 C CNN "Side"
 	1    4550 2750
 	1    0    0    -1

Commit message: schematics: Newark PN switches
Parts:
- SW1: Newark (none) -> 29P1768
Changed lines of the file:
@@
 F 8 "774-2194MST" H 8100 3300 50  0001 C CNN "Mouser"
 F 9 "CT2194MST-ND" H 8100 3300 50  0001 C CNN "Digikey"
-F 10 "C319050" H 8100 3300 50  0001 C CNN "LCSC"
-F 11 "FSW002" H 8100 3300 50  0001 C CNN "Koncar"
-F 12 "T" H 8100 3300 50  0001 C CNN "Side"
+F 10 "29P1768" H 8100 3300 50  0001 C CNN "Newark"
+F 11 "C319050" H 8100 3300 50  0001 C CNN "LCSC"
+F 12 "FSW002" H 8100 3300 50  0001 C CNN "Koncar"
+F 13 "T" H 8100 3300 50  0001 C CNN "Side"
 	1    8100 3300
 	1    0    0    -1

Commit message: schematics: LEDs PN Newark update
Parts:
- D0: Newar_k2 (none) -> 61AC0090; Newark 61AC0090 -> 75R0581
- D1: Newar_k2 (none) -> 61AC0088; Newark 61AC0088 -> 75R0583
Changed lines of the file:
@@
 F 7 "743-IN-S85ATR" H 4550 2550 50  0001 C CNN "Mouse_r2"
 F 8 "160-1415-1-ND" H 4550 2550 50  0001 C CNN "Digikey"
-F 9 "61AC0090" H 4550 2550 50  0001 C CNN "Newark"
-F 10 "C94868" H 4550 2550 50  0001 C CNN "LCSC"
-F 11 "0.0195$" H 4550 2550 50  0001 C CNN "price400_LCSC"
-F 12 "FV007" H 4550 2550 50  0001 C CNN "Koncar"
-F 13 "TB" H 4550 2550 50  0001 C CNN "Side"
+F 9 "75R0581" H 4550 2550 50  0001 C CNN "Newark"
+F 10 "61AC0090" H 4550 2550 50  0001 C CNN "Newar_k2"
+F 11 "C94868" H 4550 2550 50  0001 C CNN "LCSC"
+F 12 "0.0195$" H 4550 2550 50  0001 C CNN "price400_LCSC"
+F 13 "FV007" H 4550 2550 50  0001 C CNN "Koncar"
+F 14 "TB" H 4550 2550 50  0001 C CNN "Side"
 	1    4550 2550
 	1    0    0    -1
@@
 F 6 "859-LTST-C170KFKT" H 4550 2750 60  0001 C CNN "Mouser"
 F 7 "160-1413-1-ND" H 4550 2750 50  0001 C CNN "Digikey"
-F 8 "61AC0088" H 4550 2750 50  0001 C CNN "Newark"
-F 9 "C284931" H 4550 2750 50  0001 C CNN "LCSC"
-F 10 "0.02075$" H 4550 2750 50  0001 C CNN "price200_LCSC"
-F 11 "LTST-C170KRKT" H 4550 2750 50  0001 C CNN "LowCost"
-F 12 "FV006" H 4550 2750 50  0001 C CNN "Koncar"
-F 13 "T" H 4550 2750 50  0001 C CNN "Side"
+F 8 "75R0583" H 4550 2750 50  0001 C CNN "Newark"
+F 9 "61AC0088" H 4550 2750 50  0001 C CNN "Newar_k2"
+F 10 "C284931" H 4550 2750 50  0001 C CNN "LCSC"
+F 11 "0.02075$" H 4550 2750 50  0001 C CNN "price200_LCSC"
+F 12 "LTST-C170KRKT" H 4550 2750 50  0001 C CNN "LowCost"
+F 13 "FV006" H 4550 2750 50  0001 C CNN "Koncar"
+F 14 "T" H 4550 2750 50  0001 C CNN "Side"
 	1    4550 2750
 	1    0    0    -1

Commit message: schematics: PN newark, lcsc R
Parts:
- D18: Newark (none) -> 75R0588
- D22: Newark (none) -> 94T2911
Changed lines of the file:
@@
 F 13 "859-LTST-C171TBKT" H 5500 5850 50  0001 C CNN "Mouse_r3"
 F 14 "160-1579-1-ND" H 5500 5850 50  0001 C CNN "Digikey"
-F 15 "C375453" H 5500 5850 50  0001 C CNN "LCSC"
-F 16 "FV004" H 5500 5850 50  0001 C CNN "Koncar"
-F 17 "T" H 5500 5850 50  0001 C CNN "Side"
+F 15 "94T2911" H 5500 5850 50  0001 C CNN "Newark"
+F 16 "C375453" H 5500 5850 50  0001 C CNN "LCSC"
+F 17 "FV004" H 5500 5850 50  0001 C CNN "Koncar"
+F 18 "T" H 5500 5850 50  0001 C CNN "Side"
 	1    5500 5850
 	-1   0    0    1
@@
 F 6 "859-LTST-C170TGKT" H 5500 4600 50  0001 C CNN "Mouser"
 F 7 "160-1887-1-ND" H 5500 4600 50  0001 C CNN "Digikey"
-F 8 "C364562" H 5500 4600 50  0001 C CNN "LCSC"
-F 9 "FV005" H 5500 4600 50  0001 C CNN "Koncar"
-F 10 "T" H 5500 4600 50  0001 C CNN "Side"
+F 8 "75R0588" H 5500 4600 50  0001 C CNN "Newark"
+F 9 "C364562" H 5500 4600 50  0001 C CNN "LCSC"
+F 10 "FV005" H 5500 4600 50  0001 C CNN "Koncar"
+F 11 "T" H 5500 4600 50  0001 C CNN "Side"
 	1    5500 4600
 	1    0    0    -1

Commit message: schematics: BOM update with currently available mouser PN's
Parts:
- D0: Mouse_r1 (none) -> 859-LTST-C170KRKT; Mouser 859-LTST-C170KRKT -> 859-LTST-C171KRKT
- D1: Mouse_r1 (none) -> 859-LTST-C170KFKT; Mouser 859-LTST-C170KFKT -> 859-LTST-C171KFKT
Changed lines of the file:
@@
 F 4 "www.liteon.com" H 4550 2550 60  0001 C CNN "MNF1_URL"
 F 5 "LTST-C170KRKT" H 4550 2550 60  0001 C CNN "MPN"
-F 6 "859-LTST-C170KRKT" H 4550 2550 60  0001 C CNN "Mouser"
-F 7 "743-IN-S85ATR" H 4550 2550 50  0001 C CNN "Mouse_r2"
-F 8 "160-1415-1-ND" H 4550 2550 50  0001 C CNN "Digikey"
-F 9 "75R0581" H 4550 2550 50  0001 C CNN "Newark"
-F 10 "61AC0090" H 4550 2550 50  0001 C CNN "Newar_k2"
-F 11 "C94868" H 4550 2550 50  0001 C CNN "LCSC"
-F 12 "0.0195$" H 4550 2550 50  0001 C CNN "price400_LCSC"
-F 13 "FV007" H 4550 2550 50  0001 C CNN "Koncar"
-F 14 "TB" H 4550 2550 50  0001 C CNN "Side"
+F 6 "859-LTST-C171KRKT" H 4550 2550 50  0001 C CNN "Mouser"
+F 7 "859-LTST-C170KRKT" H 4550 2550 60  0001 C CNN "Mouse_r1"
+F 8 "743-IN-S85ATR" H 4550 2550 50  0001 C CNN "Mouse_r2"
+F 9 "160-1415-1-ND" H 4550 2550 50  0001 C CNN "Digikey"
+F 10 "75R0581" H 4550 2550 50  0001 C CNN "Newark"
+F 11 "61AC0090" H 4550 2550 50  0001 C CNN "Newar_k2"
+F 12 "C94868" H 4550 2550 50  0001 C CNN "LCSC"
+F 13 "0.0195$" H 4550 2550 50  0001 C CNN "price400_LCSC"
+F 14 "FV007" H 4550 2550 50  0001 C CNN "Koncar"
+F 15 "TB" H 4550 2550 50  0001 C CNN "Side"
 	1    4550 2550
 	1    0    0    -1
@@
 F 4 "www.liteon.com" H 4550 2750 60  0001 C CNN "MNF1_URL"
 F 5 "LTST-C170KFKT" H 4550 2750 60  0001 C CNN "MPN"
-F 6 "859-LTST-C170KFKT" H 4550 2750 60  0001 C CNN "Mouser"
-F 7 "160-1413-1-ND" H 4550 2750 50  0001 C CNN "Digikey"
-F 8 "75R0583" H 4550 2750 50  0001 C CNN "Newark"
-F 9 "61AC0088" H 4550 2750 50  0001 C CNN "Newar_k2"
-F 10 "C284931" H 4550 2750 50  0001 C CNN "LCSC"
-F 11 "0.02075$" H 4550 2750 50  0001 C CNN "price200_LCSC"
-F 12 "LTST-C170KRKT" H 4550 2750 50  0001 C CNN "LowCost"
-F 13 "FV006" H 4550 2750 50  0001 C CNN "Koncar"
-F 14 "T" H 4550 2750 50  0001 C CNN "Side"
+F 6 "859-LTST-C171KFKT" H 4550 2750 50  0001 C CNN "Mouser"
+F 7 "859-LTST-C170KFKT" H 4550 2750 60  0001 C CNN "Mouse_r1"
+F 8 "160-1413-1-ND" H 4550 2750 50  0001 C CNN "Digikey"
+F 9 "75R0583" H 4550 2750 50  0001 C CNN "Newark"
+F 10 "61AC0088" H 4550 2750 50  0001 C CNN "Newar_k2"
+F 11 "C284931" H 4550 2750 50  0001 C CNN "LCSC"
+F 12 "0.02075$" H 4550 2750 50  0001 C CNN "price200_LCSC"
+F 13 "LTST-C170KRKT" H 4550 2750 50  0001 C CNN "LowCost"
+F 14 "FV006" H 4550 2750 50  0001 C CNN "Koncar"
+F 15 "T" H 4550 2750 50  0001 C CNN "Side"
 	1    4550 2750
 	1    0    0    -1

Commit message: schematics: PN alternatives for dialight red and orange LEDs
Parts:
- D0: Mouse_r3 (none) -> 645-598-8110-107F
- D1: Mouse_r3 (none) -> 645-598-8130-107F
Changed lines of the file:
@@
 F 7 "859-LTST-C170KRKT" H 4550 2550 60  0001 C CNN "Mouse_r1"
 F 8 "743-IN-S85ATR" H 4550 2550 50  0001 C CNN "Mouse_r2"
-F 9 "160-1415-1-ND" H 4550 2550 50  0001 C CNN "Digikey"
-F 10 "75R0581" H 4550 2550 50  0001 C CNN "Newark"
-F 11 "61AC0090" H 4550 2550 50  0001 C CNN "Newar_k2"
-F 12 "C94868" H 4550 2550 50  0001 C CNN "LCSC"
-F 13 "0.0195$" H 4550 2550 50  0001 C CNN "price400_LCSC"
-F 14 "FV007" H 4550 2550 50  0001 C CNN "Koncar"
-F 15 "TB" H 4550 2550 50  0001 C CNN "Side"
+F 9 "645-598-8110-107F" H 4550 2550 50  0001 C CNN "Mouse_r3"
+F 10 "160-1415-1-ND" H 4550 2550 50  0001 C CNN "Digikey"
+F 11 "75R0581" H 4550 2550 50  0001 C CNN "Newark"
+F 12 "61AC0090" H 4550 2550 50  0001 C CNN "Newar_k2"
+F 13 "C94868" H 4550 2550 50  0001 C CNN "LCSC"
+F 14 "0.0195$" H 4550 2550 50  0001 C CNN "price400_LCSC"
+F 15 "FV007" H 4550 2550 50  0001 C CNN "Koncar"
+F 16 "TB" H 4550 2550 50  0001 C CNN "Side"
 	1    4550 2550
 	1    0    0    -1
@@
 F 6 "859-LTST-C171KFKT" H 4550 2750 50  0001 C CNN "Mouser"
 F 7 "859-LTST-C170KFKT" H 4550 2750 60  0001 C CNN "Mouse_r1"
-F 8 "160-1413-1-ND" H 4550 2750 50  0001 C CNN "Digikey"
-F 9 "75R0583" H 4550 2750 50  0001 C CNN "Newark"
-F 10 "61AC0088" H 4550 2750 50  0001 C CNN "Newar_k2"
-F 11 "C284931" H 4550 2750 50  0001 C CNN "LCSC"
-F 12 "0.02075$" H 4550 2750 50  0001 C CNN "price200_LCSC"
-F 13 "LTST-C170KRKT" H 4550 2750 50  0001 C CNN "LowCost"
-F 14 "FV006" H 4550 2750 50  0001 C CNN "Koncar"
-F 15 "T" H 4550 2750 50  0001 C CNN "Side"
+F 8 "645-598-8130-107F" H 4550 2750 50  0001 C CNN "Mouse_r3"
+F 9 "160-1413-1-ND" H 4550 2750 50  0001 C CNN "Digikey"
+F 10 "75R0583" H 4550 2750 50  0001 C CNN "Newark"
+F 11 "61AC0088" H 4550 2750 50  0001 C CNN "Newar_k2"
+F 12 "C284931" H 4550 2750 50  0001 C CNN "LCSC"
+F 13 "0.02075$" H 4550 2750 50  0001 C CNN "price200_LCSC"
+F 14 "LTST-C170KRKT" H 4550 2750 50  0001 C CNN "LowCost"
+F 15 "FV006" H 4550 2750 50  0001 C CNN "Koncar"
+F 16 "T" H 4550 2750 50  0001 C CNN "Side"
 	1    4550 2750
 	1    0    0    -1

Commit message: schematics: update mouser PN's
Parts:
- D0: Mouse_r1 859-LTST-C170KRKT -> 859-LTST-C171KRKT; Mouser 859-LTST-C171KRKT -> 859-LTST-C170KRKT
- D1: Mouse_r1 859-LTST-C170KFKT -> 859-LTST-C171KFKT; Mouser 859-LTST-C171KFKT -> 859-LTST-C170KFKT
Changed lines of the file:
@@
 F 4 "www.liteon.com" H 4550 2550 60  0001 C CNN "MNF1_URL"
 F 5 "LTST-C170KRKT" H 4550 2550 60  0001 C CNN "MPN"
-F 6 "859-LTST-C171KRKT" H 4550 2550 50  0001 C CNN "Mouser"
-F 7 "859-LTST-C170KRKT" H 4550 2550 60  0001 C CNN "Mouse_r1"
+F 6 "859-LTST-C170KRKT" H 4550 2550 60  0001 C CNN "Mouser"
+F 7 "859-LTST-C171KRKT" H 4550 2550 50  0001 C CNN "Mouse_r1"
 F 8 "743-IN-S85ATR" H 4550 2550 50  0001 C CNN "Mouse_r2"
 F 9 "645-598-8110-107F" H 4550 2550 50  0001 C CNN "Mouse_r3"
@@
 F 4 "www.liteon.com" H 4550 2750 60  0001 C CNN "MNF1_URL"
 F 5 "LTST-C170KFKT" H 4550 2750 60  0001 C CNN "MPN"
-F 6 "859-LTST-C171KFKT" H 4550 2750 50  0001 C CNN "Mouser"
-F 7 "859-LTST-C170KFKT" H 4550 2750 60  0001 C CNN "Mouse_r1"
+F 6 "859-LTST-C170KFKT" H 4550 2750 60  0001 C CNN "Mouser"
+F 7 "859-LTST-C171KFKT" H 4550 2750 50  0001 C CNN "Mouse_r1"
 F 8 "645-598-8130-107F" H 4550 2750 50  0001 C CNN "Mouse_r3"
 F 9 "160-1413-1-ND" H 4550 2750 50  0001 C CNN "Digikey"

Commit message: schematics: DIP SW Mouser PN
Parts:
- SW1: Mouse_r0 (none) -> 774-2194MST; Mouse_r1 (none) -> 774-219-4LPS; Mouser 774-2194MST -> 774-219-4MSTF
Changed lines of the file:
@@
 F 6 "https://datasheet.lcsc.com/szlcsc/1912111437_XKB-Enterprise-DSHP04TS-S_C319050.pdf" H 8100 3300 50  0001 C CNN "MNF2_URL"
 F 7 "DSHP04TS-S" H 8100 3300 50  0001 C CNN "MPN2"
-F 8 "774-2194MST" H 8100 3300 50  0001 C CNN "Mouser"
-F 9 "CT2194MST-ND" H 8100 3300 50  0001 C CNN "Digikey"
-F 10 "29P1768" H 8100 3300 50  0001 C CNN "Newark"
-F 11 "C319050" H 8100 3300 50  0001 C CNN "LCSC"
-F 12 "FSW002" H 8100 3300 50  0001 C CNN "Koncar"
-F 13 "T" H 8100 3300 50  0001 C CNN "Side"
+F 8 "774-219-4MSTF" H 8100 3300 50  0001 C CNN "Mouser"
+F 9 "774-2194MST" H 8100 3300 50  0001 C CNN "Mouse_r0"
+F 10 "774-219-4LPS" H 8100 3300 50  0001 C CNN "Mouse_r1"
+F 11 "CT2194MST-ND" H 8100 3300 50  0001 C CNN "Digikey"
+F 12 "29P1768" H 8100 3300 50  0001 C CNN "Newark"
+F 13 "C319050" H 8100 3300 50  0001 C CNN "LCSC"
+F 14 "FSW002" H 8100 3300 50  0001 C CNN "Koncar"
+F 15 "T" H 8100 3300 50  0001 C CNN "Side"
 	1    8100 3300
 	1    0    0    -1
