File: flash.sch (KiCad schematic (older format))
At the start: 12 parts, among them U1 LFE5U-85F-6BG381C, U10 IS25LP032D-JNLE-TR

Commit message: schematics: SPI flash chip schematic symbol changed from FRAM to EEPROM It has same pinout but looks better in BOM.
Parts:
- U10: symbol Memory_NVRAM:MB85RS16 -> Memory_EEPROM:25LCxxx
Changed lines of the file:
@@
 $EndDescr
 $Comp
-L Memory_NVRAM:MB85RS16 U10
+L Memory_EEPROM:25LCxxx U10
 U 1 1 58D913F5
 P 3650 4350

Commit message: schematics: changing all resistor footprints to normal 0603 (not handsoldering)
Parts:
- R11, R12, R27, R28, R30, R31, R32, R33, R55: footprint Resistor_SMD:R_0603_1608Metric_Pad0.84x1.00mm_HandSolder -> Resistor_SMD:R_0603_1608Metric
Changed lines of the file:
@@
 F 0 "R27" V 3530 2350 50  0000 C CNN
 F 1 "10k" V 3450 2350 50  0000 C CNN
-F 2 "Resistor_SMD:R_0603_1608Metric_Pad0.84x1.00mm_HandSolder" V 3380 2350 50  0001 C CNN
+F 2 "Resistor_SMD:R_0603_1608Metric" V 3380 2350 50  0001 C CNN
 F 3 "" H 3450 2350 50  0000 C CNN
 F 4 "www.yageo.com" V 3450 2350 50  0001 C CNN "MFG_URL"
@@
 F 0 "R28" V 3730 2350 50  0000 C CNN
 F 1 "10k" V 3650 2350 50  0000 C CNN
-F 2 "Resistor_SMD:R_0603_1608Metric_Pad0.84x1.00mm_HandSolder" V 3580 2350 50  0001 C CNN
+F 2 "Resistor_SMD:R_0603_1608Metric" V 3580 2350 50  0001 C CNN
 F 3 "" H 3650 2350 50  0000 C CNN
 F 4 "www.yageo.com" V 3650 2350 50  0001 C CNN "MFG_URL"
@@
 F 0 "R30" V 4130 2350 50  0000 C CNN
 F 1 "4.7k" V 4050 2350 50  0000 C CNN
-F 2 "Resistor_SMD:R_0603_1608Metric_Pad0.84x1.00mm_HandSolder" V 3980 2350 50  0001 C CNN
+F 2 "Resistor_SMD:R_0603_1608Metric" V 3980 2350 50  0001 C CNN
 F 3 "" H 4050 2350 50  0000 C CNN
 F 4 "www.yageo.com" V 4050 2350 50  0001 C CNN "MFG_URL"
@@
 F 0 "R11" V 3130 2350 50  0000 C CNN
 F 1 "10k" V 3050 2350 50  0000 C CNN
-F 2 "Resistor_SMD:R_0603_1608Metric_Pad0.84x1.00mm_HandSolder" V 2980 2350 50  0001 C CNN
+F 2 "Resistor_SMD:R_0603_1608Metric" V 2980 2350 50  0001 C CNN
 F 3 "" H 3050 2350 50  0000 C CNN
 F 4 "www.yageo.com" V 3050 2350 50  0001 C CNN "MFG_URL"
@@
 F 0 "R12" V 3330 2350 50  0000 C CNN
 F 1 "10k" V 3250 2350 50  0000 C CNN
-F 2 "Resistor_SMD:R_0603_1608Metric_Pad0.84x1.00mm_HandSolder" V 3180 2350 50  0001 C CNN
+F 2 "Resistor_SMD:R_0603_1608Metric" V 3180 2350 50  0001 C CNN
 F 3 "" H 3250 2350 50  0000 C CNN
 F 4 "www.yageo.com" V 3250 2350 50  0001 C CNN "MFG_URL"
@@
 F 0 "R31" V 5280 2350 50  0000 C CNN
 F 1 "10k" V 5200 2350 50  0000 C CNN
-F 2 "Resistor_SMD:R_0603_1608Metric_Pad0.84x1.00mm_HandSolder" V 5130 2350 50  0001 C CNN
+F 2 "Resistor_SMD:R_0603_1608Metric" V 5130 2350 50  0001 C CNN
 F 3 "" H 5200 2350 50  0000 C CNN
 F 4 "www.yageo.com" V 5200 2350 50  0001 C CNN "MFG_URL"
@@
 F 0 "R32" V 5480 2350 50  0000 C CNN
 F 1 "10k" V 5400 2350 50  0000 C CNN
-F 2 "Resistor_SMD:R_0603_1608Metric_Pad0.84x1.00mm_HandSolder" V 5330 2350 50  0001 C CNN
+F 2 "Resistor_SMD:R_0603_1608Metric" V 5330 2350 50  0001 C CNN
 F 3 "" H 5400 2350 50  0000 C CNN
 F 4 "www.yageo.com" V 5400 2350 50  0001 C CNN "MFG_URL"
@@
 F 0 "R33" V 5680 2350 50  0000 C CNN
 F 1 "10k" V 5600 2350 50  0000 C CNN
-F 2 "Resistor_SMD:R_0603_1608Metric_Pad0.84x1.00mm_HandSolder" V 5530 2350 50  0001 C CNN
+F 2 "Resistor_SMD:R_0603_1608Metric" V 5530 2350 50  0001 C CNN
 F 3 "" H 5600 2350 50  0000 C CNN
 F 4 "www.yageo.com" V 5600 2350 50  0001 C CNN "MFG_URL"
@@
 F 0 "R55" V 5430 4800 50  0000 C CNN
 F 1 "15k" V 5350 4800 50  0000 C CNN
-F 2 "Resistor_SMD:R_0603_1608Metric_Pad0.84x1.00mm_HandSolder" V 5280 4800 50  0001 C CNN
+F 2 "Resistor_SMD:R_0603_1608Metric" V 5280 4800 50  0001 C CNN
 F 3 "" H 5350 4800 50  0000 C CNN
 F 4 "AC0603FR-1015KL" V 5350 4800 50  0001 C CNN "MFG_PN"

Commit message: schematics: change filed names for parts BOM suitable for 1-click-bom.tsv MFG_PN->MPN, Distributor1_PN->Mouser, Distributor1_URL->Mouser_URL
Parts:
- R11, R12, R27, R28, R31, R32, R33: MFG_PN AC0603FR-0710KL -> (none); MPN (none) -> AC0603FR-0710KL
- R29: MFG_PN RC0603FR-071KL -> (none); MPN (none) -> RC0603FR-071KL
- R30: MFG_PN AC0603FR-104K7L -> (none); MPN (none) -> AC0603FR-104K7L
- R55: MFG_PN AC0603FR-1015KL -> (none); MPN (none) -> AC0603FR-1015KL
- U1: Distributor1_PN 842-LFE5U85F6BG381C -> (none); Distributor1_URL www.mouser.com -> (none); MFG_PN LFE5U-85F-6BG381C -> (none); MPN (none) -> LFE5U-85F-6BG381C; Mouser (none) -> 842-LFE5U85F6BG381C; Mouser_URL (none) -> www.mouser.com
- U10: Distributor1_PN 870-IS25LP032DJNLETR -> (none); Distributor1_URL www.mouser.com -> (none); MFG_PN IS25LP032D-JNLE-TR -> (none); MPN (none) -> IS25LP032D-JNLE-TR; Mouser (none) -> 870-IS25LP032DJNLETR; Mouser_URL (none) -> www.mouser.com
Changed lines of the file:
@@
 F 3 "http://www.issi.com/WW/pdf/25LP-WP032D.pdf" H 3300 4300 50  0001 C CNN
 F 4 "www.issi.com" H 3650 4350 60  0001 C CNN "MFG_URL"
-F 5 "IS25LP032D-JNLE-TR" H 3650 4350 60  0001 C CNN "MFG_PN"
-F 6 "www.mouser.com" H 3650 4350 60  0001 C CNN "Distributor1_URL"
-F 7 "870-IS25LP032DJNLETR" H 3650 4350 60  0001 C CNN "Distributor1_PN"
+F 5 "IS25LP032D-JNLE-TR" H 3650 4350 60  0001 C CNN "MPN"
+F 6 "www.mouser.com" H 3650 4350 60  0001 C CNN "Mouser_URL"
+F 7 "870-IS25LP032DJNLETR" H 3650 4350 60  0001 C CNN "Mouser"
 	1    3650 4350
 	1    0    0    -1
@@
 F 3 "" H 3450 2350 50  0000 C CNN
 F 4 "www.yageo.com" V 3450 2350 50  0001 C CNN "MFG_URL"
-F 5 "AC0603FR-0710KL" V 3450 2350 50  0001 C CNN "MFG_PN"
+F 5 "AC0603FR-0710KL" V 3450 2350 50  0001 C CNN "MPN"
 	1    3450 2350
 	1    0    0    -1
@@
 F 3 "" H 3650 2350 50  0000 C CNN
 F 4 "www.yageo.com" V 3650 2350 50  0001 C CNN "MFG_URL"
-F 5 "AC0603FR-0710KL" V 3650 2350 50  0001 C CNN "MFG_PN"
+F 5 "AC0603FR-0710KL" V 3650 2350 50  0001 C CNN "MPN"
 	1    3650 2350
 	1    0    0    -1
@@
 F 3 "" H 3850 2350 50  0000 C CNN
 F 4 "www.yageo.com" V 3850 2350 50  0001 C CNN "MFG_URL"
-F 5 "RC0603FR-071KL" V 3850 2350 50  0001 C CNN "MFG_PN"
+F 5 "RC0603FR-071KL" V 3850 2350 50  0001 C CNN "MPN"
 	1    3850 2350
 	1    0    0    -1
@@
 F 3 "" H 4050 2350 50  0000 C CNN
 F 4 "www.yageo.com" V 4050 2350 50  0001 C CNN "MFG_URL"
-F 5 "AC0603FR-104K7L" V 4050 2350 50  0001 C CNN "MFG_PN"
+F 5 "AC0603FR-104K7L" V 4050 2350 50  0001 C CNN "MPN"
 	1    4050 2350
 	1    0    0    -1
@@
 F 3 "" H 3050 2350 50  0000 C CNN
 F 4 "www.yageo.com" V 3050 2350 50  0001 C CNN "MFG_URL"
-F 5 "AC0603FR-0710KL" V 3050 2350 50  0001 C CNN "MFG_PN"
+F 5 "AC0603FR-0710KL" V 3050 2350 50  0001 C CNN "MPN"
 	1    3050 2350
 	1    0    0    -1
@@
 F 3 "" H 3250 2350 50  0000 C CNN
 F 4 "www.yageo.com" V 3250 2350 50  0001 C CNN "MFG_URL"
-F 5 "AC0603FR-0710KL" V 3250 2350 50  0001 C CNN "MFG_PN"
+F 5 "AC0603FR-0710KL" V 3250 2350 50  0001 C CNN "MPN"
 	1    3250 2350
 	1    0    0    -1
@@
 F 3 "" H 5200 2350 50  0000 C CNN
 F 4 "www.yageo.com" V 5200 2350 50  0001 C CNN "MFG_URL"
-F 5 "AC0603FR-0710KL" V 5200 2350 50  0001 C CNN "MFG_PN"
+F 5 "AC0603FR-0710KL" V 5200 2350 50  0001 C CNN "MPN"
 	1    5200 2350
 	1    0    0    -1
@@
 F 3 "" H 5400 2350 50  0000 C CNN
 F 4 "www.yageo.com" V 5400 2350 50  0001 C CNN "MFG_URL"
-F 5 "AC0603FR-0710KL" V 5400 2350 50  0001 C CNN "MFG_PN"
+F 5 "AC0603FR-0710KL" V 5400 2350 50  0001 C CNN "MPN"
 	1    5400 2350
 	1    0    0    -1
@@
 F 3 "" H 5600 2350 50  0000 C CNN
 F 4 "www.yageo.com" V 5600 2350 50  0001 C CNN "MFG_URL"
-F 5 "AC0603FR-0710KL" V 5600 2350 50  0001 C CNN "MFG_PN"
+F 5 "AC0603FR-0710KL" V 5600 2350 50  0001 C CNN "MPN"
 	1    5600 2350
 	1    0    0    -1
@@
 F 2 "Resistor_SMD:R_0603_1608Metric" V 5280 4800 50  0001 C CNN
 F 3 "" H 5350 4800 50  0000 C CNN
-F 4 "AC0603FR-1015KL" V 5350 4800 50  0001 C CNN "MFG_PN"
+F 4 "AC0603FR-1015KL" V 5350 4800 50  0001 C CNN "MPN"
 	1    5350 4800
 	0    1    1    0
@@
 F 2 "lfe5bg381:BGA-381_pitch0.8mm_dia0.4mm" H 6200 5450 60  0001 C CNN
 F 3 "http://www.latticesemi.com/~/media/LatticeSemi/Documents/ApplicationNotes/EH/TN1260.pdf" H 6200 5450 60  0001 C CNN
-F 4 "LFE5U-85F-6BG381C" H 7250 4500 60  0001 C CNN "MFG_PN"
-F 5 "www.mouser.com" H 7250 4500 60  0001 C CNN "Distributor1_URL"
-F 6 "842-LFE5U85F6BG381C" H 7250 4500 60  0001 C CNN "Distributor1_PN"
+F 4 "LFE5U-85F-6BG381C" H 7250 4500 60  0001 C CNN "MPN"
+F 5 "www.mouser.com" H 7250 4500 60  0001 C CNN "Mouser_URL"
+F 6 "842-LFE5U85F6BG381C" H 7250 4500 60  0001 C CNN "Mouser"
 	7    7250 4500
 	1    0    0    -1

Commit message: schematics: Mouser PN for R,C,BTN
Parts:
- R11: Mouser (none) -> 603-AC0603FR-0710KL
Changed lines of the file:
@@
 F 4 "www.yageo.com" V 3050 2350 50  0001 C CNN "MFG_URL"
 F 5 "AC0603FR-0710KL" V 3050 2350 50  0001 C CNN "MPN"
+F 6 "603-AC0603FR-0710KL" V 3050 2350 50  0001 C CNN "Mouser"
 	1    3050 2350
 	1    0    0    -1

Commit message: schematics: Digikey PN for most parts except R
Parts:
- U10: Digikey (none) -> 706-1607-1-ND
Changed lines of the file:
@@
 F 6 "www.mouser.com" H 3650 4350 60  0001 C CNN "Mouser_URL"
 F 7 "870-IS25LP032DJNLETR" H 3650 4350 60  0001 C CNN "Mouser"
+F 8 "706-1607-1-ND" H 3650 4350 50  0001 C CNN "Digikey"
 	1    3650 4350
 	1    0    0    -1

Commit message: schematics: rename MFG_URL -> MFG1_URL
Parts:
- R11, R12, R27, R28, R29, R30, R31, R32, R33: MFG1_URL (none) -> www.yageo.com; MFG_URL www.yageo.com -> (none)
- U10: MFG1_URL (none) -> www.issi.com; MFG_URL www.issi.com -> (none)
Changed lines of the file:
@@
 F 2 "SOA008-150mil:SOA008-150mil" H 3300 4300 50  0001 C CNN
 F 3 "http://www.issi.com/WW/pdf/25LP-WP032D.pdf" H 3300 4300 50  0001 C CNN
-F 4 "www.issi.com" H 3650 4350 60  0001 C CNN "MFG_URL"
+F 4 "www.issi.com" H 3650 4350 60  0001 C CNN "MFG1_URL"
 F 5 "IS25LP032D-JNLE-TR" H 3650 4350 60  0001 C CNN "MPN"
 F 6 "www.mouser.com" H 3650 4350 60  0001 C CNN "Mouser_URL"
@@
 F 2 "Resistor_SMD:R_0603_1608Metric" V 3380 2350 50  0001 C CNN
 F 3 "" H 3450 2350 50  0000 C CNN
-F 4 "www.yageo.com" V 3450 2350 50  0001 C CNN "MFG_URL"
+F 4 "www.yageo.com" V 3450 2350 50  0001 C CNN "MFG1_URL"
 F 5 "AC0603FR-0710KL" V 3450 2350 50  0001 C CNN "MPN"
 	1    3450 2350
@@
 F 2 "Resistor_SMD:R_0603_1608Metric" V 3580 2350 50  0001 C CNN
 F 3 "" H 3650 2350 50  0000 C CNN
-F 4 "www.yageo.com" V 3650 2350 50  0001 C CNN "MFG_URL"
+F 4 "www.yageo.com" V 3650 2350 50  0001 C CNN "MFG1_URL"
 F 5 "AC0603FR-0710KL" V 3650 2350 50  0001 C CNN "MPN"
 	1    3650 2350
@@
 F 2 "Resistor_SMD:R_0603_1608Metric" V 3780 2350 50  0001 C CNN
 F 3 "" H 3850 2350 50  0000 C CNN
-F 4 "www.yageo.com" V 3850 2350 50  0001 C CNN "MFG_URL"
+F 4 "www.yageo.com" V 3850 2350 50  0001 C CNN "MFG1_URL"
 F 5 "RC0603FR-071KL" V 3850 2350 50  0001 C CNN "MPN"
 	1    3850 2350
@@
 F 2 "Resistor_SMD:R_0603_1608Metric" V 3980 2350 50  0001 C CNN
 F 3 "" H 4050 2350 50  0000 C CNN
-F 4 "www.yageo.com" V 4050 2350 50  0001 C CNN "MFG_URL"
+F 4 "www.yageo.com" V 4050 2350 50  0001 C CNN "MFG1_URL"
 F 5 "AC0603FR-104K7L" V 4050 2350 50  0001 C CNN "MPN"
 	1    4050 2350
@@
 F 2 "Resistor_SMD:R_0603_1608Metric" V 2980 2350 50  0001 C CNN
 F 3 "" H 3050 2350 50  0000 C CNN
-F 4 "www.yageo.com" V 3050 2350 50  0001 C CNN "MFG_URL"
+F 4 "www.yageo.com" V 3050 2350 50  0001 C CNN "MFG1_URL"
 F 5 "AC0603FR-0710KL" V 3050 2350 50  0001 C CNN "MPN"
 F 6 "603-AC0603FR-0710KL" V 3050 2350 50  0001 C CNN "Mouser"
@@
 F 2 "Resistor_SMD:R_0603_1608Metric" V 3180 2350 50  0001 C CNN
 F 3 "" H 3250 2350 50  0000 C CNN
-F 4 "www.yageo.com" V 3250 2350 50  0001 C CNN "MFG_URL"
+F 4 "www.yageo.com" V 3250 2350 50  0001 C CNN "MFG1_URL"
 F 5 "AC0603FR-0710KL" V 3250 2350 50  0001 C CNN "MPN"
 	1    3250 2350
@@
 F 2 "Resistor_SMD:R_0603_1608Metric" V 5130 2350 50  0001 C CNN
 F 3 "" H 5200 2350 50  0000 C CNN
-F 4 "www.yageo.com" V 5200 2350 50  0001 C CNN "MFG_URL"
+F 4 "www.yageo.com" V 5200 2350 50  0001 C CNN "MFG1_URL"
 F 5 "AC0603FR-0710KL" V 5200 2350 50  0001 C CNN "MPN"
 	1    5200 2350
@@
 F 2 "Resistor_SMD:R_0603_1608Metric" V 5330 2350 50  0001 C CNN
 F 3 "" H 5400 2350 50  0000 C CNN
-F 4 "www.yageo.com" V 5400 2350 50  0001 C CNN "MFG_URL"
+F 4 "www.yageo.com" V 5400 2350 50  0001 C CNN "MFG1_URL"
 F 5 "AC0603FR-0710KL" V 5400 2350 50  0001 C CNN "MPN"
 	1    5400 2350
@@
 F 2 "Resistor_SMD:R_0603_1608Metric" V 5530 2350 50  0001 C CNN
 F 3 "" H 5600 2350 50  0000 C CNN
-F 4 "www.yageo.com" V 5600 2350 50  0001 C CNN "MFG_URL"
+F 4 "www.yageo.com" V 5600 2350 50  0001 C CNN "MFG1_URL"
 F 5 "AC0603FR-0710KL" V 5600 2350 50  0001 C CNN "MPN"
 	1    5600 2350

Commit message: schematics: add alternate PNs for some parts
Parts:
- U10: MFG2_URL (none) -> www.issi.com; MPN2 (none) -> IS25LP032D-JNLA3; Mouser2 (none) -> 870-IS25LP032DJNLA3T
Changed lines of the file:
@@
 F 2 "SOA008-150mil:SOA008-150mil" H 3300 4300 50  0001 C CNN
 F 3 "http://www.issi.com/WW/pdf/25LP-WP032D.pdf" H 3300 4300 50  0001 C CNN
-F 4 "www.issi.com" H 3650 4350 60  0001 C CNN "MFG1_URL"
+F 4 "www.issi.com" H 3650 4350 50  0001 C CNN "MFG1_URL"
 F 5 "IS25LP032D-JNLE-TR" H 3650 4350 60  0001 C CNN "MPN"
-F 6 "www.mouser.com" H 3650 4350 60  0001 C CNN "Mouser_URL"
-F 7 "870-IS25LP032DJNLETR" H 3650 4350 60  0001 C CNN "Mouser"
-F 8 "706-1607-1-ND" H 3650 4350 50  0001 C CNN "Digikey"
+F 6 "www.issi.com" H 3650 4350 60  0001 C CNN "MFG2_URL"
+F 7 "IS25LP032D-JNLA3" H 3650 4350 50  0001 C CNN "MPN2"
+F 8 "www.mouser.com" H 3650 4350 60  0001 C CNN "Mouser_URL"
+F 9 "870-IS25LP032DJNLETR" H 3650 4350 60  0001 C CNN "Mouser"
+F 10 "870-IS25LP032DJNLA3T" H 3650 4350 50  0001 C CNN "Mouser2"
+F 11 "706-1607-1-ND" H 3650 4350 50  0001 C CNN "Digikey"
 	1    3650 4350
 	1    0    0    -1

Commit message: schematics: Digikey PN for R
Parts:
- R11: Digikey (none) -> 311-10KLMCT-ND
Changed lines of the file:
@@
 F 5 "AC0603FR-0710KL" V 3050 2350 50  0001 C CNN "MPN"
 F 6 "603-AC0603FR-0710KL" V 3050 2350 50  0001 C CNN "Mouser"
+F 7 "311-10KLMCT-ND" V 3050 2350 50  0001 C CNN "Digikey"
 	1    3050 2350
 	1    0    0    -1
