File: flash.sch (KiCad schematic (older format))
At the start: 12 parts, among them U1 LFE5U-85F-6BG381C, U10 IS25LP032D-JNLE-TR

Commit message: schematics: flash chip use combo 150/208 mil footprint
Parts:
- U10: value IS25LP032D-JNLE-TR -> IS25LP128F-JBLE; footprint SOA008-150mil:SOA008-150mil -> SOA008-150mil:SOA008-150-208mil; Datasheet2 (none) -> http://www.issi.com/WW/pdf/25LP-WP032D.pdf; Digikey2 (none) -> IS25LP128F-JBLE-ND; MNF3_URL (none) -> www.issi.com; MPN IS25LP032D-JNLE-TR -> IS25LP128F-JBLE; MPN2 IS25LP032D-JNLA3 -> IS25LP032D-JNLE-TR; MPN3 (none) -> IS25LP032D-JNLA3; Mouser 870-IS25LP032DJNLETR -> 870-IS25LP128F-JBLE; Mouser2 870-IS25LP032DJNLA3T -> 870-IS25LP032DJNLETR; Mouser3 (none) -> 870-IS25LP032DJNLA3T
Changed lines of the file:
@@
 P 3650 4350
 F 0 "U10" H 3350 4600 50  0000 L CNN
-F 1 "IS25LP032D-JNLE-TR" H 3700 4600 50  0000 L CNN
-F 2 "SOA008-150mil:SOA008-150mil" H 3300 4300 50  0001 C CNN
-F 3 "http://www.issi.com/WW/pdf/25LP-WP032D.pdf" H 3300 4300 50  0001 C CNN
+F 1 "IS25LP128F-JBLE" H 3700 4600 50  0000 L CNN
+F 2 "SOA008-150mil:SOA008-150-208mil" H 3300 4300 50  0001 C CNN
+F 3 "http://www.issi.com/WW/pdf/25LP-WP128F.pdf" H 3300 4300 50  0001 C CNN
 F 4 "www.issi.com" H 3650 4350 50  0001 C CNN "MNF1_URL"
-F 5 "IS25LP032D-JNLE-TR" H 3650 4350 60  0001 C CNN "MPN"
-F 6 "www.issi.com" H 3650 4350 60  0001 C CNN "MNF2_URL"
-F 7 "IS25LP032D-JNLA3" H 3650 4350 50  0001 C CNN "MPN2"
-F 8 "www.mouser.com" H 3650 4350 60  0001 C CNN "Mouser_URL"
-F 9 "870-IS25LP032DJNLETR" H 3650 4350 60  0001 C CNN "Mouser"
-F 10 "870-IS25LP032DJNLA3T" H 3650 4350 50  0001 C CNN "Mouser2"
-F 11 "706-1607-1-ND" H 3650 4350 50  0001 C CNN "Digikey"
+F 5 "IS25LP128F-JBLE" H 3650 4350 50  0001 C CNN "MPN"
+F 6 "www.issi.com" H 3650 4350 50  0001 C CNN "MNF2_URL"
+F 7 "http://www.issi.com/WW/pdf/25LP-WP032D.pdf" H 3650 4350 50  0001 C CNN "Datasheet2"
+F 8 "IS25LP032D-JNLE-TR" H 3650 4350 60  0001 C CNN "MPN2"
+F 9 "www.issi.com" H 3650 4350 60  0001 C CNN "MNF3_URL"
+F 10 "IS25LP032D-JNLA3" H 3650 4350 50  0001 C CNN "MPN3"
+F 11 "www.mouser.com" H 3650 4350 60  0001 C CNN "Mouser_URL"
+F 12 "870-IS25LP128F-JBLE" H 3650 4350 50  0001 C CNN "Mouser"
+F 13 "870-IS25LP032DJNLETR" H 3650 4350 60  0001 C CNN "Mouser2"
+F 14 "870-IS25LP032DJNLA3T" H 3650 4350 50  0001 C CNN "Mouser3"
+F 15 "706-1607-1-ND" H 3650 4350 50  0001 C CNN "Digikey"
+F 16 "IS25LP128F-JBLE-ND" H 3650 4350 50  0001 C CNN "Digikey2"
 	1    3650 4350
 	1    0    0    -1

Commit message: schematics: flash digikey PN
Parts:
- U10: Digikey 706-1607-1-ND -> IS25LP128F-JBLE-ND; Digikey2 IS25LP128F-JBLE-ND -> 706-1607-1-ND
Changed lines of the file:
@@
 F 13 "870-IS25LP032DJNLETR" H 3650 4350 60  0001 C CNN "Mouser2"
 F 14 "870-IS25LP032DJNLA3T" H 3650 4350 50  0001 C CNN "Mouser3"
-F 15 "706-1607-1-ND" H 3650 4350 50  0001 C CNN "Digikey"
-F 16 "IS25LP128F-JBLE-ND" H 3650 4350 50  0001 C CNN "Digikey2"
+F 15 "IS25LP128F-JBLE-ND" H 3650 4350 50  0001 C CNN "Digikey"
+F 16 "706-1607-1-ND" H 3650 4350 50  0001 C CNN "Digikey2"
 	1    3650 4350
 	1    0    0    -1

Commit message: schematics: using new footprints
Parts:
- U10: Digikey IS25LP128F-JBLE-ND -> W25Q128JVSIQCT-ND; Digikey2 706-1607-1-ND -> IS25LP128F-JBLE-ND; Digikey3 (none) -> 706-1607-1-ND
Changed lines of the file:
@@
 F 13 "870-IS25LP032DJNLETR" H 3650 4350 60  0001 C CNN "Mouser2"
 F 14 "870-IS25LP032DJNLA3T" H 3650 4350 50  0001 C CNN "Mouser3"
-F 15 "IS25LP128F-JBLE-ND" H 3650 4350 50  0001 C CNN "Digikey"
-F 16 "706-1607-1-ND" H 3650 4350 50  0001 C CNN "Digikey2"
+F 15 "W25Q128JVSIQCT-ND " H 3650 4350 50  0001 C CNN "Digikey"
+F 16 "IS25LP128F-JBLE-ND" H 3650 4350 50  0001 C CNN "Digikey2"
+F 17 "706-1607-1-ND" H 3650 4350 50  0001 C CNN "Digikey3"
 	1    3650 4350
 	1    0    0    -1

Commit message: schematics: PN cleanup
Parts:
- R29: MNF1_URL www.yageo.com -> (none); MPN RC0603FR-071KL -> (none)
- R55: MPN AC0603FR-1015KL -> (none)
Changed lines of the file:
@@
 F 2 "Resistor_SMD:R_0603_1608Metric" V 3780 2350 50  0001 C CNN
 F 3 "" H 3850 2350 50  0000 C CNN
-F 4 "www.yageo.com" V 3850 2350 50  0001 C CNN "MNF1_URL"
-F 5 "RC0603FR-071KL" V 3850 2350 50  0001 C CNN "MPN"
 	1    3850 2350
 	1    0    0    -1
@@
 F 2 "Resistor_SMD:R_0603_1608Metric" V 5280 4800 50  0001 C CNN
 F 3 "" H 5350 4800 50  0000 C CNN
-F 4 "AC0603FR-1015KL" V 5350 4800 50  0001 C CNN "MPN"
 	1    5350 4800
 	0    1    1    0

Commit message: schematics: LowCost field for the parts
Parts:
- U10: LowCost (none) -> 870-IS25LP032DJBLETR
Changed lines of the file:
@@
 F 16 "IS25LP128F-JBLE-ND" H 3650 4350 50  0001 C CNN "Digikey2"
 F 17 "706-1607-1-ND" H 3650 4350 50  0001 C CNN "Digikey3"
+F 18 "870-IS25LP032DJBLETR" H 3650 4350 50  0001 C CNN "LowCost"
 	1    3650 4350
 	1    0    0    -1

Commit message: schematics v2.0.3: Diode D28 for BTN0 to PROGRAMN wiring
Parts:
- added D28: 1N4148, Diode_SMD:D_SOD-323_HandSoldering, symbol Device:D
Connections:
- net labels added: PWRBTn
Changed lines of the file:
@@
 Title "ULX3S"
 Date ""
-Rev "1.0.0"
+Rev "1.0.1"
 Comp "EMARD"
 Comment1 "SPI flash"
@@
 Text Notes 2900 3650 0    60   ~ 0
 Deviation from TN1260 in pullup:\nvalues for BOM simplification.\nCorrect values should be 10k and 1k \nbut 15k and 1.2k are used.
+Text GLabel 5200 4500 0    60   Input ~ 0
+PWRBTn
+$Comp
+L Device:D D28
+U 1 1 5B5DD430
+P 5350 4500
+F 0 "D28" H 5350 4600 50  0000 C CNN
+F 1 "1N4148" H 5350 4400 50  0000 C CNN
+F 2 "Diode_SMD:D_SOD-323_HandSoldering" H 5350 4500 50  0001 C CNN
+F 3 "~" H 5350 4500 50  0001 C CNN
+	1    5350 4500
+	1    0    0    -1
+$EndComp
 $EndSCHEMATC

Commit message: schematics v2.0.4 signal USER_PROGRAMN
Parts:
- added D29: 1N4148, Diode_SMD:D_SOD-323_HandSoldering, symbol Device:D
Connections:
- net labels added: USER_PROGRAMN
- wire segments 25 -> 27
Changed lines of the file:
@@
 Title "ULX3S"
 Date ""
-Rev "1.0.1"
+Rev "1.0.2"
 Comp "EMARD"
 Comment1 "SPI flash"
@@
 Text Notes 9050 4000 0    60   ~ 0
 BTN_R v1.7
-Text Notes 2900 3650 0    60   ~ 0
+Text Notes 1200 2550 0    60   ~ 0
 Deviation from TN1260 in pullup:\nvalues for BOM simplification.\nCorrect values should be 10k and 1k \nbut 15k and 1.2k are used.
 Text GLabel 5200 4500 0    60   Input ~ 0
@@
 	1    0    0    -1
 $EndComp
+Text GLabel 5150 3700 0    60   Input ~ 0
+USER_PROGRAMN
+Wire Wire Line
+	5150 3700 5200 3700
+Wire Wire Line
+	5200 3700 5200 3650
+$Comp
+L Device:D D29
+U 1 1 5B526A74
+P 5200 3500
+F 0 "D29" H 5200 3600 50  0000 C CNN
+F 1 "1N4148" H 5200 3400 50  0000 C CNN
+F 2 "Diode_SMD:D_SOD-323_HandSoldering" H 5200 3500 50  0001 C CNN
+F 3 "~" H 5200 3500 50  0001 C CNN
+	1    5200 3500
+	0    -1   -1   0
+$EndComp
 $EndSCHEMATC

Commit message: schematics update
Connections:
- wire segments 27 -> 28
Other:
- moved on the sheet: D28, D29
Changed lines of the file:
@@
 	1    0    0    -1
 $EndComp
-Wire Wire Line
-	5200 2500 5200 3350
 Text Label 5200 3300 1    60   ~ 0
 FPGA_PROGRAMN
@@
 Text Notes 1200 2550 0    60   ~ 0
 Deviation from TN1260 in pullup:\nvalues for BOM simplification.\nCorrect values should be 10k and 1k \nbut 15k and 1.2k are used.
-Text GLabel 5200 4500 0    60   Input ~ 0
+Text GLabel 4850 3400 0    60   Input ~ 0
 PWRBTn
 $Comp
 L Device:D D28
 U 1 1 5B5DD430
-P 5350 4500
-F 0 "D28" H 5350 4600 50  0000 C CNN
-F 1 "1N4148" H 5350 4400 50  0000 C CNN
-F 2 "Diode_SMD:D_SOD-323_HandSoldering" H 5350 4500 50  0001 C CNN
-F 3 "~" H 5350 4500 50  0001 C CNN
-	1    5350 4500
+P 5000 3400
+F 0 "D28" H 5000 3500 50  0000 C CNN
+F 1 "1N4148" H 5400 3400 50  0000 C CNN
+F 2 "Diode_SMD:D_SOD-323_HandSoldering" H 5000 3400 50  0001 C CNN
+F 3 "~" H 5000 3400 50  0001 C CNN
+	1    5000 3400
 	1    0    0    -1
 $EndComp
-Text GLabel 5150 3700 0    60   Input ~ 0
+Text GLabel 4850 3550 0    60   Input ~ 0
 USER_PROGRAMN
-Wire Wire Line
-	5150 3700 5200 3700
-Wire Wire Line
-	5200 3700 5200 3650
 $Comp
 L Device:D D29
 U 1 1 5B526A74
-P 5200 3500
-F 0 "D29" H 5200 3600 50  0000 C CNN
-F 1 "1N4148" H 5200 3400 50  0000 C CNN
-F 2 "Diode_SMD:D_SOD-323_HandSoldering" H 5200 3500 50  0001 C CNN
-F 3 "~" H 5200 3500 50  0001 C CNN
-	1    5200 3500
-	0    -1   -1   0
+P 5000 3550
+F 0 "D29" H 5000 3450 50  0000 C CNN
+F 1 "1N4148" H 5400 3550 50  0000 C CNN
+F 2 "Diode_SMD:D_SOD-323_HandSoldering" H 5000 3550 50  0001 C CNN
+F 3 "~" H 5000 3550 50  0001 C CNN
+	1    5000 3550
+	1    0    0    -1
 $EndComp
+Wire Wire Line
+	5150 3400 5200 3400
+Wire Wire Line
+	5200 2500 5200 3400
+Wire Wire Line
+	5150 3550 5200 3550
+Wire Wire Line
+	5200 3550 5200 3400
+Connection ~ 5200 3400
 $EndSCHEMATC
