File: flash.sch (KiCad schematic (older format))
At the start: 14 parts, among them U1 LFE5U-85F-6BG381C, U10 IS25LP128F-JBLE

Commit message: schematics v2.0.5: NOP change, comments about PROGRAMN not connected on v1.7
Other:
- note added: "NC v1.7"
Changed lines of the file:
@@
 Title "ULX3S"
 Date ""
-Rev "1.0.2"
+Rev "1.0.3"
 Comp "EMARD"
 Comment1 "SPI flash"
@@
 	5200 3550 5200 3400
 Connection ~ 5200 3400
+Text Notes 4000 3450 0    60   ~ 0
+NC v1.7
+Text Notes 3600 3600 0    60   ~ 0
+NC v1.7
 $EndSCHEMATC

Commit message: schematics v2.0.10: some additional text notes, a NOP change
Other:
- note added: "PWRBTn\non "power" sheet"
- note added: "USER_PROGRAMN\non "usb" sheet"
Changed lines of the file:
@@
 Title "ULX3S"
 Date ""
-Rev "1.0.3"
+Rev "1.0.4"
 Comp "EMARD"
 Comment1 "SPI flash"
@@
 Text Notes 3600 3600 0    60   ~ 0
 NC v1.7
+Text Notes 4000 3800 0    60   ~ 0
+USER_PROGRAMN\non "usb" sheet
+Text Notes 4100 3300 0    60   ~ 0
+PWRBTn\non "power" sheet
 $EndSCHEMATC

Commit message: schematics: Additional field "Koncar" with their specific part number aliases
Parts:
- U10: Koncar (none) -> FU003
Changed lines of the file:
@@
 F 17 "706-1607-1-ND" H 3650 4350 50  0001 C CNN "Digikey3"
 F 18 "870-IS25LP032DJBLETR" H 3650 4350 50  0001 C CNN "LowCost"
+F 19 "FU003" H 3650 4350 50  0001 C CNN "Koncar"
 	1    3650 4350
 	1    0    0    -1

Commit message: schematics: update for D28 to have Note: Leave empty
Parts:
- D28: value 1N4148 -> 1N914; symbol Device:D -> Device:D_ALT; Digikey (none) -> 1N4148WXTPMSCT-ND; EMPTY_MPN (none) -> MMDL914T1G; Koncar (none) -> FV001; Mouser (none) -> 863-MMDL914T1G; Note (none) -> Leave empty
- D29: value 1N4148 -> 1N914
Changed lines of the file:
@@
 PWRBTn
 $Comp
-L Device:D D28
+L Device:D_ALT D28
 U 1 1 5B5DD430
 P 5000 3400
 F 0 "D28" H 5000 3500 50  0000 C CNN
-F 1 "1N4148" H 5400 3400 50  0000 C CNN
+F 1 "1N914" H 5400 3400 50  0000 C CNN
 F 2 "Diode_SMD:D_SOD-323_HandSoldering" H 5000 3400 50  0001 C CNN
 F 3 "~" H 5000 3400 50  0001 C CNN
+F 4 "Leave empty" H 5000 3400 50  0001 C CNN "Note"
+F 5 "MMDL914T1G" H 5000 3400 50  0001 C CNN "EMPTY_MPN"
+F 6 "863-MMDL914T1G" H 5000 3400 50  0001 C CNN "Mouser"
+F 7 "1N4148WXTPMSCT-ND" H 5000 3400 50  0001 C CNN "Digikey"
+F 8 "FV001" H 5000 3400 50  0001 C CNN "Koncar"
 	1    5000 3400
 	1    0    0    -1
@@
 P 5000 3550
 F 0 "D29" H 5000 3450 50  0000 C CNN
-F 1 "1N4148" H 5400 3550 50  0000 C CNN
+F 1 "1N914" H 5400 3550 50  0000 C CNN
 F 2 "Diode_SMD:D_SOD-323_HandSoldering" H 5000 3550 50  0001 C CNN
 F 3 "~" H 5000 3550 50  0001 C CNN

Commit message: schematics 2.1.10: Flash pull up resistors R11 R12 R27 R28 15k -> 10k
Parts:
- R11: value 15k -> 10k; Digikey (none) -> 311-10KLMCT-ND; Koncar (none) -> FR014; MNF1_URL (none) -> www.yageo.com; MPN (none) -> RC0603FR-0710KL; Mouser (none) -> 603-RC0603FR-0710KL
- R12, R27, R28: value 15k -> 10k
Other:
- note added: "Deviation from TN1260 in pullup:\nvalues for BOM simplification.\nCorrect values should be 1k \nbut 1.2k are used."
- note removed: "Deviation from TN1260 in pullup:\nvalues for BOM simplification.\nCorrect values should be 10k and 1k \nbut 15k and 1.2k are used."
Changed lines of the file:
@@
 Title "ULX3S"
 Date ""
-Rev "1.0.4"
+Rev "1.0.5"
 Comp "EMARD"
 Comment1 "SPI flash"
@@
 P 3450 2350
 F 0 "R27" V 3530 2350 50  0000 C CNN
-F 1 "15k" V 3450 2350 50  0000 C CNN
+F 1 "10k" V 3450 2350 50  0000 C CNN
 F 2 "Resistor_SMD:R_0603_1608Metric" V 3380 2350 50  0001 C CNN
 F 3 "" H 3450 2350 50  0000 C CNN
@@
 P 3650 2350
 F 0 "R28" V 3730 2350 50  0000 C CNN
-F 1 "15k" V 3650 2350 50  0000 C CNN
+F 1 "10k" V 3650 2350 50  0000 C CNN
 F 2 "Resistor_SMD:R_0603_1608Metric" V 3580 2350 50  0001 C CNN
 F 3 "" H 3650 2350 50  0000 C CNN
@@
 P 3050 2350
 F 0 "R11" V 3130 2350 50  0000 C CNN
-F 1 "15k" V 3050 2350 50  0000 C CNN
+F 1 "10k" V 3050 2350 50  0000 C CNN
 F 2 "Resistor_SMD:R_0603_1608Metric" V 2980 2350 50  0001 C CNN
 F 3 "" H 3050 2350 50  0000 C CNN
+F 4 "www.yageo.com" V 3050 2350 50  0001 C CNN "MNF1_URL"
+F 5 "RC0603FR-0710KL" V 3050 2350 50  0001 C CNN "MPN"
+F 6 "603-RC0603FR-0710KL" V 3050 2350 50  0001 C CNN "Mouser"
+F 7 "311-10KLMCT-ND" V 3050 2350 50  0001 C CNN "Digikey"
+F 8 "FR014" V 3050 2350 50  0001 C CNN "Koncar"
 	1    3050 2350
 	1    0    0    -1
@@
 P 3250 2350
 F 0 "R12" V 3330 2350 50  0000 C CNN
-F 1 "15k" V 3250 2350 50  0000 C CNN
+F 1 "10k" V 3250 2350 50  0000 C CNN
 F 2 "Resistor_SMD:R_0603_1608Metric" V 3180 2350 50  0001 C CNN
 F 3 "" H 3250 2350 50  0000 C CNN
@@
 BTN_R v1.7
 Text Notes 1200 2550 0    60   ~ 0
-Deviation from TN1260 in pullup:\nvalues for BOM simplification.\nCorrect values should be 10k and 1k \nbut 15k and 1.2k are used.
+Deviation from TN1260 in pullup:\nvalues for BOM simplification.\nCorrect values should be 1k \nbut 1.2k are used.
 Text GLabel 4850 3400 0    60   Input ~ 0
 PWRBTn

Commit message: schematics: updating DAC 550->549 ohm, 1.2k->1.1k
Parts:
- R29: value 1.2k -> 1.1k
Other:
- note added: "Deviation from TN1260 in pullup:\nvalues for BOM simplification.\nCorrect values should be 1k \nbut 1.1k is used."
- note removed: "Deviation from TN1260 in pullup:\nvalues for BOM simplification.\nCorrect values should be 1k \nbut 1.2k are used."
Changed lines of the file:
@@
 P 3850 2350
 F 0 "R29" V 3930 2350 50  0000 C CNN
-F 1 "1.2k" V 3850 2350 50  0000 C CNN
+F 1 "1.1k" V 3850 2350 50  0000 C CNN
 F 2 "Resistor_SMD:R_0603_1608Metric" V 3780 2350 50  0001 C CNN
 F 3 "" H 3850 2350 50  0000 C CNN
@@
 BTN_R v1.7
 Text Notes 1200 2550 0    60   ~ 0
-Deviation from TN1260 in pullup:\nvalues for BOM simplification.\nCorrect values should be 1k \nbut 1.2k are used.
+Deviation from TN1260 in pullup:\nvalues for BOM simplification.\nCorrect values should be 1k \nbut 1.1k is used.
 Text GLabel 4850 3400 0    60   Input ~ 0
 PWRBTn

Commit message: schemtics: mouser PN for 128 Mbit flash chip in tapek&reel package
Parts:
- U10: Mouser 870-IS25LP128F-JBLE -> 870-IS25LP128F-JBLE-TR
Changed lines of the file:
@@
 F 10 "IS25LP032D-JNLA3" H 3650 4350 50  0001 C CNN "MPN3"
 F 11 "www.mouser.com" H 3650 4350 60  0001 C CNN "Mouser_URL"
-F 12 "870-IS25LP128F-JBLE" H 3650 4350 50  0001 C CNN "Mouser"
+F 12 "870-IS25LP128F-JBLE-TR" H 3650 4350 50  0001 C CNN "Mouser"
 F 13 "870-IS25LP032DJNLETR" H 3650 4350 60  0001 C CNN "Mouser2"
 F 14 "870-IS25LP032DJNLA3T" H 3650 4350 50  0001 C CNN "Mouser3"

Commit message: schematics: cheaper manufacturers PNs and some prices
Parts:
- U10: LCSC (none) -> C97521; LCSC_price100 (none) -> 0.7796$
Changed lines of the file:
@@
 F 16 "IS25LP128F-JBLE-ND" H 3650 4350 50  0001 C CNN "Digikey2"
 F 17 "706-1607-1-ND" H 3650 4350 50  0001 C CNN "Digikey3"
-F 18 "870-IS25LP032DJBLETR" H 3650 4350 50  0001 C CNN "LowCost"
-F 19 "FU003" H 3650 4350 50  0001 C CNN "Koncar"
+F 18 "C97521" H 3650 4350 50  0001 C CNN "LCSC"
+F 19 "0.7796$" H 3650 4350 50  0001 C CNN "LCSC_price100"
+F 20 "870-IS25LP032DJBLETR" H 3650 4350 50  0001 C CNN "LowCost"
+F 21 "FU003" H 3650 4350 50  0001 C CNN "Koncar"
 	1    3650 4350
 	1    0    0    -1
