File: power.sch (KiCad schematic (older format))
At the start: 79 parts, among them J5 VJ1, Q1 BC857, Q2 2N7002, U1 LFE5U-85F-6BG381C, U3 TLV62569DBV, U4 TLV62569DBV, U5 TLV62569DBV, U7 PCF8523, Y2 32768Hz

Commit message: schematics: clean up Mouser PN
Parts:
- D15: Distributor1_PN2 621-BAT54WSQ-7-F -> (none); Mouser2 (none) -> 621-BAT54WSQ-7-F
- RV3: EMPTY_PN (none) -> RC0603JR-070RL; MFG_PN RC0603JR-070RL -> (none)
Changed lines of the file:
@@
 F 4 "www.mouser.com" H 1300 1300 60  0001 C CNN "Mouser_URL"
 F 5 "www.yageo.com" H 1300 1300 50  0001 C CNN "MFG1_URL"
-F 6 "RC0603JR-070RL" H 1300 1300 50  0001 C CNN "MFG_PN"
+F 6 "RC0603JR-070RL" H 1300 1300 50  0001 C CNN "EMPTY_PN"
 F 7 "Leave empty" H 1300 1300 50  0001 C CNN "Note"
 	1    1300 1300
@@
 F 8 "www.mouser.com" H 3100 5600 50  0001 C CNN "Mouser_URL"
 F 9 "863-NSR0530HT1G " H 3100 5600 50  0001 C CNN "Mouser"
-F 10 "621-BAT54WSQ-7-F " H 3100 5600 50  0001 C CNN "Distributor1_PN2"
+F 10 "621-BAT54WSQ-7-F " H 3100 5600 50  0001 C CNN "Mouser2"
 	1    3100 5600
 	-1   0    0    1

Commit message: schematics: 470pF more suitable digikey PN
Parts:
- C2: Digikey CS0603KRX7R9BB471-ND -> 399-9086-1-ND
Changed lines of the file:
@@
 F 5 "CS0603KRX7R9BB471" H 9100 3300 50  0001 C CNN "MPN"
 F 6 "603-CS0603KRX79BB471" H 9100 3300 50  0001 C CNN "Mouser"
-F 7 "CS0603KRX7R9BB471-ND" H 9100 3300 50  0001 C CNN "Digikey"
+F 7 "399-9086-1-ND" H 9100 3300 50  0001 C CNN "Digikey"
 	1    9100 3300
 	1    0    0    -1

Commit message: schematics: Digikey currently available PN for C
Parts:
- C1: Digikey 311-3443-1-ND -> 1276-2911-1-ND
- C13: Digikey 311-3438-1-ND -> 1276-2904-1-ND
- C14: Digikey 311-1341-1-ND -> 399-6353-1-ND
- C25: Digikey 311-3107-1-ND -> 1276-2000-1-ND
Changed lines of the file:
@@
 F 4 "CC0805ZKY5V5BB226 " H 7400 3700 50  0001 C CNN "MPN"
 F 5 "603-CC805ZKY5V5BB226" H 7400 3700 50  0001 C CNN "Mouser"
-F 6 "311-3443-1-ND" H 7400 3700 50  0001 C CNN "Digikey"
+F 6 "1276-2911-1-ND" H 7400 3700 50  0001 C CNN "Digikey"
 	1    7400 3700
 	1    0    0    -1
@@
 F 4 "CC0805MRX5R6BB225" H 4300 3750 50  0001 C CNN "MPN"
 F 5 "603-CC805MRX5R6BB225" H 4300 3750 50  0001 C CNN "Mouser"
-F 6 "311-3438-1-ND" H 4300 3750 50  0001 C CNN "Digikey"
+F 6 "1276-2904-1-ND" H 4300 3750 50  0001 C CNN "Digikey"
 	1    4300 3750
 	1    0    0    -1
@@
 F 5 "CC0603KRX7R8BB104" H 3700 5850 50  0001 C CNN "MPN"
 F 6 "603-CC603KRX7R8BB104" H 3700 5850 50  0001 C CNN "Mouser"
-F 7 "311-1341-1-ND" H 3700 5850 50  0001 C CNN "Digikey"
+F 7 "399-6353-1-ND" H 3700 5850 50  0001 C CNN "Digikey"
 	1    3700 5850
 	1    0    0    -1
@@
 F 4 "CX0603MRX7R8BB223" H 5500 4750 50  0001 C CNN "MPN"
 F 5 "603-AC603KRX7R7BB223" H 5500 4750 50  0001 C CNN "Mouser"
-F 6 "311-3107-1-ND" H 5500 4750 50  0001 C CNN "Digikey"
+F 6 "1276-2000-1-ND" H 5500 4750 50  0001 C CNN "Digikey"
 	1    5500 4750
 	1    0    0    -1

Commit message: schematics: Digikey PN for R
Parts:
- R1: Digikey (none) -> YAG3569CT-ND
- R2: Digikey (none) -> 311-47.0KHRCT-ND
- R3: Digikey (none) -> YAG3613CT-ND
- R5: Digikey (none) -> 311-4.70MHRCT-ND
- R6: Digikey (none) -> 311-1.00KHRCT-ND
- RB1: Digikey (none) -> 311-18.0KHRCT-ND
- RB3: Digikey (none) -> YAG3605CT-ND
- RP1: Digikey (none) -> 541-2970-1-ND
Changed lines of the file:
@@
 F 5 "RC0603FR-1018KL" V 9600 3500 50  0001 C CNN "MPN"
 F 6 "603-RC0603FR-1018KL" V 9600 3500 50  0001 C CNN "Mouser"
+F 7 " 311-18.0KHRCT-ND" V 9600 3500 50  0001 C CNN "Digikey"
 	1    9600 3500
 	0    1    1    0
@@
 F 5 "RT0603FRE073K3L" V 9600 5900 50  0001 C CNN "MPN"
 F 6 "603-RT0603FRE073K3L" V 9600 5900 50  0001 C CNN "Mouser"
+F 7 "YAG3605CT-ND" V 9600 5900 50  0001 C CNN "Digikey"
 	1    9600 5900
 	0    1    1    0
@@
 F 4 "AC0603FR-1015KL" V 4300 4700 50  0001 C CNN "MPN"
 F 5 "603-AC0603FR-1015KL" V 4300 4700 50  0001 C CNN "Mouser"
+F 6 "YAG3569CT-ND" V 4300 4700 50  0001 C CNN "Digikey"
 	1    4300 4700
 	1    0    0    -1
@@
 F 5 "AC0603FR-0747KL" V 4300 5600 50  0001 C CNN "MPN"
 F 6 "603-AC0603FR-0747KL" V 4300 5600 50  0001 C CNN "Mouser"
+F 7 "311-47.0KHRCT-ND" V 4300 5600 50  0001 C CNN "Digikey"
 	1    4300 5600
 	1    0    0    -1
@@
 F 5 "www.bourns.com" V 3400 5850 50  0001 C CNN "MFG1_URL"
 F 6 "652-CR0603JW-475ELF" V 3400 5850 50  0001 C CNN "Mouser"
+F 7 "311-4.70MHRCT-ND" V 3400 5850 50  0001 C CNN "Digikey"
 	1    3400 5850
 	1    0    0    -1
@@
 F 4 "RC0603FR-071KL" V 3400 3750 50  0001 C CNN "MPN"
 F 5 "603-RC0603FR-071KL" V 3400 3750 50  0001 C CNN "Mouser"
+F 6 "311-1.00KHRCT-ND" V 3400 3750 50  0001 C CNN "Digikey"
 	1    3400 3750
 	0    1    1    0
@@
 F 4 "AC0603FR-104K7L" V 3150 4400 50  0001 C CNN "MPN"
 F 5 "603-AC0603FR-104K7L" V 3150 4400 50  0001 C CNN "Mouser"
+F 6 "YAG3613CT-ND" V 3150 4400 50  0001 C CNN "Digikey"
 	1    3150 4400
 	0    1    1    0
@@
 F 6 "RC0603JR-070RL" H 10700 3100 50  0001 C CNN "MPN"
 F 7 "603-RC0603JR-070RL" H 10700 3100 50  0001 C CNN "Mouser"
+F 8 "541-2970-1-ND" H 10700 3100 50  0001 C CNN "Digikey"
 	1    10700 3100
 	1    0    0    -1

Commit message: schematics: replacement for Digikey 2.2uF problematic part
Parts:
- C13: Digikey 1276-2904-1-ND -> 1276-2903-1-ND
Changed lines of the file:
@@
 F 4 "CC0805MRX5R6BB225" H 4300 3750 50  0001 C CNN "MPN"
 F 5 "603-CC805MRX5R6BB225" H 4300 3750 50  0001 C CNN "Mouser"
-F 6 "1276-2904-1-ND" H 4300 3750 50  0001 C CNN "Digikey"
+F 6 "1276-2903-1-ND" H 4300 3750 50  0001 C CNN "Digikey"
 	1    4300 3750
 	1    0    0    -1

Commit message: schematics: reducing number of different resistors, using 4x 1N4148 instead of 4x BAT54 schottky diodes.
Parts:
- R6: value 1k -> 1.2k; Digikey 311-1.00KHRCT-ND -> (none); MPN RC0603FR-071KL -> (none); Mouser 603-RC0603FR-071KL -> (none)
- R65: value 1k -> 680
- R8: value 1k -> 1.2k
Changed lines of the file:
@@
 AR Path="/58D51CAD/58D7B291" Ref="R6"  Part="1"
 F 0 "R6" V 3480 3750 50  0000 C CNN
-F 1 "1k" V 3400 3750 50  0000 C CNN
+F 1 "1.2k" V 3400 3750 50  0000 C CNN
 F 2 "Resistor_SMD:R_0603_1608Metric" V 3330 3750 50  0001 C CNN
 F 3 "" H 3400 3750 50  0000 C CNN
-F 4 "RC0603FR-071KL" V 3400 3750 50  0001 C CNN "MPN"
-F 5 "603-RC0603FR-071KL" V 3400 3750 50  0001 C CNN "Mouser"
-F 6 "311-1.00KHRCT-ND" V 3400 3750 50  0001 C CNN "Digikey"
 	1    3400 3750
 	0    1    1    0
@@
 AR Path="/58D51CAD/58D8111E" Ref="R8"  Part="1"
 F 0 "R8" V 4180 5200 50  0000 C CNN
-F 1 "1k" V 4100 5200 50  0000 C CNN
+F 1 "1.2k" V 4100 5200 50  0000 C CNN
 F 2 "Resistor_SMD:R_0603_1608Metric" V 4030 5200 50  0001 C CNN
 F 3 "" H 4100 5200 50  0000 C CNN
@@
 P 1500 2650
 F 0 "R65" V 1580 2650 50  0000 C CNN
-F 1 "1k" V 1500 2650 50  0000 C CNN
+F 1 "680" V 1500 2650 50  0000 C CNN
 F 2 "Resistor_SMD:R_0603_1608Metric" V 1430 2650 50  0001 C CNN
 F 3 "" H 1500 2650 50  0000 C CNN

Commit message: schematics: Available PN for Q1 Q2
Parts:
- Q1: Digikey 1727-2926-1-ND -> TBC857BLMCT-ND; Mouser 771-BC857B-T/R -> 863-BC857BLT1G
- Q2: Digikey 1727-4692-1-ND -> 2N7002K-TPMSCT-ND; Mouser 771-2N7002P-215 -> 512-2N7002
Changed lines of the file:
@@
 F 5 "2N7002P,215" H 4000 5600 60  0001 C CNN "MPN"
 F 6 "www.mouser.com" H 4000 5600 60  0001 C CNN "Mouser_URL"
-F 7 "771-2N7002P-215" H 4000 5600 60  0001 C CNN "Mouser"
-F 8 "1727-4692-1-ND" H 4000 5600 50  0001 C CNN "Digikey"
+F 7 "512-2N7002" H 4000 5600 60  0001 C CNN "Mouser"
+F 8 "2N7002K-TPMSCT-ND" H 4000 5600 50  0001 C CNN "Digikey"
 	1    4000 5600
 	1    0    0    -1
@@
 F 5 "BC857" H 3950 3750 60  0001 C CNN "MPN"
 F 6 "www.mouser.com" H 3950 3750 60  0001 C CNN "Mouser_URL"
-F 7 "771-BC857B-T/R" H 3950 3750 60  0001 C CNN "Mouser"
-F 8 "1727-2926-1-ND" H 3950 3750 50  0001 C CNN "Digikey"
+F 7 "863-BC857BLT1G" H 3950 3750 60  0001 C CNN "Mouser"
+F 8 "TBC857BLMCT-ND" H 3950 3750 50  0001 C CNN "Digikey"
 	1    3950 3750
 	1    0    0    1

Commit message: schematics: updating available PN for R,C
Parts:
- C1: Digikey 1276-2911-1-ND -> 1276-2412-1-ND
- C14: Digikey 399-6353-1-ND -> 445-8129-1-ND; Mouser 603-CC603KRX7R8BB104 -> C0603C104Z3VACTU
- R1: Mouser 603-AC0603FR-1015KL -> 603-RC0603FR-1015KL
- R2: Digikey 311-47.0KHRCT-ND -> P47.0KHCT-ND
- R3: Mouser 603-AC0603FR-104K7L -> 603-RC0603FR-074K7L
- RB1: Mouser 603-RC0603FR-1018KL -> 71-CRCW060318K0FKEAC
- RB3: Mouser 603-RT0603FRE073K3L -> 603-RC0603FR-103K3L
- RP1: Digikey 541-2970-1-ND -> 541-2968-1-ND
Changed lines of the file:
@@
 F 4 "CC0805ZKY5V5BB226 " H 7400 3700 50  0001 C CNN "MPN"
 F 5 "603-CC805ZKY5V5BB226" H 7400 3700 50  0001 C CNN "Mouser"
-F 6 "1276-2911-1-ND" H 7400 3700 50  0001 C CNN "Digikey"
+F 6 "1276-2412-1-ND" H 7400 3700 50  0001 C CNN "Digikey"
 	1    7400 3700
 	1    0    0    -1
@@
 F 4 "www.yageo.com" V 9600 3500 50  0001 C CNN "MFG1_URL"
 F 5 "RC0603FR-1018KL" V 9600 3500 50  0001 C CNN "MPN"
-F 6 "603-RC0603FR-1018KL" V 9600 3500 50  0001 C CNN "Mouser"
+F 6 "71-CRCW060318K0FKEAC" V 9600 3500 50  0001 C CNN "Mouser"
 F 7 " 311-18.0KHRCT-ND" V 9600 3500 50  0001 C CNN "Digikey"
 	1    9600 3500
@@
 F 4 "www.yageo.com" V 9600 5900 50  0001 C CNN "MFG1_URL"
 F 5 "RT0603FRE073K3L" V 9600 5900 50  0001 C CNN "MPN"
-F 6 "603-RT0603FRE073K3L" V 9600 5900 50  0001 C CNN "Mouser"
+F 6 "603-RC0603FR-103K3L" V 9600 5900 50  0001 C CNN "Mouser"
 F 7 "YAG3605CT-ND" V 9600 5900 50  0001 C CNN "Digikey"
 	1    9600 5900
@@
 F 3 "" H 4300 4700 50  0000 C CNN
 F 4 "AC0603FR-1015KL" V 4300 4700 50  0001 C CNN "MPN"
-F 5 "603-AC0603FR-1015KL" V 4300 4700 50  0001 C CNN "Mouser"
+F 5 "603-RC0603FR-1015KL" V 4300 4700 50  0001 C CNN "Mouser"
 F 6 "YAG3569CT-ND" V 4300 4700 50  0001 C CNN "Digikey"
 	1    4300 4700
@@
 F 5 "AC0603FR-0747KL" V 4300 5600 50  0001 C CNN "MPN"
 F 6 "603-AC0603FR-0747KL" V 4300 5600 50  0001 C CNN "Mouser"
-F 7 "311-47.0KHRCT-ND" V 4300 5600 50  0001 C CNN "Digikey"
+F 7 "P47.0KHCT-ND" V 4300 5600 50  0001 C CNN "Digikey"
 	1    4300 5600
 	1    0    0    -1
@@
 F 4 "www.yageo.com" H 3700 5850 50  0001 C CNN "MFG1_URL"
 F 5 "CC0603KRX7R8BB104" H 3700 5850 50  0001 C CNN "MPN"
-F 6 "603-CC603KRX7R8BB104" H 3700 5850 50  0001 C CNN "Mouser"
-F 7 "399-6353-1-ND" H 3700 5850 50  0001 C CNN "Digikey"
+F 6 "C0603C104Z3VACTU" H 3700 5850 50  0001 C CNN "Mouser"
+F 7 "445-8129-1-ND" H 3700 5850 50  0001 C CNN "Digikey"
 	1    3700 5850
 	1    0    0    -1
@@
 F 3 "" H 3150 4400 50  0000 C CNN
 F 4 "AC0603FR-104K7L" V 3150 4400 50  0001 C CNN "MPN"
-F 5 "603-AC0603FR-104K7L" V 3150 4400 50  0001 C CNN "Mouser"
+F 5 "603-RC0603FR-074K7L" V 3150 4400 50  0001 C CNN "Mouser"
 F 6 "YAG3613CT-ND" V 3150 4400 50  0001 C CNN "Digikey"
 	1    3150 4400
@@
 F 6 "RC0603JR-070RL" H 10700 3100 50  0001 C CNN "MPN"
 F 7 "603-RC0603JR-070RL" H 10700 3100 50  0001 C CNN "Mouser"
-F 8 "541-2970-1-ND" H 10700 3100 50  0001 C CNN "Digikey"
+F 8 "541-2968-1-ND" H 10700 3100 50  0001 C CNN "Digikey"
 	1    10700 3100
 	1    0    0    -1
