File: power.sch (KiCad schematic (older format))
At the start: 84 parts, among them J5 VJ1, Q1 BC857, Q2 2N7002, U1 LFE5U-85F-6BG381C, U3 TLV62569DBV, U4 TLV62569DBV, U5 TLV62569DBV, U7 MCP7940NT, Y2 32768Hz

Commit message: schematics: update mouser and digikey available PN for 2.2uH inductor
Parts:
- BAT1: Digike_y1 (none) -> BK-885-ND; Digike_y3 952-1662-1-ND -> (none); Digikey BK-885-ND -> 952-1662-1-ND
- L1: Digike_y1 (none) -> 490-18405-1-ND; Digikey 490-18405-1-ND -> 445-TFM322512ALMA2R2MTAACT-ND; Mouse_r2 810-TFM322512ALMA2R2 -> (none); Mouse_r3 (none) -> 81-DFE322520FD2R2MP2; Mouser 81-DFE322520FD2R2MP2 -> 810-TFM322512ALMA2R2
Changed lines of the file:
@@
 F 15 "855-S8201-46R" H 2650 4100 50  0001 C CNN "Mouse_r2"
 F 16 "534-3000TR" H 2650 4100 50  0001 C CNN "Mouse_r3"
-F 17 "BK-885-ND" H 2650 4100 50  0001 C CNN "Digikey"
-F 18 "36-3000CT-ND" H 2650 4100 50  0001 C CNN "Digike_y2"
-F 19 "952-1662-1-ND" H 2650 4100 50  0001 C CNN "Digike_y3"
+F 17 "952-1662-1-ND" H 2650 4100 50  0001 C CNN "Digikey"
+F 18 "BK-885-ND" H 2650 4100 50  0001 C CNN "Digike_y1"
+F 19 "36-3000CT-ND" H 2650 4100 50  0001 C CNN "Digike_y2"
 F 20 "C238097" H 2650 4100 50  0001 C CNN "LCSC"
 F 21 "1613707" H 2650 4100 50  0001 C CNN "RS"
@@
 F 14 "HEI322512A-2R2M-Q8" V 8900 3100 50  0001 C CNN "MP_N4"
 F 15 "81-LQH32PB2R2NN0L" V 8900 3100 50  0001 C CNN "MP_N5"
-F 16 "81-DFE322520FD2R2MP2" V 8900 3100 50  0001 C CNN "Mouser"
+F 16 "810-TFM322512ALMA2R2" V 8900 3100 50  0001 C CNN "Mouser"
 F 17 "81-DFE322512F-2R2MP2" V 8900 3100 50  0001 C CNN "Mouse_r1"
-F 18 "810-TFM322512ALMA2R2" V 8900 3100 50  0001 C CNN "Mouse_r2"
-F 19 "490-18405-1-ND" V 8900 3100 50  0001 C CNN "Digikey"
-F 20 "490-10649-1-ND" V 8900 3100 50  0001 C CNN "Digike_y2"
-F 21 "DFE322512F-2R2M=P2" V 8900 3100 50  0001 C CNN "Vertical"
-F 22 "0.48360$" V 8900 3100 50  0001 C CNN "price300_Vertical"
-F 23 "C285914" V 8900 3100 50  0001 C CNN "LCSC"
-F 24 "0.1082$" V 8900 3100 50  0001 C CNN "price300_LCSC"
-F 25 "https://datasheet.octopart.com/LQH32PB2R2NN0L-Murata-datasheet-20916646.pdf" V 8900 3100 50  0001 C CNN "DatasheetLC"
-F 26 "81-DFE252012P-2R2MP2" V 8900 3100 50  0001 C CNN "LowCost"
-F 27 "FL001" V 8900 3100 50  0001 C CNN "Koncar"
+F 18 "81-DFE322520FD2R2MP2" V 8900 3100 50  0001 C CNN "Mouse_r3"
+F 19 "445-TFM322512ALMA2R2MTAACT-ND" V 8900 3100 50  0001 C CNN "Digikey"
+F 20 "490-18405-1-ND" V 8900 3100 50  0001 C CNN "Digike_y1"
+F 21 "490-10649-1-ND" V 8900 3100 50  0001 C CNN "Digike_y2"
+F 22 "DFE322512F-2R2M=P2" V 8900 3100 50  0001 C CNN "Vertical"
+F 23 "0.48360$" V 8900 3100 50  0001 C CNN "price300_Vertical"
+F 24 "C285914" V 8900 3100 50  0001 C CNN "LCSC"
+F 25 "0.1082$" V 8900 3100 50  0001 C CNN "price300_LCSC"
+F 26 "https://datasheet.octopart.com/LQH32PB2R2NN0L-Murata-datasheet-20916646.pdf" V 8900 3100 50  0001 C CNN "DatasheetLC"
+F 27 "81-DFE252012P-2R2MP2" V 8900 3100 50  0001 C CNN "LowCost"
+F 28 "FL001" V 8900 3100 50  0001 C CNN "Koncar"
 	1    8900 3100
 	0    -1   -1   0

Commit message: schematics: untested mouser PN TI switcher 1.5A (not default)
Parts:
- U3: Mouse_r3 (none) -> 595-TLV62565DBVR
Changed lines of the file:
@@
 F 10 "595-TLV62569DBVR" H 8050 3400 50  0001 C CNN "Mouser"
 F 11 "453-DIO6015BCST5" H 8050 3400 50  0001 C CNN "Mouse_r2"
-F 12 "296-47360-1-ND" H 8050 3400 50  0001 C CNN "Digikey"
-F 13 "C141836" H 8050 3400 50  0001 C CNN "LCSC"
-F 14 "0.1843$" H 8050 3400 50  0001 C CNN "price100_LCSC"
-F 15 "http://www.dioo.com/attachments/files/20161031180022_361.pdf" H 8050 3400 50  0001 C CNN "DatasheetLC"
-F 16 "453-DIO6015BCST5" H 8050 3400 50  0001 C CNN "LowCost"
-F 17 "FU009" H 8050 3400 50  0001 C CNN "Koncar"
+F 12 "595-TLV62565DBVR" H 8050 3400 50  0001 C CNN "Mouse_r3"
+F 13 "296-47360-1-ND" H 8050 3400 50  0001 C CNN "Digikey"
+F 14 "C141836" H 8050 3400 50  0001 C CNN "LCSC"
+F 15 "0.1843$" H 8050 3400 50  0001 C CNN "price100_LCSC"
+F 16 "http://www.dioo.com/attachments/files/20161031180022_361.pdf" H 8050 3400 50  0001 C CNN "DatasheetLC"
+F 17 "453-DIO6015BCST5" H 8050 3400 50  0001 C CNN "LowCost"
+F 18 "FU009" H 8050 3400 50  0001 C CNN "Koncar"
 	1    8050 3400
 	1    0    0    -1

Commit message: schematics: 470pF->100pF
Parts:
- C10, C6: value 470pF -> 100pF
- C2: value 470pF -> 100pF; Digike_y2 (none) -> 399-9086-1-ND; Digikey 399-9086-1-ND -> 311-4078-1-ND; LCSC C22396 -> C14665; LCS_C2 (none) -> C22396; Mouse_r1 603-CC603KRX7R9BB471 -> 710-885012206081; Mouse_r4 (none) -> 603-CC603KRX7R9BB471; Mouser 710-885012206081 -> 603-CC603JRNPO9BN101
Changed lines of the file:
@@
 Title "ULX3S"
 Date ""
-Rev "1.0.7"
+Rev "1.0.8"
 Comp "EMARD"
 Comment1 "Power"
@@
 AR Path="/58D51CAD/58D5A146" Ref="C2"  Part="1"
 F 0 "C2" H 9125 3400 50  0000 L CNN
-F 1 "470pF" H 9125 3200 50  0000 L CNN
+F 1 "100pF" H 9125 3200 50  0000 L CNN
 F 2 "Capacitor_SMD:C_0603_1608Metric" H 9138 3150 50  0001 C CNN
 F 3 "" H 9100 3300 50  0000 C CNN
 F 4 "www.yageo.com" H 9100 3300 50  0001 C CNN "MNF1_URL"
 F 5 "CS0603KRX7R9BB471" H 9100 3300 50  0001 C CNN "MPN"
-F 6 "710-885012206081" H 9100 3300 50  0001 C CNN "Mouser"
-F 7 "603-CC603KRX7R9BB471 " H 9100 3300 50  0001 C CNN "Mouse_r1"
-F 8 "603-CS0603KRX79BB471" H 9100 3300 50  0001 C CNN "Mouse_r2"
-F 9 "399-9086-1-ND" H 9100 3300 50  0001 C CNN "Digikey"
-F 10 "C22396" H 9100 3300 50  0001 C CNN "LCSC"
-F 11 "FC006" H 9100 3300 50  0001 C CNN "Koncar"
+F 6 "603-CC603JRNPO9BN101" H 9100 3300 50  0001 C CNN "Mouser"
+F 7 "710-885012206081" H 9100 3300 50  0001 C CNN "Mouse_r1"
+F 8 "603-CC603KRX7R9BB471 " H 9100 3300 50  0001 C CNN "Mouse_r4"
+F 9 "603-CS0603KRX79BB471" H 9100 3300 50  0001 C CNN "Mouse_r2"
+F 10 "311-4078-1-ND" H 9100 3300 50  0001 C CNN "Digikey"
+F 11 "399-9086-1-ND" H 9100 3300 50  0001 C CNN "Digike_y2"
+F 12 "C14665" H 9100 3300 50  0001 C CNN "LCSC"
+F 13 "C22396" H 9100 3300 50  0001 C CNN "LCS_C2"
+F 14 "FC006" H 9100 3300 50  0001 C CNN "Koncar"
 	1    9100 3300
 	1    0    0    -1
@@
 AR Path="/58D51CAD/58D6296A" Ref="C6"  Part="1"
 F 0 "C6" H 9125 5800 50  0000 L CNN
-F 1 "470pF" H 9125 5600 50  0000 L CNN
+F 1 "100pF" H 9125 5600 50  0000 L CNN
 F 2 "Capacitor_SMD:C_0603_1608Metric" H 9138 5550 50  0001 C CNN
 F 3 "" H 9100 5700 50  0000 C CNN
@@
 AR Path="/58D51CAD/58D67BDE" Ref="C10"  Part="1"
 F 0 "C10" H 9125 4600 50  0000 L CNN
-F 1 "470pF" H 9125 4400 50  0000 L CNN
+F 1 "100pF" H 9125 4400 50  0000 L CNN
 F 2 "Capacitor_SMD:C_0603_1608Metric" H 9138 4350 50  0001 C CNN
 F 3 "" H 9100 4500 50  0000 C CNN

Commit message: schematics: digikey PN for 85F
Parts:
- U1: Mouser 842-LFE5U85F6BG381C -> (none)
Changed lines of the file:
@@
 F 4 "www.latticesemi.com" H 6200 1800 60  0001 C CNN "MNF1_URL"
 F 5 "LFE5U-85F-6BG381C" H 6200 1800 60  0001 C CNN "MPN"
-F 6 "842-LFE5U85F6BG381C" H 6200 1800 60  0001 C CNN "Mouser"
 	9    6200 1800
 	1    0    0    -1

Commit message: schematics: LCSC PN 2.2uH inductor
Parts:
- L1: LCSC C285914 -> C285758; LCS_C2 (none) -> C285914
Changed lines of the file:
@@
 F 22 "DFE322512F-2R2M=P2" V 8900 3100 50  0001 C CNN "Vertical"
 F 23 "0.48360$" V 8900 3100 50  0001 C CNN "price300_Vertical"
-F 24 "C285914" V 8900 3100 50  0001 C CNN "LCSC"
-F 25 "0.1082$" V 8900 3100 50  0001 C CNN "price300_LCSC"
-F 26 "https://datasheet.octopart.com/LQH32PB2R2NN0L-Murata-datasheet-20916646.pdf" V 8900 3100 50  0001 C CNN "DatasheetLC"
-F 27 "81-DFE252012P-2R2MP2" V 8900 3100 50  0001 C CNN "LowCost"
-F 28 "FL001" V 8900 3100 50  0001 C CNN "Koncar"
+F 24 "C285758" V 8900 3100 50  0001 C CNN "LCSC"
+F 25 "C285914" V 8900 3100 50  0001 C CNN "LCS_C2"
+F 26 "0.1082$" V 8900 3100 50  0001 C CNN "price300_LCSC"
+F 27 "https://datasheet.octopart.com/LQH32PB2R2NN0L-Murata-datasheet-20916646.pdf" V 8900 3100 50  0001 C CNN "DatasheetLC"
+F 28 "81-DFE252012P-2R2MP2" V 8900 3100 50  0001 C CNN "LowCost"
+F 29 "FL001" V 8900 3100 50  0001 C CNN "Koncar"
 	1    8900 3100
 	0    -1   -1   0

Commit message: schematics: newark PNs for some semiconductors and connectors (not all)
Parts:
- BAT1: Newark (none) -> 65T3841
- D15: Newark (none) -> 83H6419
- D16: Mouser 512-1N914BWS -> 512-1N914BWS; Newark (none) -> 12T2305
- L1: Newark (none) -> 57AC6667
- Q1: Mouser 583-BC856A-T -> 583-BC856A-T; Newark (none) -> 45J0600
- Q2: Newark (none) -> 65W8792
- U3: Newark (none) -> 54AH1585
- U7: Newark (none) -> 57AC2515
- Y2: Newark (none) -> 94X0923
Changed lines of the file:
@@
 F 12 "MCP7940NT-I/SNCT-ND" H 1950 3650 50  0001 C CNN "Digikey"
 F 13 "568-5306-1-ND" H 1950 3650 50  0001 C CNN "Digike_y2"
-F 14 "C148052" H 1950 3650 50  0001 C CNN "LCSC"
-F 15 "MCP7940NT-I/SN" H 1950 3650 50  0001 C CNN "Arrow"
-F 16 "0.6427$" H 1950 3650 50  0001 C CNN "price100_Arrow"
-F 17 "FU006" H 1950 3650 50  0001 C CNN "Koncar"
+F 14 "57AC2515" H 1950 3650 50  0001 C CNN "Newark"
+F 15 "C148052" H 1950 3650 50  0001 C CNN "LCSC"
+F 16 "MCP7940NT-I/SN" H 1950 3650 50  0001 C CNN "Arrow"
+F 17 "0.6427$" H 1950 3650 50  0001 C CNN "price100_Arrow"
+F 18 "FU006" H 1950 3650 50  0001 C CNN "Koncar"
 	1    1950 3650
 	1    0    0    -1
@@
 F 19 "36-3000CT-ND" H 2650 4100 50  0001 C CNN "Digike_y2"
 F 20 "C238097" H 2650 4100 50  0001 C CNN "LCSC"
-F 21 "1613707" H 2650 4100 50  0001 C CNN "RS"
-F 22 "0.33296$" H 2650 4100 50  0001 C CNN "price100_RS"
-F 23 "FBAT001" H 2650 4100 50  0001 C CNN "Koncar"
+F 21 "65T3841" H 2650 4100 50  0001 C CNN "Newark"
+F 22 "1613707" H 2650 4100 50  0001 C CNN "RS"
+F 23 "0.33296$" H 2650 4100 50  0001 C CNN "price100_RS"
+F 24 "FBAT001" H 2650 4100 50  0001 C CNN "Koncar"
 	1    2650 4100
 	1    0    0    -1
@@
 F 12 "0.093$" H 3100 5600 50  0001 C CNN "price200_Mouser"
 F 13 "NSR0530HT1GOSCT-ND" H 3100 5600 50  0001 C CNN "Digikey"
-F 14 "C12744" H 3100 5600 50  0001 C CNN "LCSC"
-F 15 "FV003" H 3100 5600 50  0001 C CNN "Koncar"
+F 14 "83H6419" H 3100 5600 50  0001 C CNN "Newark"
+F 15 "C12744" H 3100 5600 50  0001 C CNN "LCSC"
+F 16 "FV003" H 3100 5600 50  0001 C CNN "Koncar"
 	1    3100 5600
 	-1   0    0    1
@@
 F 12 "1923-1021-1-ND" V 900 3650 50  0001 C CNN "Digikey"
 F 13 "1923-1019-1-ND" V 900 3650 50  0001 C CNN "Digike_y2"
-F 14 "C252402" V 900 3650 50  0001 C CNN "LCSC"
-F 15 "32.768K-855MXR" V 900 3650 50  0001 C CNN "TME"
-F 16 "0.30226$" V 900 3650 50  0001 C CNN "price100_TME"
-F 17 "FQ002" V 900 3650 50  0001 C CNN "Koncar"
+F 14 "94X0923" V 900 3650 50  0001 C CNN "Newark"
+F 15 "C252402" V 900 3650 50  0001 C CNN "LCSC"
+F 16 "32.768K-855MXR" V 900 3650 50  0001 C CNN "TME"
+F 17 "0.30226$" V 900 3650 50  0001 C CNN "price100_TME"
+F 18 "FQ002" V 900 3650 50  0001 C CNN "Koncar"
 	1    900  3650
 	0    1    -1   0
@@
 F 7 "512-2N7002L" H 4000 5600 60  0001 C CNN "Mouse_r2"
 F 8 "2N7002K-TPMSCT-ND" H 4000 5600 50  0001 C CNN "Digikey"
-F 9 "C179727" H 4000 5600 50  0001 C CNN "LCSC"
-F 10 "T2N7002AK,LM" H 4000 5600 50  0001 C CNN "Arrow"
-F 11 "0.0437$" H 4000 5600 50  0001 C CNN "price_Arrow"
-F 12 "FT002" H 4000 5600 50  0001 C CNN "Koncar"
+F 9 "65W8792" H 4000 5600 50  0001 C CNN "Newark"
+F 10 "C179727" H 4000 5600 50  0001 C CNN "LCSC"
+F 11 "T2N7002AK,LM" H 4000 5600 50  0001 C CNN "Arrow"
+F 12 "0.0437$" H 4000 5600 50  0001 C CNN "price_Arrow"
+F 13 "FT002" H 4000 5600 50  0001 C CNN "Koncar"
 	1    4000 5600
 	1    0    0    -1
@@
 F 4 "www.nxp.com" H 3950 3750 50  0001 C CNN "MNF1_URL"
 F 5 "BC857" H 3950 3750 60  0001 C CNN "MPN"
-F 6 " 583-BC856A-T" H 3950 3750 50  0001 C CNN "Mouser"
+F 6 "583-BC856A-T" H 3950 3750 50  0001 C CNN "Mouser"
 F 7 "863-BC857BLT1G" H 3950 3750 60  0001 C CNN "Mouse_r2"
 F 8 "0.06$" H 3950 3750 50  0001 C CNN "price100_Mouser"
 F 9 "TBC857BLMCT-ND" H 3950 3750 50  0001 C CNN "Digikey"
-F 10 "C181146" H 3950 3750 50  0001 C CNN "LCSC"
-F 11 "FT001" H 3950 3750 50  0001 C CNN "Koncar"
+F 10 "45J0600" H 3950 3750 50  0001 C CNN "Newark"
+F 11 "C181146" H 3950 3750 50  0001 C CNN "LCSC"
+F 12 "FT001" H 3950 3750 50  0001 C CNN "Koncar"
 	1    3950 3750
 	1    0    0    1
@@
 F 4 "www.fairchildsemi.com" H 2900 3950 50  0001 C CNN "MNF1_URL"
 F 5 "1N4148WS " H 2900 3950 50  0001 C CNN "MPN"
-F 6 "512-1N914BWS " H 2900 3950 50  0001 C CNN "Mouser"
+F 6 "512-1N914BWS" H 2900 3950 50  0001 C CNN "Mouser"
 F 7 "833-1N4148WX-TP" H 2900 3950 50  0001 C CNN "Mouse_r1"
 F 8 "863-MMDL914T1G" H 2900 3950 50  0001 C CNN "Mouse_r2"
@@
 F 10 "1N4148WXTPMSCT-ND" H 2900 3950 50  0001 C CNN "Digike_y3"
 F 11 "1N4148WSFSCT-ND" H 2900 3950 50  0001 C CNN "Digike_y2"
-F 12 "C258181" H 2900 3950 50  0001 C CNN "LCSC"
-F 13 "C1S541901230010" H 2900 3950 50  0001 C CNN "Chip1stop"
-F 14 "0.01209$" H 2900 3950 50  0001 C CNN "price1200_Chip1stop"
-F 15 "FV001" H 2900 3950 50  0001 C CNN "Koncar"
+F 12 "12T2305" H 2900 3950 50  0001 C CNN "Newark"
+F 13 "C258181" H 2900 3950 50  0001 C CNN "LCSC"
+F 14 "C1S541901230010" H 2900 3950 50  0001 C CNN "Chip1stop"
+F 15 "0.01209$" H 2900 3950 50  0001 C CNN "price1200_Chip1stop"
+F 16 "FV001" H 2900 3950 50  0001 C CNN "Koncar"
 	1    2900 3950
 	0    -1   -1   0
@@
 F 20 "490-18405-1-ND" V 8900 3100 50  0001 C CNN "Digike_y1"
 F 21 "490-10649-1-ND" V 8900 3100 50  0001 C CNN "Digike_y2"
-F 22 "DFE322512F-2R2M=P2" V 8900 3100 50  0001 C CNN "Vertical"
-F 23 "0.48360$" V 8900 3100 50  0001 C CNN "price300_Vertical"
-F 24 "C285758" V 8900 3100 50  0001 C CNN "LCSC"
-F 25 "C285914" V 8900 3100 50  0001 C CNN "LCS_C2"
-F 26 "0.1082$" V 8900 3100 50  0001 C CNN "price300_LCSC"
-F 27 "https://datasheet.octopart.com/LQH32PB2R2NN0L-Murata-datasheet-20916646.pdf" V 8900 3100 50  0001 C CNN "DatasheetLC"
-F 28 "81-DFE252012P-2R2MP2" V 8900 3100 50  0001 C CNN "LowCost"
-F 29 "FL001" V 8900 3100 50  0001 C CNN "Koncar"
+F 22 "57AC6667" V 8900 3100 50  0001 C CNN "Newark"
+F 23 "DFE322512F-2R2M=P2" V 8900 3100 50  0001 C CNN "Vertical"
+F 24 "0.48360$" V 8900 3100 50  0001 C CNN "price300_Vertical"
+F 25 "C285758" V 8900 3100 50  0001 C CNN "LCSC"
+F 26 "C285914" V 8900 3100 50  0001 C CNN "LCS_C2"
+F 27 "0.1082$" V 8900 3100 50  0001 C CNN "price300_LCSC"
+F 28 "https://datasheet.octopart.com/LQH32PB2R2NN0L-Murata-datasheet-20916646.pdf" V 8900 3100 50  0001 C CNN "DatasheetLC"
+F 29 "81-DFE252012P-2R2MP2" V 8900 3100 50  0001 C CNN "LowCost"
+F 30 "FL001" V 8900 3100 50  0001 C CNN "Koncar"
 	1    8900 3100
 	0    -1   -1   0
@@
 F 12 "595-TLV62565DBVR" H 8050 3400 50  0001 C CNN "Mouse_r3"
 F 13 "296-47360-1-ND" H 8050 3400 50  0001 C CNN "Digikey"
-F 14 "C141836" H 8050 3400 50  0001 C CNN "LCSC"
-F 15 "0.1843$" H 8050 3400 50  0001 C CNN "price100_LCSC"
-F 16 "http://www.dioo.com/attachments/files/20161031180022_361.pdf" H 8050 3400 50  0001 C CNN "DatasheetLC"
-F 17 "453-DIO6015BCST5" H 8050 3400 50  0001 C CNN "LowCost"
-F 18 "FU009" H 8050 3400 50  0001 C CNN "Koncar"
+F 14 "54AH1585" H 8050 3400 50  0001 C CNN "Newark"
+F 15 "C141836" H 8050 3400 50  0001 C CNN "LCSC"
+F 16 "0.1843$" H 8050 3400 50  0001 C CNN "price100_LCSC"
+F 17 "http://www.dioo.com/attachments/files/20161031180022_361.pdf" H 8050 3400 50  0001 C CNN "DatasheetLC"
+F 18 "453-DIO6015BCST5" H 8050 3400 50  0001 C CNN "LowCost"
+F 19 "FU009" H 8050 3400 50  0001 C CNN "Koncar"
 	1    8050 3400
 	1    0    0    -1

Commit message: schematics: Newark PN switches
Parts:
- B0: Newark (none) -> 79AH5908
Changed lines of the file:
@@
 F 6 "611-PTS645SL50SMTR92" H 2200 4600 50  0001 C CNN "Mouser"
 F 7 "CKN9088CT-ND" H 2200 4600 50  0001 C CNN "Digikey"
-F 8 "C285463" H 2200 4600 50  0001 C CNN "LCSC"
-F 9 "0.09966$" H 2200 4600 50  0001 C CNN "price700_LCSC"
-F 10 "FSW001" H 2200 4600 50  0001 C CNN "Koncar"
-F 11 "T" H 2200 4600 50  0001 C CNN "Side"
+F 8 "79AH5908" H 2200 4600 50  0001 C CNN "Newark"
+F 9 "C285463" H 2200 4600 50  0001 C CNN "LCSC"
+F 10 "0.09966$" H 2200 4600 50  0001 C CNN "price700_LCSC"
+F 11 "FSW001" H 2200 4600 50  0001 C CNN "Koncar"
+F 12 "T" H 2200 4600 50  0001 C CNN "Side"
 	1    2200 4600
 	-1   0    0    -1

Commit message: schematics: newark PN capacitors
Parts:
- C1: Newark (none) -> 08P5169
- C13: Newar_k2 (none) -> 70K9141; Newark (none) -> 73AH0064
- C14: Newark (none) -> 82AC9347
- C2: Newark (none) -> 38K9273
- C25: Newark (none) -> 82AC9346
- C56: Newark (none) -> 96Y8338
Changed lines of the file:
@@
 F 10 "1276-2413-1-ND" H 7400 3700 50  0001 C CNN "Digikey"
 F 11 "1276-2412-1-ND" H 7400 3700 50  0001 C CNN "Digike_y2"
-F 12 "C29277" H 7400 3700 50  0001 C CNN "LCSC"
-F 13 "FC004" H 7400 3700 50  0001 C CNN "Koncar"
+F 12 "08P5169" H 7400 3700 50  0001 C CNN "Newark"
+F 13 "C29277" H 7400 3700 50  0001 C CNN "LCSC"
+F 14 "FC004" H 7400 3700 50  0001 C CNN "Koncar"
 	1    7400 3700
 	1    0    0    -1
@@
 F 10 "311-4078-1-ND" H 9100 3300 50  0001 C CNN "Digikey"
 F 11 "399-9086-1-ND" H 9100 3300 50  0001 C CNN "Digike_y2"
-F 12 "C14665" H 9100 3300 50  0001 C CNN "LCSC"
-F 13 "C22396" H 9100 3300 50  0001 C CNN "LCS_C2"
-F 14 "FC006" H 9100 3300 50  0001 C CNN "Koncar"
+F 12 "38K9273" H 9100 3300 50  0001 C CNN "Newark"
+F 13 "C14665" H 9100 3300 50  0001 C CNN "LCSC"
+F 14 "C22396" H 9100 3300 50  0001 C CNN "LCS_C2"
+F 15 "FC006" H 9100 3300 50  0001 C CNN "Koncar"
 	1    9100 3300
 	1    0    0    -1
@@
 F 7 "587-5918-1-ND" H 4300 3750 50  0001 C CNN "Digikey"
 F 8 "1276-2903-1-ND" H 4300 3750 50  0001 C CNN "Digike_y2"
-F 9 "C87995" H 4300 3750 50  0001 C CNN "LCSC"
-F 10 "FC001" H 4300 3750 50  0001 C CNN "Koncar"
+F 9 "73AH0064" H 4300 3750 50  0001 C CNN "Newark"
+F 10 "70K9141" H 4300 3750 50  0001 C CNN "Newar_k2"
+F 11 "C87995" H 4300 3750 50  0001 C CNN "LCSC"
+F 12 "FC001" H 4300 3750 50  0001 C CNN "Koncar"
 	1    4300 3750
 	1    0    0    -1
@@
 F 7 "81-GCM188R71E224K55D" H 3700 5850 50  0001 C CNN "Mouse_r1"
 F 8 "1276-1112-1-ND" H 3700 5850 50  0001 C CNN "Digikey"
-F 9 "C326805" H 3700 5850 50  0001 C CNN "LCSC"
-F 10 "FC002" H 3700 5850 50  0001 C CNN "Koncar"
-F 11 "TB" H 3700 5850 50  0001 C CNN "Side"
+F 9 "82AC9347" H 3700 5850 50  0001 C CNN "Newark"
+F 10 "C326805" H 3700 5850 50  0001 C CNN "LCSC"
+F 11 "FC002" H 3700 5850 50  0001 C CNN "Koncar"
+F 12 "TB" H 3700 5850 50  0001 C CNN "Side"
 	1    3700 5850
 	1    0    0    -1
@@
 F 9 "587-1238-1-ND" H 5250 4750 50  0001 C CNN "Digikey"
 F 10 "1276-2000-1-ND" H 5250 4750 50  0001 C CNN "Digike_y2"
-F 11 "C107137" H 5250 4750 50  0001 C CNN "LCSC"
-F 12 "FC003" H 5250 4750 50  0001 C CNN "Koncar"
+F 11 "82AC9346" H 5250 4750 50  0001 C CNN "Newark"
+F 12 "C107137" H 5250 4750 50  0001 C CNN "LCSC"
+F 13 "FC003" H 5250 4750 50  0001 C CNN "Koncar"
 	1    5250 4750
 	1    0    0    -1
@@
 F 9 "311-3848-1-ND" H 900 3250 50  0001 C CNN "Digike_y1"
 F 10 "311-3855-1-ND" H 900 3250 50  0001 C CNN "Digike_y2"
-F 11 "C314302" H 900 3250 50  0001 C CNN "LCSC"
-F 12 "C85300" H 900 3250 50  0001 C CNN "LCS_C2"
-F 13 "FC005" H 900 3250 50  0001 C CNN "Koncar"
+F 11 "96Y8338" H 900 3250 50  0001 C CNN "Newark"
+F 12 "C314302" H 900 3250 50  0001 C CNN "LCSC"
+F 13 "C85300" H 900 3250 50  0001 C CNN "LCS_C2"
+F 14 "FC005" H 900 3250 50  0001 C CNN "Koncar"
 	1    900  3250
 	1    0    0    -1
