File: ram.sch (KiCad schematic (older format))
At the start: 7 parts, among them U1 LFE5U-85F-6BG381C, U9 MT48LC16M16A2TG

Commit message: schematics: Additional field "Koncar" with their specific part number aliases
Parts:
- U9: Koncar (none) -> FU007
Changed lines of the file:
@@
 F 12 "870-IS42S16160G7TLTR" H 5450 3500 50  0001 C CNN "Mouser2"
 F 13 "1450-1352-1-ND" H 5450 3500 50  0001 C CNN "Digikey"
+F 14 "FU007" H 5450 3500 50  0001 C CNN "Koncar"
 	1    5450 3500
 	1    0    0    -1

Commit message: schematics: add "Side" field for parts which appear on top side
Parts:
- U9: Side (none) -> T
Changed lines of the file:
@@
 F 13 "1450-1352-1-ND" H 5450 3500 50  0001 C CNN "Digikey"
 F 14 "FU007" H 5450 3500 50  0001 C CNN "Koncar"
+F 15 "T" H 5450 3500 50  0001 C CNN "Side"
 	1    5450 3500
 	1    0    0    -1

Commit message: schematics: cheaper manufacturers PNs and some prices
Parts:
- U9: Mouser_price100 (none) -> 1.6€
Changed lines of the file:
@@
 F 10 "www.mouser.com" H 5450 3500 60  0001 C CNN "Mouser_URL"
 F 11 "913-4816M16A2TG6AGTR" H 5450 3500 60  0001 C CNN "Mouser"
-F 12 "870-IS42S16160G7TLTR" H 5450 3500 50  0001 C CNN "Mouser2"
-F 13 "1450-1352-1-ND" H 5450 3500 50  0001 C CNN "Digikey"
-F 14 "FU007" H 5450 3500 50  0001 C CNN "Koncar"
-F 15 "T" H 5450 3500 50  0001 C CNN "Side"
+F 12 "1.6€" H 5450 3500 50  0001 C CNN "Mouser_price100"
+F 13 "870-IS42S16160G7TLTR" H 5450 3500 50  0001 C CNN "Mouser2"
+F 14 "1450-1352-1-ND" H 5450 3500 50  0001 C CNN "Digikey"
+F 15 "FU007" H 5450 3500 50  0001 C CNN "Koncar"
+F 16 "T" H 5450 3500 50  0001 C CNN "Side"
 	1    5450 3500
 	1    0    0    -1

Commit message: schematics: cheaper SDRAM
Parts:
- U9: LCSC (none) -> C62379; LCSC_price100 (none) -> 0.7137$; MFG3 (none) -> Winbond; MPN3 (none) -> W9812G6KH-6
Changed lines of the file:
@@
 F 8 "ISSI" H 5450 3500 50  0001 C CNN "MFG2"
 F 9 "IS42S16160G-7TL-TR" H 5450 3500 50  0001 C CNN "MPN2"
-F 10 "www.mouser.com" H 5450 3500 60  0001 C CNN "Mouser_URL"
-F 11 "913-4816M16A2TG6AGTR" H 5450 3500 60  0001 C CNN "Mouser"
-F 12 "1.6€" H 5450 3500 50  0001 C CNN "Mouser_price100"
-F 13 "870-IS42S16160G7TLTR" H 5450 3500 50  0001 C CNN "Mouser2"
-F 14 "1450-1352-1-ND" H 5450 3500 50  0001 C CNN "Digikey"
-F 15 "FU007" H 5450 3500 50  0001 C CNN "Koncar"
-F 16 "T" H 5450 3500 50  0001 C CNN "Side"
+F 10 "Winbond" H 5450 3500 50  0001 C CNN "MFG3"
+F 11 "W9812G6KH-6" H 5450 3500 50  0001 C CNN "MPN3"
+F 12 "www.mouser.com" H 5450 3500 60  0001 C CNN "Mouser_URL"
+F 13 "913-4816M16A2TG6AGTR" H 5450 3500 60  0001 C CNN "Mouser"
+F 14 "1.6€" H 5450 3500 50  0001 C CNN "Mouser_price100"
+F 15 "870-IS42S16160G7TLTR" H 5450 3500 50  0001 C CNN "Mouser2"
+F 16 "1450-1352-1-ND" H 5450 3500 50  0001 C CNN "Digikey"
+F 17 "C62379" H 5450 3500 50  0001 C CNN "LCSC"
+F 18 "0.7137$" H 5450 3500 50  0001 C CNN "LCSC_price100"
+F 19 "FU007" H 5450 3500 50  0001 C CNN "Koncar"
+F 20 "T" H 5450 3500 50  0001 C CNN "Side"
 	1    5450 3500
 	1    0    0    -1

Commit message: renaming *_price -> price_* fields that may be misinterpreted by 1-clock-bom
Parts:
- U9: LCSC_price100 0.7137$ -> (none); Mouser_price100 1.6€ -> (none); price100_LCSC (none) -> 0.7137$; price100_Mouser (none) -> 1.6€
Changed lines of the file:
@@
 F 12 "www.mouser.com" H 5450 3500 60  0001 C CNN "Mouser_URL"
 F 13 "913-4816M16A2TG6AGTR" H 5450 3500 60  0001 C CNN "Mouser"
-F 14 "1.6€" H 5450 3500 50  0001 C CNN "Mouser_price100"
+F 14 "1.6€" H 5450 3500 50  0001 C CNN "price100_Mouser"
 F 15 "870-IS42S16160G7TLTR" H 5450 3500 50  0001 C CNN "Mouser2"
 F 16 "1450-1352-1-ND" H 5450 3500 50  0001 C CNN "Digikey"
 F 17 "C62379" H 5450 3500 50  0001 C CNN "LCSC"
-F 18 "0.7137$" H 5450 3500 50  0001 C CNN "LCSC_price100"
+F 18 "0.7137$" H 5450 3500 50  0001 C CNN "price100_LCSC"
 F 19 "FU007" H 5450 3500 50  0001 C CNN "Koncar"
 F 20 "T" H 5450 3500 50  0001 C CNN "Side"

Commit message: schematics: PN for 64MB SDRAM
Parts:
- U9: Datasheet4 (none) -> https://www.alliancememory.com/wp-content/uploads/pdf/dram/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; MFG4 (none) -> Alliance; MPN4 (none) -> AS4C32M16SB-7TCN; Mouser4 (none) -> 913-AS4C32M16SB-7TCN
Changed lines of the file:
@@
 F 10 "Winbond" H 5450 3500 50  0001 C CNN "MFG3"
 F 11 "W9812G6KH-6" H 5450 3500 50  0001 C CNN "MPN3"
-F 12 "www.mouser.com" H 5450 3500 60  0001 C CNN "Mouser_URL"
-F 13 "913-4816M16A2TG6AGTR" H 5450 3500 60  0001 C CNN "Mouser"
-F 14 "1.6€" H 5450 3500 50  0001 C CNN "price100_Mouser"
-F 15 "870-IS42S16160G7TLTR" H 5450 3500 50  0001 C CNN "Mouser2"
-F 16 "1450-1352-1-ND" H 5450 3500 50  0001 C CNN "Digikey"
-F 17 "C62379" H 5450 3500 50  0001 C CNN "LCSC"
-F 18 "0.7137$" H 5450 3500 50  0001 C CNN "price100_LCSC"
-F 19 "FU007" H 5450 3500 50  0001 C CNN "Koncar"
-F 20 "T" H 5450 3500 50  0001 C CNN "Side"
+F 12 "https://www.alliancememory.com/wp-content/uploads/pdf/dram/512M%20SDRAM_%20B%20die_AS4C32M16SB-7TCN-7TIN-6TIN_Rev%201.0%20June%202016.pdf" H 5450 3500 50  0001 C CNN "Datasheet4"
+F 13 "Alliance" H 5450 3500 50  0001 C CNN "MFG4"
+F 14 "AS4C32M16SB-7TCN" H 5450 3500 50  0001 C CNN "MPN4"
+F 15 "www.mouser.com" H 5450 3500 60  0001 C CNN "Mouser_URL"
+F 16 "913-4816M16A2TG6AGTR" H 5450 3500 60  0001 C CNN "Mouser"
+F 17 "1.6€" H 5450 3500 50  0001 C CNN "price100_Mouser"
+F 18 "870-IS42S16160G7TLTR" H 5450 3500 50  0001 C CNN "Mouser2"
+F 19 "913-AS4C32M16SB-7TCN" H 5450 3500 50  0001 C CNN "Mouser4"
+F 20 "1450-1352-1-ND" H 5450 3500 50  0001 C CNN "Digikey"
+F 21 "C62379" H 5450 3500 50  0001 C CNN "LCSC"
+F 22 "0.7137$" H 5450 3500 50  0001 C CNN "price100_LCSC"
+F 23 "FU007" H 5450 3500 50  0001 C CNN "Koncar"
+F 24 "T" H 5450 3500 50  0001 C CNN "Side"
 	1    5450 3500
 	1    0    0    -1

Commit message: schematics: update PN
Parts:
- U9: Mouse_r1 (none) -> 913-4816M16A2TG6AGTR; Mouse_r2 (none) -> 870-IS42S16160G7TLTR; Mouser 913-4816M16A2TG6AGTR -> 913-AS4C32M16SB-7TCN; Mouser2 870-IS42S16160G7TLTR -> (none); Mouser4 913-AS4C32M16SB-7TCN -> (none); Mouser_URL www.mouser.com -> (none)
Changed lines of the file:
@@
 F 13 "Alliance" H 5450 3500 50  0001 C CNN "MFG4"
 F 14 "AS4C32M16SB-7TCN" H 5450 3500 50  0001 C CNN "MPN4"
-F 15 "www.mouser.com" H 5450 3500 60  0001 C CNN "Mouser_URL"
-F 16 "913-4816M16A2TG6AGTR" H 5450 3500 60  0001 C CNN "Mouser"
+F 15 "913-AS4C32M16SB-7TCN" H 5450 3500 50  0001 C CNN "Mouser"
+F 16 "913-4816M16A2TG6AGTR" H 5450 3500 60  0001 C CNN "Mouse_r1"
 F 17 "1.6€" H 5450 3500 50  0001 C CNN "price100_Mouser"
-F 18 "870-IS42S16160G7TLTR" H 5450 3500 50  0001 C CNN "Mouser2"
-F 19 "913-AS4C32M16SB-7TCN" H 5450 3500 50  0001 C CNN "Mouser4"
-F 20 "1450-1352-1-ND" H 5450 3500 50  0001 C CNN "Digikey"
-F 21 "C62379" H 5450 3500 50  0001 C CNN "LCSC"
-F 22 "0.7137$" H 5450 3500 50  0001 C CNN "price100_LCSC"
-F 23 "FU007" H 5450 3500 50  0001 C CNN "Koncar"
-F 24 "T" H 5450 3500 50  0001 C CNN "Side"
+F 18 "870-IS42S16160G7TLTR" H 5450 3500 50  0001 C CNN "Mouse_r2"
+F 19 "1450-1352-1-ND" H 5450 3500 50  0001 C CNN "Digikey"
+F 20 "C62379" H 5450 3500 50  0001 C CNN "LCSC"
+F 21 "0.7137$" H 5450 3500 50  0001 C CNN "price100_LCSC"
+F 22 "FU007" H 5450 3500 50  0001 C CNN "Koncar"
+F 23 "T" H 5450 3500 50  0001 C CNN "Side"
 	1    5450 3500
 	1    0    0    -1

Commit message: schematics: PN update
Parts:
- U9: Mouse_r1 913-4816M16A2TG6AGTR -> (none); Mouse_r2 870-IS42S16160G7TLTR -> 913-4816M16A2TG6AGTR; price100_Mouse_r2 (none) -> 1.6€; price100_Mouser 1.6€ -> (none)
Changed lines of the file:
@@
 F 14 "AS4C32M16SB-7TCN" H 5450 3500 50  0001 C CNN "MPN4"
 F 15 "913-AS4C32M16SB-7TCN" H 5450 3500 50  0001 C CNN "Mouser"
-F 16 "913-4816M16A2TG6AGTR" H 5450 3500 60  0001 C CNN "Mouse_r1"
-F 17 "1.6€" H 5450 3500 50  0001 C CNN "price100_Mouser"
-F 18 "870-IS42S16160G7TLTR" H 5450 3500 50  0001 C CNN "Mouse_r2"
-F 19 "1450-1352-1-ND" H 5450 3500 50  0001 C CNN "Digikey"
-F 20 "C62379" H 5450 3500 50  0001 C CNN "LCSC"
-F 21 "0.7137$" H 5450 3500 50  0001 C CNN "price100_LCSC"
-F 22 "FU007" H 5450 3500 50  0001 C CNN "Koncar"
-F 23 "T" H 5450 3500 50  0001 C CNN "Side"
+F 16 "913-4816M16A2TG6AGTR" H 5450 3500 60  0001 C CNN "Mouse_r2"
+F 17 "1.6€" H 5450 3500 50  0001 C CNN "price100_Mouse_r2"
+F 18 "1450-1352-1-ND" H 5450 3500 50  0001 C CNN "Digikey"
+F 19 "C62379" H 5450 3500 50  0001 C CNN "LCSC"
+F 20 "0.7137$" H 5450 3500 50  0001 C CNN "price100_LCSC"
+F 21 "FU007" H 5450 3500 50  0001 C CNN "Koncar"
+F 22 "T" H 5450 3500 50  0001 C CNN "Side"
 	1    5450 3500
 	1    0    0    -1
