File: ram.sch (KiCad schematic (older format))
At the start: 7 parts, among them U1 LFE5U-85F-6BG381C, U9 MT48LC16M16A2TG

Commit message: schematics: PN update for digikey
Parts:
- U9: Digike_y2 (none) -> 1450-1352-1-ND; Digikey 1450-1352-1-ND -> 1450-1385-1-ND
Changed lines of the file:
@@
 F 16 "913-4816M16A2TG6AGTR" H 5450 3500 60  0001 C CNN "Mouse_r2"
 F 17 "1.6€" H 5450 3500 50  0001 C CNN "price100_Mouse_r2"
-F 18 "1450-1352-1-ND" H 5450 3500 50  0001 C CNN "Digikey"
-F 19 "C62379" H 5450 3500 50  0001 C CNN "LCSC"
-F 20 "0.7137$" H 5450 3500 50  0001 C CNN "price100_LCSC"
-F 21 "FU007" H 5450 3500 50  0001 C CNN "Koncar"
-F 22 "T" H 5450 3500 50  0001 C CNN "Side"
+F 18 "1450-1385-1-ND" H 5450 3500 50  0001 C CNN "Digikey"
+F 19 "1450-1352-1-ND" H 5450 3500 50  0001 C CNN "Digike_y2"
+F 20 "C62379" H 5450 3500 50  0001 C CNN "LCSC"
+F 21 "0.7137$" H 5450 3500 50  0001 C CNN "price100_LCSC"
+F 22 "FU007" H 5450 3500 50  0001 C CNN "Koncar"
+F 23 "T" H 5450 3500 50  0001 C CNN "Side"
 	1    5450 3500
 	1    0    0    -1

Commit message: schematics: PN update
Parts:
- U1: Mouser_URL www.mouser.com -> (none)
Changed lines of the file:
@@
 F 3 "http://www.latticesemi.com/~/media/LatticeSemi/Documents/DataSheets/ECP5/FPGA-DS-02012.pdf" H 8250 4100 60  0001 C CNN
 F 4 "LFE5U-85F-6BG381C" H 9300 3150 60  0001 C CNN "MPN"
-F 5 "www.mouser.com" H 9300 3150 60  0001 C CNN "Mouser_URL"
-F 6 "842-LFE5U85F6BG381C" H 9300 3150 60  0001 C CNN "Mouser"
+F 5 "842-LFE5U85F6BG381C" H 9300 3150 60  0001 C CNN "Mouser"
 	3    9300 3150
 	1    0    0    -1
@@
 F 3 "http://www.latticesemi.com/~/media/LatticeSemi/Documents/DataSheets/ECP5/FPGA-DS-02012.pdf" H 8250 6200 60  0001 C CNN
 F 4 "LFE5U-85F-6BG381C" H 9300 5250 60  0001 C CNN "MPN"
-F 5 "www.mouser.com" H 9300 5250 60  0001 C CNN "Mouser_URL"
-F 6 "842-LFE5U85F6BG381C" H 9300 5250 60  0001 C CNN "Mouser"
+F 5 "842-LFE5U85F6BG381C" H 9300 5250 60  0001 C CNN "Mouser"
 	4    9300 5250
 	1    0    0    -1

Commit message: schematics: SDRAM winbond 32MB mouser PN
Parts:
- U9: Mouse_r1 (none) -> 454-W9825G6KH-6
Changed lines of the file:
@@
 F 14 "AS4C32M16SB-7TCN" H 5450 3500 50  0001 C CNN "MPN4"
 F 15 "913-AS4C32M16SB-7TCN" H 5450 3500 50  0001 C CNN "Mouser"
-F 16 "913-4816M16A2TG6AGTR" H 5450 3500 60  0001 C CNN "Mouse_r2"
-F 17 "1.6€" H 5450 3500 50  0001 C CNN "price100_Mouse_r2"
-F 18 "1450-1385-1-ND" H 5450 3500 50  0001 C CNN "Digikey"
-F 19 "1450-1352-1-ND" H 5450 3500 50  0001 C CNN "Digike_y2"
-F 20 "C62379" H 5450 3500 50  0001 C CNN "LCSC"
-F 21 "0.7137$" H 5450 3500 50  0001 C CNN "price100_LCSC"
-F 22 "FU007" H 5450 3500 50  0001 C CNN "Koncar"
-F 23 "T" H 5450 3500 50  0001 C CNN "Side"
+F 16 "454-W9825G6KH-6" H 5450 3500 50  0001 C CNN "Mouse_r1"
+F 17 "913-4816M16A2TG6AGTR" H 5450 3500 60  0001 C CNN "Mouse_r2"
+F 18 "1.6€" H 5450 3500 50  0001 C CNN "price100_Mouse_r2"
+F 19 "1450-1385-1-ND" H 5450 3500 50  0001 C CNN "Digikey"
+F 20 "1450-1352-1-ND" H 5450 3500 50  0001 C CNN "Digike_y2"
+F 21 "C62379" H 5450 3500 50  0001 C CNN "LCSC"
+F 22 "0.7137$" H 5450 3500 50  0001 C CNN "price100_LCSC"
+F 23 "FU007" H 5450 3500 50  0001 C CNN "Koncar"
+F 24 "T" H 5450 3500 50  0001 C CNN "Side"
 	1    5450 3500
 	1    0    0    -1

Commit message: schematics: LCSC RAM update
Parts:
- U9: LCSC C62379 -> C492195; LCS_C1 (none) -> C524867; MPN5 (none) -> M12L2561616A-6TG2T
Changed lines of the file:
@@
 F 13 "Alliance" H 5450 3500 50  0001 C CNN "MFG4"
 F 14 "AS4C32M16SB-7TCN" H 5450 3500 50  0001 C CNN "MPN4"
-F 15 "913-AS4C32M16SB-7TCN" H 5450 3500 50  0001 C CNN "Mouser"
-F 16 "454-W9825G6KH-6" H 5450 3500 50  0001 C CNN "Mouse_r1"
-F 17 "913-4816M16A2TG6AGTR" H 5450 3500 60  0001 C CNN "Mouse_r2"
-F 18 "1.6€" H 5450 3500 50  0001 C CNN "price100_Mouse_r2"
-F 19 "1450-1385-1-ND" H 5450 3500 50  0001 C CNN "Digikey"
-F 20 "1450-1352-1-ND" H 5450 3500 50  0001 C CNN "Digike_y2"
-F 21 "C62379" H 5450 3500 50  0001 C CNN "LCSC"
-F 22 "0.7137$" H 5450 3500 50  0001 C CNN "price100_LCSC"
-F 23 "FU007" H 5450 3500 50  0001 C CNN "Koncar"
-F 24 "T" H 5450 3500 50  0001 C CNN "Side"
+F 15 "M12L2561616A-6TG2T" H 5450 3500 50  0001 C CNN "MPN5"
+F 16 "913-AS4C32M16SB-7TCN" H 5450 3500 50  0001 C CNN "Mouser"
+F 17 "454-W9825G6KH-6" H 5450 3500 50  0001 C CNN "Mouse_r1"
+F 18 "913-4816M16A2TG6AGTR" H 5450 3500 60  0001 C CNN "Mouse_r2"
+F 19 "1.6€" H 5450 3500 50  0001 C CNN "price100_Mouse_r2"
+F 20 "1450-1385-1-ND" H 5450 3500 50  0001 C CNN "Digikey"
+F 21 "1450-1352-1-ND" H 5450 3500 50  0001 C CNN "Digike_y2"
+F 22 "C492195" H 5450 3500 50  0001 C CNN "LCSC"
+F 23 "C524867" H 5450 3500 50  0001 C CNN "LCS_C1"
+F 24 "0.7137$" H 5450 3500 50  0001 C CNN "price100_LCSC"
+F 25 "FU007" H 5450 3500 50  0001 C CNN "Koncar"
+F 26 "T" H 5450 3500 50  0001 C CNN "Side"
 	1    5450 3500
 	1    0    0    -1

Commit message: schematics: RAM PN for LCSC
Parts:
- U9: MPN3 W9812G6KH-6 -> (none); MP_N3 (none) -> W9812G6KH-6; price100_LCSC 0.7137$ -> (none); price500_LCSC (none) -> 0.9227$
Changed lines of the file:
@@
 F 9 "IS42S16160G-7TL-TR" H 5450 3500 50  0001 C CNN "MPN2"
 F 10 "Winbond" H 5450 3500 50  0001 C CNN "MFG3"
-F 11 "W9812G6KH-6" H 5450 3500 50  0001 C CNN "MPN3"
+F 11 "W9812G6KH-6" H 5450 3500 50  0001 C CNN "MP_N3"
 F 12 "https://www.alliancememory.com/wp-content/uploads/pdf/dram/512M%20SDRAM_%20B%20die_AS4C32M16SB-7TCN-7TIN-6TIN_Rev%201.0%20June%202016.pdf" H 5450 3500 50  0001 C CNN "Datasheet4"
 F 13 "Alliance" H 5450 3500 50  0001 C CNN "MFG4"
@@
 F 22 "C492195" H 5450 3500 50  0001 C CNN "LCSC"
 F 23 "C524867" H 5450 3500 50  0001 C CNN "LCS_C1"
-F 24 "0.7137$" H 5450 3500 50  0001 C CNN "price100_LCSC"
+F 24 "0.9227$" H 5450 3500 50  0001 C CNN "price500_LCSC"
 F 25 "FU007" H 5450 3500 50  0001 C CNN "Koncar"
 F 26 "T" H 5450 3500 50  0001 C CNN "Side"

Commit message: schematics: RAM mouser PN update, 64MB for 10€
Parts:
- U9: Mouse_r0 (none) -> 913-AS4C32M16SB-7TCN; Mouser 913-AS4C32M16SB-7TCN -> 870-IS42S16320D-7TL
Changed lines of the file:
@@
 F 14 "AS4C32M16SB-7TCN" H 5450 3500 50  0001 C CNN "MPN4"
 F 15 "M12L2561616A-6TG2T" H 5450 3500 50  0001 C CNN "MPN5"
-F 16 "913-AS4C32M16SB-7TCN" H 5450 3500 50  0001 C CNN "Mouser"
-F 17 "454-W9825G6KH-6" H 5450 3500 50  0001 C CNN "Mouse_r1"
-F 18 "913-4816M16A2TG6AGTR" H 5450 3500 60  0001 C CNN "Mouse_r2"
-F 19 "1.6€" H 5450 3500 50  0001 C CNN "price100_Mouse_r2"
-F 20 "1450-1385-1-ND" H 5450 3500 50  0001 C CNN "Digikey"
-F 21 "1450-1352-1-ND" H 5450 3500 50  0001 C CNN "Digike_y2"
-F 22 "C492195" H 5450 3500 50  0001 C CNN "LCSC"
-F 23 "C524867" H 5450 3500 50  0001 C CNN "LCS_C1"
-F 24 "0.9227$" H 5450 3500 50  0001 C CNN "price500_LCSC"
-F 25 "FU007" H 5450 3500 50  0001 C CNN "Koncar"
-F 26 "T" H 5450 3500 50  0001 C CNN "Side"
+F 16 "870-IS42S16320D-7TL" H 5450 3500 50  0001 C CNN "Mouser"
+F 17 "913-AS4C32M16SB-7TCN" H 5450 3500 50  0001 C CNN "Mouse_r0"
+F 18 "454-W9825G6KH-6" H 5450 3500 50  0001 C CNN "Mouse_r1"
+F 19 "913-4816M16A2TG6AGTR" H 5450 3500 60  0001 C CNN "Mouse_r2"
+F 20 "1.6€" H 5450 3500 50  0001 C CNN "price100_Mouse_r2"
+F 21 "1450-1385-1-ND" H 5450 3500 50  0001 C CNN "Digikey"
+F 22 "1450-1352-1-ND" H 5450 3500 50  0001 C CNN "Digike_y2"
+F 23 "C492195" H 5450 3500 50  0001 C CNN "LCSC"
+F 24 "C524867" H 5450 3500 50  0001 C CNN "LCS_C1"
+F 25 "0.9227$" H 5450 3500 50  0001 C CNN "price500_LCSC"
+F 26 "FU007" H 5450 3500 50  0001 C CNN "Koncar"
+F 27 "T" H 5450 3500 50  0001 C CNN "Side"
 	1    5450 3500
 	1    0    0    -1
